File: VariClock1.kicad_sch (KiCad schematic)
At the start: 71 parts, among them U32 40106, U33 4013, U34 40106, U35 40193, U36 TL074, U37 4042, U38 40193

Commit message: more work...
Parts:
- C2, C6, C7: footprint Capacitor_SMD:C_0805_2012Metric_Pad1.18x1.45mm_HandSolder -> Capacitor_SMD:C_0603_1608Metric
- C2, C3, C4, C5: footprint Capacitor_SMD:C_0805_2012Metric_Pad1.18x1.45mm_HandSolder -> Capacitor_SMD:C_0805_2012Metric
- C? (x4): footprint Capacitor_SMD:C_0805_2012Metric -> Capacitor_SMD:C_0603_1608Metric
- R? (x32): footprint Resistor_SMD:R_0805_2012Metric -> Resistor_SMD:R_0603_1608Metric
- U32, U33, U34: footprint (none) -> Package_SO:SOIC-14_3.9x8.7mm_P1.27mm
- U35, U38: footprint (none) -> Package_SO:SOIC-16W_5.3x10.2mm_P1.27mm
- U36: footprint (none) -> Package_SO:SO-14_3.9x8.65mm_P1.27mm
- U37: footprint (none) -> Package_SO:SOP-16_3.9x9.9mm_P1.27mm

Commit message: finishing schematic 1.0
Parts:
- renumbered C2 to C?, C4 to C?, C5 to C?, C3 to C?, C6 to C?, C7 to C?, D30 to D?, RV30 to RV?, U34 to U32, U32 to U34
