File: VariClock2.kicad_sch (KiCad schematic)
At the start: 29 parts, among them Q25 2N3904, Q26 2N3906, Q27 2N3904, SW11 SW_SPDT, U32 40106, U36 TL074, U37 4013

Commit message: more work...
Parts:
- C2, C3, C4, C5: footprint Capacitor_SMD:C_0805_2012Metric_Pad1.18x1.45mm_HandSolder -> Capacitor_SMD:C_0805_2012Metric
- C6, C7: footprint Capacitor_SMD:C_0805_2012Metric_Pad1.18x1.45mm_HandSolder -> Capacitor_SMD:C_0603_1608Metric
- R? (x9): footprint Resistor_SMD:R_0805_2012Metric -> Resistor_SMD:R_0603_1608Metric
- U32, U37: footprint (none) -> Package_SO:SOIC-14_3.9x8.7mm_P1.27mm
- U36: footprint (none) -> Package_SO:SO-14_3.9x8.65mm_P1.27mm
Changed lines of the file:
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@@
       (effects (font (size 1.27 1.27)))
     )
-    (property "Footprint" "Resistor_SMD:R_0805_2012Metric" (at 169.164 77.089 90)
+    (property "Footprint" "Resistor_SMD:R_0603_1608Metric" (at 169.164 77.089 90)
       (effects (font (size 1.27 1.27)) hide)
     )
@@
       (effects (font (size 1.27 1.27)))
     )
-    (property "Footprint" "Capacitor_SMD:C_0805_2012Metric_Pad1.18x1.45mm_HandSolder" (at 157.7848 179.07 0)
+    (property "Footprint" "Capacitor_SMD:C_0603_1608Metric" (at 157.7848 179.07 0)
       (effects (font (size 1.27 1.27)) hide)
     )
@@
       (effects (font (size 1.27 1.27)))
     )
-    (property "Footprint" "Capacitor_SMD:C_0805_2012Metric_Pad1.18x1.45mm_HandSolder" (at 118.4148 40.64 0)
+    (property "Footprint" "Capacitor_SMD:C_0603_1608Metric" (at 118.4148 40.64 0)
       (effects (font (size 1.27 1.27)) hide)
     )
@@
       (effects (font (size 1.27 1.27)))
     )
-    (property "Footprint" "Resistor_SMD:R_0805_2012Metric" (at 188.214 115.189 90)
+    (property "Footprint" "Resistor_SMD:R_0603_1608Metric" (at 188.214 115.189 90)
       (effects (font (size 1.27 1.27)) hide)
     )
@@
       (effects (font (size 1.27 1.27)))
     )
-    (property "Footprint" "Capacitor_SMD:C_0805_2012Metric_Pad1.18x1.45mm_HandSolder" (at 145.0848 171.45 0)
+    (property "Footprint" "Capacitor_SMD:C_0805_2012Metric" (at 145.0848 171.45 0)
       (effects (font (size 1.27 1.27)) hide)
     )
@@
       (effects (font (size 1.27 1.27)))
     )
-    (property "Footprint" "Capacitor_SMD:C_0805_2012Metric_Pad1.18x1.45mm_HandSolder" (at 145.0848 179.07 0)
+    (property "Footprint" "Capacitor_SMD:C_0805_2012Metric" (at 145.0848 179.07 0)
       (effects (font (size 1.27 1.27)) hide)
     )
@@
       (effects (font (size 1.27 1.27)))
     )
-    (property "Footprint" "Resistor_SMD:R_0805_2012Metric" (at 148.209 96.774 90)
+    (property "Footprint" "Resistor_SMD:R_0603_1608Metric" (at 148.209 96.774 90)
       (effects (font (size 1.27 1.27)) hide)
     )
@@
       (effects (font (size 1.27 1.27)))
     )
-    (property "Footprint" "Resistor_SMD:R_0805_2012Metric" (at 204.089 79.121 90)
+    (property "Footprint" "Resistor_SMD:R_0603_1608Metric" (at 204.089 79.121 90)
       (effects (font (size 1.27 1.27)) hide)
     )
@@
       (effects (font (size 1.27 1.27)))
     )
-    (property "Footprint" "Resistor_SMD:R_0805_2012Metric" (at 143.764 124.714 90)
+    (property "Footprint" "Resistor_SMD:R_0603_1608Metric" (at 143.764 124.714 90)
       (effects (font (size 1.27 1.27)) hide)
     )
@@
       (effects (font (size 1.27 1.27)))
     )
-    (property "Footprint" "Capacitor_SMD:C_0805_2012Metric_Pad1.18x1.45mm_HandSolder" (at 157.7848 171.45 0)
+    (property "Footprint" "Capacitor_SMD:C_0603_1608Metric" (at 157.7848 171.45 0)
       (effects (font (size 1.27 1.27)) hide)
     )
@@
       (effects (font (size 1.27 1.27)))
     )
-    (property "Footprint" "Resistor_SMD:R_0805_2012Metric" (at 143.764 134.239 90)
+    (property "Footprint" "Resistor_SMD:R_0603_1608Metric" (at 143.764 134.239 90)
       (effects (font (size 1.27 1.27)) hide)
     )
@@
       (effects (font (size 1.27 1.27)))
     )
-    (property "Footprint" "Resistor_SMD:R_0805_2012Metric" (at 169.164 48.641 90)
+    (property "Footprint" "Resistor_SMD:R_0603_1608Metric" (at 169.164 48.641 90)
       (effects (font (size 1.27 1.27)) hide)
     )
@@
       (effects (font (size 1.27 1.27)))
     )
-    (property "Footprint" "" (at 136.525 97.79 0)
+    (property "Footprint" "Package_SO:SOIC-14_3.9x8.7mm_P1.27mm" (at 136.525 97.79 0)
       (effects (font (size 1.27 1.27)) hide)
     )
@@
       (effects (font (size 1.27 1.27)))
     )
-    (property "Footprint" "Resistor_SMD:R_0805_2012Metric" (at 120.396 52.324 90)
+    (property "Footprint" "Resistor_SMD:R_0603_1608Metric" (at 120.396 52.324 90)
       (effects (font (size 1.27 1.27)) hide)
     )
@@
       (effects (font (size 1.27 1.27)) (justify left))
     )
-    (property "Footprint" "" (at 130.175 64.135 0)
+    (property "Footprint" "Package_SO:SOIC-14_3.9x8.7mm_P1.27mm" (at 130.175 64.135 0)
       (effects (font (size 1.27 1.27)) hide)
     )
@@
       (effects (font (size 1.27 1.27)))
     )
-    (property "Footprint" "Capacitor_SMD:C_0805_2012Metric_Pad1.18x1.45mm_HandSolder" (at 151.4348 179.07 0)
+    (property "Footprint" "Capacitor_SMD:C_0805_2012Metric" (at 151.4348 179.07 0)
       (effects (font (size 1.27 1.27)) hide)
     )
@@
       (effects (font (size 1.27 1.27)))
     )
-    (property "Footprint" "" (at 164.465 116.205 0)
+    (property "Footprint" "Package_SO:SOIC-14_3.9x8.7mm_P1.27mm" (at 164.465 116.205 0)
       (effects (font (size 1.27 1.27)) hide)
     )
@@
       (effects (font (size 1.27 1.27)))
     )
-    (property "Footprint" "" (at 118.11 167.64 0)
+    (property "Footprint" "Package_SO:SO-14_3.9x8.65mm_P1.27mm" (at 118.11 167.64 0)
       (effects (font (size 1.27 1.27)) hide)
     )
@@
       (effects (font (size 1.27 1.27)))
     )
-    (property "Footprint" "Resistor_SMD:R_0805_2012Metric" (at 161.544 77.089 90)
+    (property "Footprint" "Resistor_SMD:R_0603_1608Metric" (at 161.544 77.089 90)
       (effects (font (size 1.27 1.27)) hide)
     )
@@
       (effects (font (size 1.27 1.27)))
     )
-    (property "Footprint" "Capacitor_SMD:C_0805_2012Metric_Pad1.18x1.45mm_HandSolder" (at 151.4348 171.45 0)
-      (effects (font (size 1.27 1.27)) hide)
-    )
+    (property "Footprint" "Capacitor_SMD:C_0805_2012Metric" (at 151.4348 171.45 0)
+      (effects (font (size 1.27 1.27)) hide)
+    )

Commit message: finishing schematic 1.0
Parts:
- SW?: footprint (none) -> SynthProjConnectors:MTS-203-A1-T0
- SW? (x2): renamed from SW11; footprint SynthProjConnectors:ST-0-102-A01-T000-LF -> SynthProjConnectors:MTS-103-A01-T0
- renumbered C7 to C?, C6 to C?, C2 to C?, C3 to C?, C5 to C?, C4 to C?, D30 to D?, U32 to U?, U37 to U?, U36 to U?
