File: VariClock3.kicad_sch (KiCad schematic)
At the start: 24 parts, among them U39 CD74HC4067SM

Commit message: more work...
Parts:
- C2, C3, C4, C5: footprint Capacitor_SMD:C_0805_2012Metric_Pad1.18x1.45mm_HandSolder -> Capacitor_SMD:C_0805_2012Metric
- C2, C6, C7: footprint Capacitor_SMD:C_0805_2012Metric_Pad1.18x1.45mm_HandSolder -> Capacitor_SMD:C_0603_1608Metric
Changed lines of the file:
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@@
       (effects (font (size 1.27 1.27)))
     )
-    (property "Footprint" "Capacitor_SMD:C_0805_2012Metric_Pad1.18x1.45mm_HandSolder" (at 93.6498 138.43 0)
+    (property "Footprint" "Capacitor_SMD:C_0805_2012Metric" (at 93.6498 138.43 0)
       (effects (font (size 1.27 1.27)) hide)
     )
@@
       (effects (font (size 1.27 1.27)))
     )
-    (property "Footprint" "Capacitor_SMD:C_0805_2012Metric_Pad1.18x1.45mm_HandSolder" (at 93.6498 146.05 0)
+    (property "Footprint" "Capacitor_SMD:C_0805_2012Metric" (at 93.6498 146.05 0)
       (effects (font (size 1.27 1.27)) hide)
     )
@@
       (effects (font (size 1.27 1.27)))
     )
-    (property "Footprint" "Capacitor_SMD:C_0805_2012Metric_Pad1.18x1.45mm_HandSolder" (at 106.3498 138.43 0)
+    (property "Footprint" "Capacitor_SMD:C_0603_1608Metric" (at 106.3498 138.43 0)
       (effects (font (size 1.27 1.27)) hide)
     )
@@
       (effects (font (size 1.27 1.27)))
     )
-    (property "Footprint" "Capacitor_SMD:C_0805_2012Metric_Pad1.18x1.45mm_HandSolder" (at 99.9998 146.05 0)
+    (property "Footprint" "Capacitor_SMD:C_0805_2012Metric" (at 99.9998 146.05 0)
       (effects (font (size 1.27 1.27)) hide)
     )
@@
       (effects (font (size 1.27 1.27)))
     )
-    (property "Footprint" "Capacitor_SMD:C_0805_2012Metric_Pad1.18x1.45mm_HandSolder" (at 106.3498 146.05 0)
+    (property "Footprint" "Capacitor_SMD:C_0603_1608Metric" (at 106.3498 146.05 0)
       (effects (font (size 1.27 1.27)) hide)
     )
@@
       (effects (font (size 1.27 1.27)))
     )
-    (property "Footprint" "Capacitor_SMD:C_0805_2012Metric_Pad1.18x1.45mm_HandSolder" (at 139.3698 50.8 0)
+    (property "Footprint" "Capacitor_SMD:C_0603_1608Metric" (at 139.3698 50.8 0)
       (effects (font (size 1.27 1.27)) hide)
     )
@@
       (effects (font (size 1.27 1.27)))
     )
-    (property "Footprint" "Capacitor_SMD:C_0805_2012Metric_Pad1.18x1.45mm_HandSolder" (at 99.9998 138.43 0)
-      (effects (font (size 1.27 1.27)) hide)
-    )
+    (property "Footprint" "Capacitor_SMD:C_0805_2012Metric" (at 99.9998 138.43 0)
+      (effects (font (size 1.27 1.27)) hide)
+    )

Commit message: finishing schematic 1.0
Parts:
- renumbered C2 to C?, C3 to C?, C6 to C?, C5 to C?, C7 to C?, C4 to C?
