File: page1.kicad_sch (KiCad schematic)
At the start: 84 parts

Commit message: more work...
Parts:
- C? (x13): footprint Capacitor_SMD:C_0805_2012Metric -> Capacitor_SMD:C_0603_1608Metric
- R? (x31): footprint Resistor_SMD:R_0805_2012Metric -> Resistor_SMD:R_0603_1608Metric

Commit message: finishing schematic 1.0
Parts:
- SW? (x4): footprint (none) -> Button_Switch_THT:SW_PUSH_6mm_H13mm
