File: page2.kicad_sch (KiCad schematic)
At the start: 74 parts

Commit message: more work...
Parts:
- C? (x5): footprint Capacitor_SMD:C_0805_2012Metric -> Capacitor_SMD:C_0603_1608Metric
- R? (x6): footprint Resistor_SMD:R_0805_2012Metric -> Resistor_SMD:R_0603_1608Metric
Changed lines of the file:
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@@
       (effects (font (size 1.27 1.27)) (justify left))
     )
-    (property "Footprint" "Capacitor_SMD:C_0805_2012Metric" (at 60.6552 161.925 0)
+    (property "Footprint" "Capacitor_SMD:C_0603_1608Metric" (at 60.6552 161.925 0)
       (effects (font (size 1.27 1.27)) hide)
     )
@@
       (effects (font (size 1.27 1.27)) (justify left))
     )
-    (property "Footprint" "Resistor_SMD:R_0805_2012Metric" (at 135.636 32.004 90)
+    (property "Footprint" "Resistor_SMD:R_0603_1608Metric" (at 135.636 32.004 90)
       (effects (font (size 1.27 1.27)) hide)
     )
@@
       (effects (font (size 1.27 1.27)))
     )
-    (property "Footprint" "Resistor_SMD:R_0805_2012Metric" (at 254.889 98.679 90)
+    (property "Footprint" "Resistor_SMD:R_0603_1608Metric" (at 254.889 98.679 90)
       (effects (font (size 1.27 1.27)) hide)
     )
@@
       (effects (font (size 1.27 1.27)) (justify left))
     )
-    (property "Footprint" "Capacitor_SMD:C_0805_2012Metric" (at 60.6552 154.305 0)
+    (property "Footprint" "Capacitor_SMD:C_0603_1608Metric" (at 60.6552 154.305 0)
       (effects (font (size 1.27 1.27)) hide)
     )
@@
       (effects (font (size 1.27 1.27)))
     )
-    (property "Footprint" "Capacitor_SMD:C_0805_2012Metric" (at 241.935 112.0648 0)
+    (property "Footprint" "Capacitor_SMD:C_0603_1608Metric" (at 241.935 112.0648 0)
       (effects (font (size 1.27 1.27)) hide)
     )
@@
       (effects (font (size 1.27 1.27)) (justify left))
     )
-    (property "Footprint" "Resistor_SMD:R_0805_2012Metric" (at 204.216 103.759 90)
+    (property "Footprint" "Resistor_SMD:R_0603_1608Metric" (at 204.216 103.759 90)
       (effects (font (size 1.27 1.27)) hide)
     )
@@
       (effects (font (size 1.27 1.27)) (justify right))
     )
-    (property "Footprint" "Capacitor_SMD:C_0805_2012Metric" (at 263.8298 113.03 0)
+    (property "Footprint" "Capacitor_SMD:C_0603_1608Metric" (at 263.8298 113.03 0)
       (effects (font (size 1.27 1.27)) hide)
     )
@@
       (effects (font (size 1.27 1.27)) (justify right))
     )
-    (property "Footprint" "Resistor_SMD:R_0805_2012Metric" (at 240.919 120.396 90)
+    (property "Footprint" "Resistor_SMD:R_0603_1608Metric" (at 240.919 120.396 90)
       (effects (font (size 1.27 1.27)) hide)
     )
@@
       (effects (font (size 1.27 1.27)) (justify right))
     )
-    (property "Footprint" "Capacitor_SMD:C_0805_2012Metric" (at 257.4798 99.695 0)
+    (property "Footprint" "Capacitor_SMD:C_0603_1608Metric" (at 257.4798 99.695 0)
       (effects (font (size 1.27 1.27)) hide)
     )
@@
       (effects (font (size 1.27 1.27)))
     )
-    (property "Footprint" "Resistor_SMD:R_0805_2012Metric" (at 261.239 112.014 90)
+    (property "Footprint" "Resistor_SMD:R_0603_1608Metric" (at 261.239 112.014 90)
       (effects (font (size 1.27 1.27)) hide)
     )
@@
       (effects (font (size 1.27 1.27)))
     )
-    (property "Footprint" "Resistor_SMD:R_0805_2012Metric" (at 212.344 98.679 90)
-      (effects (font (size 1.27 1.27)) hide)
-    )
+    (property "Footprint" "Resistor_SMD:R_0603_1608Metric" (at 212.344 98.679 90)
+      (effects (font (size 1.27 1.27)) hide)
+    )

Commit message: finishing schematic 1.0
Parts:
- SW28: value ~ -> SRBV141404; footprint (none) -> SynthProjConnectors:SRBV141404
- SW? (x16): footprint (none) -> SynthProjConnectors:MTS-103-A01-T0
- SW?: value SW_Rotary12 -> SR2612F-0112-21R0B-D8-N; footprint (none) -> SynthProjConnectors:SR2612F-0112
- SW?: footprint (none) -> SynthProjConnectors:MTS-203-A1-T0
Other:
- note added: "16 step sequence"
- note added: "Reset @ Count"
- note added: "Reverse @ Count"
- note added: "Stop @ Count"
