File: page3.kicad_sch (KiCad schematic)
At the start: 27 parts

Commit message: more work...
Parts:
- C? (x5): footprint Capacitor_SMD:C_0805_2012Metric -> Capacitor_SMD:C_0603_1608Metric
- R? (x9): footprint Resistor_SMD:R_0805_2012Metric -> Resistor_SMD:R_0603_1608Metric
- U23: value ~ -> CD4094; footprint (none) -> Package_SO:SOP-16_3.9x9.9mm_P1.27mm
Changed lines of the file:
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@@
       (effects (font (size 1.27 1.27)) (justify right))
     )
-    (property "Footprint" "Capacitor_SMD:C_0805_2012Metric" (at 123.4948 83.82 0)
+    (property "Footprint" "Capacitor_SMD:C_0603_1608Metric" (at 123.4948 83.82 0)
       (effects (font (size 1.27 1.27)) hide)
     )
@@
       (effects (font (size 1.27 1.27)))
     )
-    (property "Footprint" "Capacitor_SMD:C_0805_2012Metric" (at 172.72 106.3752 0)
+    (property "Footprint" "Capacitor_SMD:C_0603_1608Metric" (at 172.72 106.3752 0)
       (effects (font (size 1.27 1.27)) hide)
     )
@@
       (effects (font (size 1.27 1.27)))
     )
-    (property "Footprint" "Resistor_SMD:R_0805_2012Metric" (at 120.396 84.836 90)
+    (property "Footprint" "Resistor_SMD:R_0603_1608Metric" (at 120.396 84.836 90)
       (effects (font (size 1.27 1.27)) hide)
     )
@@
       (effects (font (size 1.27 1.27)) (justify right))
     )
-    (property "Footprint" "Resistor_SMD:R_0805_2012Metric" (at 82.169 89.916 90)
+    (property "Footprint" "Resistor_SMD:R_0603_1608Metric" (at 82.169 89.916 90)
       (effects (font (size 1.27 1.27)) hide)
     )
@@
       (effects (font (size 1.27 1.27)) (justify left))
     )
-    (property "Value" "~" (at 179.07 86.36 0)
-      (effects (font (size 1.27 1.27)))
-    )
-    (property "Footprint" "" (at 179.07 86.36 0)
+    (property "Value" "CD4094" (at 179.07 86.36 0)
+      (effects (font (size 1.27 1.27)))
+    )
+    (property "Footprint" "Package_SO:SOP-16_3.9x9.9mm_P1.27mm" (at 179.07 86.36 0)
       (effects (font (size 1.27 1.27)) hide)
     )
@@
       (effects (font (size 1.27 1.27)) (justify right))
     )
-    (property "Footprint" "Resistor_SMD:R_0805_2012Metric" (at 179.324 108.966 90)
+    (property "Footprint" "Resistor_SMD:R_0603_1608Metric" (at 179.324 108.966 90)
       (effects (font (size 1.27 1.27)) hide)
     )
@@
       (effects (font (size 1.27 1.27)) (justify right))
     )
-    (property "Footprint" "Resistor_SMD:R_0805_2012Metric" (at 148.844 84.836 90)
+    (property "Footprint" "Resistor_SMD:R_0603_1608Metric" (at 148.844 84.836 90)
       (effects (font (size 1.27 1.27)) hide)
     )
@@
       (effects (font (size 1.27 1.27)) (justify left))
     )
-    (property "Footprint" "Capacitor_SMD:C_0805_2012Metric" (at 87.9602 143.51 0)
+    (property "Footprint" "Capacitor_SMD:C_0603_1608Metric" (at 87.9602 143.51 0)
       (effects (font (size 1.27 1.27)) hide)
     )
@@
       (effects (font (size 1.27 1.27)) (justify right))
     )
-    (property "Footprint" "Resistor_SMD:R_0805_2012Metric" (at 92.964 106.426 90)
+    (property "Footprint" "Resistor_SMD:R_0603_1608Metric" (at 92.964 106.426 90)
       (effects (font (size 1.27 1.27)) hide)
     )
@@
       (effects (font (size 1.27 1.27)))
     )
-    (property "Footprint" "Resistor_SMD:R_0805_2012Metric" (at 120.396 79.756 90)
+    (property "Footprint" "Resistor_SMD:R_0603_1608Metric" (at 120.396 79.756 90)
       (effects (font (size 1.27 1.27)) hide)
     )
@@
       (effects (font (size 1.27 1.27)))
     )
-    (property "Footprint" "Resistor_SMD:R_0805_2012Metric" (at 101.346 96.266 90)
+    (property "Footprint" "Resistor_SMD:R_0603_1608Metric" (at 101.346 96.266 90)
       (effects (font (size 1.27 1.27)) hide)
     )
@@
       (effects (font (size 1.27 1.27)) (justify right))
     )
-    (property "Footprint" "Capacitor_SMD:C_0805_2012Metric" (at 149.5298 130.81 0)
+    (property "Footprint" "Capacitor_SMD:C_0603_1608Metric" (at 149.5298 130.81 0)
       (effects (font (size 1.27 1.27)) hide)
     )
@@
       (effects (font (size 1.27 1.27)) (justify right))
     )
-    (property "Footprint" "Resistor_SMD:R_0805_2012Metric" (at 67.564 75.946 90)
+    (property "Footprint" "Resistor_SMD:R_0603_1608Metric" (at 67.564 75.946 90)
       (effects (font (size 1.27 1.27)) hide)
     )
@@
       (effects (font (size 1.27 1.27)) (justify left))
     )
-    (property "Footprint" "Capacitor_SMD:C_0805_2012Metric" (at 87.9602 151.13 0)
+    (property "Footprint" "Capacitor_SMD:C_0603_1608Metric" (at 87.9602 151.13 0)
       (effects (font (size 1.27 1.27)) hide)
     )
@@
       (effects (font (size 1.27 1.27)))
     )
-    (property "Footprint" "Resistor_SMD:R_0805_2012Metric" (at 165.481 119.761 90)
-      (effects (font (size 1.27 1.27)) hide)
-    )
+    (property "Footprint" "Resistor_SMD:R_0603_1608Metric" (at 165.481 119.761 90)
+      (effects (font (size 1.27 1.27)) hide)
+    )

Commit message: finishing schematic 1.0
Other:
- moved on the sheet: C?, D?, Q?, R?, U23, U?A, U?B, U?C, U?F
