File: SynthProj.kicad_pcb (KiCad board)
At the start: 2 copper layers, 663 parts, among them J1 Exp CV In, J10 PWM IN, J11 Exp CV In, J12 Lin CV In, J13 Sync, J14 PWM IN, J15 Mixer Ext In, J16 Noise Out, J17 S&H_In, J18 S&H_Out, J2 LFOA_Out, J3 Gate, J4 1V/Oct CV, J5 Ext CV, J6 Master Output, J7 ADEG1_OUT, J8 ADEG2_OUT, J9 Lin CV In, Q10 MMBT3904-7-F, Q11 MMBT3904-7-F, Q12 MMBF4391LT1G, Q13 MMBT3904-7-F, Q14 MMBT3904-7-F, Q15 MMBT3906LT1G, Q16 MMBF5457, Q17 MMBF5457, Q18 MMBT3906LT1G, Q2 MMBT3904-7-F, Q26 MMBT3904-7-F, Q3 MMBT3906LT1G, Q4 MMBT3904-7-F, Q5 MMBT3906LT1G, Q7 MMBT3904-7-F, Q8 MMBT3904-7-F, Q9 MMBF4391LT1G, U1 TL072, U10 TL072, U11 TL071, U12 TL072, U13 TL072, U14 TL072, U15 TL074, U16 TL064, U17 PT2399, U18 TL074, U19 4013, U2 LM13700, U20 40106, U21 40106, U22 40193, U23 TL082, U24 40106, U25 4514, U26 TL082, U27 TL084, U28 CD74HC4067M, U29 LM13700, U3 TL072, U4 TL072, U5 TL072, U6 TL072, U7 TL072, U8 TL072, U9 LM13700

Commit message: finishing schematic 1.0
Parts:
- added C141: 4.7uF, Capacitor_SMD:C_0805_2012Metric, F.Cu at (-291.7, -355.1)
- added C142: 470nF, Capacitor_SMD:C_0805_2012Metric, F.Cu at (-291.7, -352.1)
- added C143: 47nF, Capacitor_SMD:C_0603_1608Metric, F.Cu at (-291.7, -349.1)
- added C147: 4.7uF, Capacitor_SMD:C_0805_2012Metric, F.Cu at (-291.7, -346.1)
- added C151: 100pF, Capacitor_SMD:C_0603_1608Metric, F.Cu at (-291.7, -343.1)
- added C163: 1nF, Capacitor_SMD:C_0603_1608Metric, F.Cu at (-531.2, 161.3)
- added C164: 1nF, Capacitor_SMD:C_0603_1608Metric, F.Cu at (-531.2, 164.3)
- added C165: 100pF, Capacitor_SMD:C_0603_1608Metric, F.Cu at (-520.4, 137.7)
- added C166: 680pF, Capacitor_SMD:C_0603_1608Metric, F.Cu at (-520.4, 140.7)
- added C167: 100pF, Capacitor_SMD:C_0603_1608Metric, F.Cu at (-520.4, 143.7)
- added C168: 4.7uF, Capacitor_SMD:C_0805_2012Metric, F.Cu at (-531.2, 167.3)
- added C169: 4.7uF, Capacitor_SMD:C_0805_2012Metric, F.Cu at (-531.2, 170.3)
- added C170: 470nF, Capacitor_SMD:C_0805_2012Metric, F.Cu at (-531.2, 173.3)
- added C171: 470nF, Capacitor_SMD:C_0805_2012Metric, F.Cu at (-526.3, 161.3)
- added C172: 680pF, Capacitor_SMD:C_0603_1608Metric, F.Cu at (-526.3, 164.3)
- added C173: 47nF, Capacitor_SMD:C_0603_1608Metric, F.Cu at (-526.3, 167.3)
- added C174: 47nF, Capacitor_SMD:C_0603_1608Metric, F.Cu at (-526.3, 170.3)
- added C175: 100pF, Capacitor_SMD:C_0603_1608Metric, F.Cu at (-520.4, 146.7)
- added C176: 100pF, Capacitor_SMD:C_0603_1608Metric, F.Cu at (-526.3, 173.3)
- added C177: 10pF, Capacitor_SMD:C_0603_1608Metric, F.Cu at (-521.5, 161.3)
- added C178: 22pF, Capacitor_SMD:C_0603_1608Metric, F.Cu at (-521.5, 164.3)
- added C179: 1uF, Capacitor_SMD:C_0805_2012Metric, F.Cu at (-521.5, 167.3)
- added C180: 20nF, Capacitor_SMD:C_0603_1608Metric, F.Cu at (-521.5, 170.3)
- added C181: 470pF, Capacitor_SMD:C_0603_1608Metric, F.Cu at (-924.2, 274.1)
- added C182: 4.7uF, Capacitor_SMD:C_0805_2012Metric, F.Cu at (-924.2, 277.1)
- added C183: 4.7uF, Capacitor_SMD:C_0805_2012Metric, F.Cu at (-924.2, 280.1)
- added C184: 470nF, Capacitor_SMD:C_0805_2012Metric, F.Cu at (-924.2, 283.1)
- added C185: 470nF, Capacitor_SMD:C_0805_2012Metric, F.Cu at (-924.2, 286.2)
- added C186: 47nF, Capacitor_SMD:C_0603_1608Metric, F.Cu at (-924.2, 289.2)
- added C187: 47nF, Capacitor_SMD:C_0603_1608Metric, F.Cu at (-924.2, 292.2)
- added C188: 4.7uF, Capacitor_SMD:C_0805_2012Metric, F.Cu at (-582.8, -73.1)
- added C189: 4.7uF, Capacitor_SMD:C_0805_2012Metric, F.Cu at (-582.8, -70.0)
- added C190: 470nF, Capacitor_SMD:C_0805_2012Metric, F.Cu at (-582.8, -67.0)
- added C191: 470nF, Capacitor_SMD:C_0805_2012Metric, F.Cu at (-582.8, -64.0)
- added C192: 47nF, Capacitor_SMD:C_0603_1608Metric, F.Cu at (-582.8, -61.0)
- added C193: 47nF, Capacitor_SMD:C_0603_1608Metric, F.Cu at (-582.8, -58.0)
- added C194: 100nF, Capacitor_SMD:C_0603_1608Metric, F.Cu at (-582.8, -55.0)
- added C195: 27pF, Capacitor_SMD:C_0603_1608Metric, F.Cu at (-142.2, -148.9)
- added C196: 27pF, Capacitor_SMD:C_0603_1608Metric, F.Cu at (-142.2, -146.9)
- added C197: 10uF, Capacitor_SMD:C_0805_2012Metric, F.Cu at (-127.8, -163.1)
- added C198: 100nF, Capacitor_SMD:C_0603_1608Metric, F.Cu at (-142.2, -145.0)
- added C199: 100nF, Capacitor_SMD:C_0603_1608Metric, F.Cu at (-142.2, -143.0)
- added C200: 10uF, Capacitor_SMD:C_0805_2012Metric, F.Cu at (-127.8, -160.1)
- added C201: 10uF, Capacitor_SMD:C_0805_2012Metric, F.Cu at (-127.8, -157.1)
- added C202: 100nF, Capacitor_SMD:C_0603_1608Metric, F.Cu at (-142.2, -141.0)
- added C203: 100nF, Capacitor_SMD:C_0603_1608Metric, F.Cu at (-139.3, -148.9)
- added C204: 1uF, Capacitor_SMD:C_0805_2012Metric, F.Cu at (-139.3, -146.9)
- added C205: 100nF, Capacitor_SMD:C_0603_1608Metric, F.Cu at (-139.3, -145.0)
- added C206: 1uF, Capacitor_SMD:C_0805_2012Metric, F.Cu at (-139.3, -143.0)
- added C207: 100nF, Capacitor_SMD:C_0603_1608Metric, F.Cu at (-139.3, -141.0)
- added C208: 100nF, Capacitor_SMD:C_0603_1608Metric, F.Cu at (-136.5, -148.9)
- added C209: 100nF, Capacitor_SMD:C_0603_1608Metric, F.Cu at (-136.5, -146.9)
- added C210: 100nF, Capacitor_SMD:C_0603_1608Metric, F.Cu at (-136.5, -145.0)
- added C211: 100nF, Capacitor_SMD:C_0603_1608Metric, F.Cu at (-136.5, -143.0)
- added C212: 100nF, Capacitor_SMD:C_0603_1608Metric, F.Cu at (-136.5, -141.0)
- added C213: 100nF, Capacitor_SMD:C_0603_1608Metric, F.Cu at (-132.4, -163.1)
- added C214: 100nF, Capacitor_SMD:C_0603_1608Metric, F.Cu at (-132.4, -160.1)
- added C215: 100nF, Capacitor_SMD:C_0603_1608Metric, F.Cu at (-132.4, -157.1)
- added C216: 100nF, Capacitor_SMD:C_0603_1608Metric, F.Cu at (-132.4, -154.1)
- added C217: 4.7uF, Capacitor_SMD:C_0805_2012Metric, F.Cu at (-55.3, -232.6)
- added C218: 4.7uF, Capacitor_SMD:C_0805_2012Metric, F.Cu at (-55.3, -229.6)
- added C219: 470nF, Capacitor_SMD:C_0805_2012Metric, F.Cu at (-55.3, -226.6)
- added C220: 470nF, Capacitor_SMD:C_0805_2012Metric, F.Cu at (-55.3, -223.5)
- added C221: 47nF, Capacitor_SMD:C_0603_1608Metric, F.Cu at (-55.3, -220.5)
- added C222: 47nF, Capacitor_SMD:C_0603_1608Metric, F.Cu at (-55.3, -217.5)
- added C223: 4.7uF, Capacitor_SMD:C_0805_2012Metric, F.Cu at (-93.6, -75.7)
- added C224: 470nF, Capacitor_SMD:C_0805_2012Metric, F.Cu at (-93.6, -72.7)
- added C225: 47nF, Capacitor_SMD:C_0603_1608Metric, F.Cu at (-79.5, -67.1)
- added C226: 470nF, Capacitor_SMD:C_0805_2012Metric, F.Cu at (-257.6, -87.0)
- added C227: 4.7uF, Capacitor_SMD:C_0805_2012Metric, F.Cu at (-257.6, -90.0)
- added C228: 4.7uF, Capacitor_SMD:C_0805_2012Metric, F.Cu at (-93.6, -66.7)
- added C229: 470nF, Capacitor_SMD:C_0805_2012Metric, F.Cu at (-93.6, -69.7)
- added C61: 22nF, Capacitor_SMD:C_0603_1608Metric, F.Cu at (214.3, 620.2)
- added D100: 1N914, Diode_SMD:D_SOD-323F, F.Cu at (-130.0, -144.0)
- added D101: LED, LED_SMD:LED_0805_2012Metric, F.Cu at (-138.2, -28.9)
- added D102: LED, LED_SMD:LED_0805_2012Metric, F.Cu at (-138.2, -25.9)
- added D103: LED, LED_SMD:LED_0805_2012Metric, F.Cu at (-138.2, -22.8)
- added D104: LED, LED_SMD:LED_0805_2012Metric, F.Cu at (-138.2, -19.8)
- added D105: LED, LED_SMD:LED_0805_2012Metric, F.Cu at (-133.8, -28.9)
- added D106: LED, LED_SMD:LED_0805_2012Metric, F.Cu at (-133.8, -25.9)
- added D107: LED, LED_SMD:LED_0805_2012Metric, F.Cu at (-133.8, -22.8)
- added D108: LED, LED_SMD:LED_0805_2012Metric, F.Cu at (-133.8, -19.8)
- added D109: LED, LED_SMD:LED_0805_2012Metric, F.Cu at (-129.3, -28.9)
- added D110: LED, LED_SMD:LED_0805_2012Metric, F.Cu at (-129.3, -25.9)
- added D111: LED, LED_SMD:LED_0805_2012Metric, F.Cu at (-129.3, -22.8)
- added D112: LED, LED_SMD:LED_0805_2012Metric, F.Cu at (-129.3, -19.8)
- added D113: LED, LED_SMD:LED_0805_2012Metric, F.Cu at (-124.9, -28.9)
- added D114: LED, LED_SMD:LED_0805_2012Metric, F.Cu at (-124.9, -25.9)
- added D115: LED, LED_SMD:LED_0805_2012Metric, F.Cu at (-124.9, -22.8)
- added D116: LED, LED_SMD:LED_0805_2012Metric, F.Cu at (-124.9, -19.8)
- added D82: 1N914, Diode_SMD:D_SOD-323F, F.Cu at (-287.1, -344.9)
- added D83: 1N914, Diode_SMD:D_SOD-323F, F.Cu at (-287.1, -342.0)
- added D84: 1N914, Diode_SMD:D_SOD-323F, F.Cu at (-529.2, 137.6)
- added D85: 1N914, Diode_SMD:D_SOD-323F, F.Cu at (-529.2, 140.6)
- added D86: 1N914, Diode_SMD:D_SOD-323F, F.Cu at (-529.2, 143.5)
- added D87: 1N914, Diode_SMD:D_SOD-323F, F.Cu at (-529.2, 146.5)
- added D88: 1N914, Diode_SMD:D_SOD-323F, F.Cu at (-529.2, 149.4)
- added D89: 1N914, Diode_SMD:D_SOD-323F, F.Cu at (-529.2, 152.4)
- added D90: 1N914, Diode_SMD:D_SOD-323F, F.Cu at (-529.2, 155.3)
- added D91: 1N914, Diode_SMD:D_SOD-323F, F.Cu at (-529.2, 158.3)
- added D92: LED, LED_SMD:LED_0805_2012Metric, F.Cu at (-524.8, 137.7)
- added D93: LED, LED_SMD:LED_0805_2012Metric, F.Cu at (-524.8, 140.7)
- added D94: LED, LED_SMD:LED_0805_2012Metric, F.Cu at (-524.8, 143.8)
- added D95: LED, LED_SMD:LED_0805_2012Metric, F.Cu at (-524.8, 146.8)
- added D96: LED, LED_SMD:LED_0805_2012Metric, F.Cu at (-919.5, 291.5)
- added D97: 1N914, Diode_SMD:D_SOD-323F, F.Cu at (-903.7, 282.9)
- added D98: 1N914, Diode_SMD:D_SOD-323F, F.Cu at (-903.7, 285.9)
- added D99: LED, LED_SMD:LED_0805_2012Metric, F.Cu at (-919.5, 294.5)
- added J13: ADEG2_OUT, SynthProjConnectors:JINJIA CK3.5-98-LF, F.Cu at (-109.9, -150.9)
- added J15: External Clock Input, SynthProjConnectors:JINJIA CK3.5-98-LF, F.Cu at (-558.9, 79.7)
- added J16: Trigger Out, SynthProjConnectors:JINJIA CK3.5-98-LF, F.Cu at (-540.6, 61.5)
- added J17: Gate Out, SynthProjConnectors:JINJIA CK3.5-98-LF, F.Cu at (-540.6, 70.6)
- added J19: External Clock Output, SynthProjConnectors:JINJIA CK3.5-98-LF, F.Cu at (-540.6, 79.7)
- added J22: Sequencer CV3, SynthProjConnectors:JINJIA CK3.5-98-LF, F.Cu at (-91.6, -160.1)
- added J23: Sequencer CV2, SynthProjConnectors:JINJIA CK3.5-98-LF, F.Cu at (-91.6, -150.9)
- added J24: Sequencer CV1, SynthProjConnectors:JINJIA CK3.5-98-LF, F.Cu at (-91.6, -141.8)
- added J25: Master Output, SynthProjConnectors:JINJIA CK3.5-98-LF, F.Cu at (-100.8, -150.9)
- added J26: Sequencer CV1, SynthProjConnectors:JINJIA CK3.5-98-LF, F.Cu at (-137.7, -9.62)
- added J27: Sequencer CV1, SynthProjConnectors:JINJIA CK3.5-98-LF, F.Cu at (-137.7, -0.49)
- added J28: Sequencer CV1, SynthProjConnectors:JINJIA CK3.5-98-LF, F.Cu at (-128.6, -9.62)
- added J29: Sequencer CV1, SynthProjConnectors:JINJIA CK3.5-98-LF, F.Cu at (-128.6, -0.49)
- added J30: Echo_DV, SynthProjConnectors:JINJIA CK3.5-98-LF, F.Cu at (-119.0, -160.1)
- added J31: Echo_Repeat, SynthProjConnectors:JINJIA CK3.5-98-LF, F.Cu at (-119.0, -150.9)
- added J32: Echo_CV_In, SynthProjConnectors:JINJIA CK3.5-98-LF, F.Cu at (-119.0, -141.8)
- added J33: Echo_ExtIn, SynthProjConnectors:JINJIA CK3.5-98-LF, F.Cu at (-109.9, -160.1)
- added J34: ADEG2_OUT, SynthProjConnectors:JINJIA CK3.5-98-LF, F.Cu at (-109.9, -141.8)
- added J35: Sequencer CV1, SynthProjConnectors:JINJIA CK3.5-98-LF, F.Cu at (-155.9, -9.62)
- added J36: Sequencer CV1, SynthProjConnectors:JINJIA CK3.5-98-LF, F.Cu at (-155.9, -0.49)
- added J37: Sequencer CV1, SynthProjConnectors:JINJIA CK3.5-98-LF, F.Cu at (-146.8, -9.62)
- added J37: Conn_02x18_Odd_Even, Connector_PinHeader_2.54mm:PinHeader_2x18_P2.54mm_Vertical, F.Cu at (-155.7, -162.3)
- added J38: Conn_02x18_Odd_Even, Connector_PinHeader_2.54mm:PinHeader_2x18_P2.54mm_Vertical, F.Cu at (-148.5, -162.3)
- added J38: Sequencer CV1, SynthProjConnectors:JINJIA CK3.5-98-LF, F.Cu at (-146.8, -0.49)
- added J40: Conn_01x02, Connector_PinHeader_2.54mm:PinHeader_1x02_P2.54mm_Vertical, F.Cu at (-129.2, -122.7)
- added J41: DIN-504D-M5, SynthProjConnectors:SD-50BV, F.Cu at (-114.5, -31.1)
- added J42: USB_B, Connector_USB:USB_B_Lumberg_2411_02_Horizontal, F.Cu at (-137.8, -40.7)
- added J43: Conn_01x02, Connector_PinHeader_2.54mm:PinHeader_1x02_P2.54mm_Vertical, F.Cu at (-145.6, -26.1)
- added J44: Jack-DC, Connector_BarrelJack:BarrelJack_CUI_PJ-063AH_Horizontal, F.Cu at (-253.3, -104.6)
- added J5: External Start, SynthProjConnectors:JINJIA CK3.5-98-LF, F.Cu at (-558.9, 61.5)
- added L1: L, Inductor_SMD:L_7.3x7.3_H3.5, F.Cu at (-86.6, -72.8)
- added Q1: MMBF4393LT1G, Package_TO_SOT_SMD:SOT-23-3, F.Cu at (-73.4, -121.8)
- added Q19: MMBF5457, Package_TO_SOT_SMD:SOT-23-3, F.Cu at (288.9, -227.0)
- added Q21: 2N3904, Package_TO_SOT_THT:TO-92_Inline, F.Cu at (-292.1, -394.2)
- added Q22: 2N3904, Package_TO_SOT_THT:TO-92_Inline, F.Cu at (-292.1, -388.4)
- added Q23: 2N3906, Package_TO_SOT_THT:TO-92_Inline, F.Cu at (-292.1, -382.7)
- added Q24: 2N3906, Package_TO_SOT_THT:TO-92_Inline, F.Cu at (-292.1, -376.9)
- added Q25: 2N3904, Package_TO_SOT_THT:TO-92_Inline, F.Cu at (-919.8, 275.9)
- added Q26: 2N3906, Package_TO_SOT_THT:TO-92_Inline, F.Cu at (-919.8, 281.7)
- added Q27: 2N3904, Package_TO_SOT_THT:TO-92_Inline, F.Cu at (-919.8, 287.4)
- added Q6: MMBF4393LT1G, Package_TO_SOT_SMD:SOT-23-3, F.Cu at (-73.4, -117.3)
- added R263: 100k, Resistor_SMD:R_0603_1608Metric, F.Cu at (-291.7, -372.9)
- added R264: 100k, Resistor_SMD:R_0603_1608Metric, F.Cu at (-291.7, -369.9)
- added R265: 1k, Resistor_SMD:R_0603_1608Metric, F.Cu at (-291.7, -367.0)
- added R266: 200k, Resistor_SMD:R_0603_1608Metric, F.Cu at (-291.7, -364.0)
- added R268: 1k, Resistor_SMD:R_0603_1608Metric, F.Cu at (-291.7, -361.1)
- added R269: 680k, Resistor_SMD:R_0603_1608Metric, F.Cu at (-291.7, -358.1)
- added R270: 270k, Resistor_SMD:R_0603_1608Metric, F.Cu at (-287.0, -372.9)
- added R273: 1M, Resistor_SMD:R_0603_1608Metric, F.Cu at (-287.0, -369.9)
- added R275: 100k, Resistor_SMD:R_0603_1608Metric, F.Cu at (-287.0, -367.0)
- added R276: 100k, Resistor_SMD:R_0603_1608Metric, F.Cu at (-287.0, -364.0)
- added R279: 3k, Resistor_SMD:R_0603_1608Metric, F.Cu at (-287.0, -361.1)
- added R280: 43k, Resistor_SMD:R_0603_1608Metric, F.Cu at (-287.0, -358.1)
- added R282: 15k, Resistor_SMD:R_0603_1608Metric, F.Cu at (-282.2, -372.9)
- added R283: 100k, Resistor_SMD:R_0603_1608Metric, F.Cu at (-282.2, -369.9)
- added R287: 43k, Resistor_SMD:R_0603_1608Metric, F.Cu at (-282.2, -367.0)
- added R288: 100k, Resistor_SMD:R_0603_1608Metric, F.Cu at (-282.2, -364.0)
- added R289: 15k, Resistor_SMD:R_0603_1608Metric, F.Cu at (-282.2, -361.1)
- added R305: 200k, Resistor_SMD:R_0603_1608Metric, F.Cu at (-546.8, 137.6)
- added R306: 4.7k, Resistor_SMD:R_0603_1608Metric, F.Cu at (-546.8, 140.6)
- added R307: 4.7k, Resistor_SMD:R_0603_1608Metric, F.Cu at (-546.8, 143.5)
- added R308: 20k, Resistor_SMD:R_0603_1608Metric, F.Cu at (-546.8, 146.5)
- added R309: 100k, Resistor_SMD:R_0603_1608Metric, F.Cu at (-546.8, 149.4)
- added R310: 47k, Resistor_SMD:R_0603_1608Metric, F.Cu at (-546.8, 152.4)
- added R311: 47k, Resistor_SMD:R_0603_1608Metric, F.Cu at (-546.8, 155.3)
- added R312: 470k, Resistor_SMD:R_0603_1608Metric, F.Cu at (-546.8, 158.3)
- added R313: 20k, Resistor_SMD:R_0603_1608Metric, F.Cu at (-542.4, 137.6)
- added R314: 1M, Resistor_SMD:R_0603_1608Metric, F.Cu at (-542.4, 140.6)
- added R315: 10k, Resistor_SMD:R_0603_1608Metric, F.Cu at (-542.4, 143.5)
- added R316: 20k, Resistor_SMD:R_0603_1608Metric, F.Cu at (-542.4, 146.5)
- added R317: 10k, Resistor_SMD:R_0603_1608Metric, F.Cu at (-542.4, 149.4)
- added R318: 47k, Resistor_SMD:R_0603_1608Metric, F.Cu at (-542.4, 152.4)
- added R319: 20k, Resistor_SMD:R_0603_1608Metric, F.Cu at (-542.4, 155.3)
- added R320: 10k, Resistor_SMD:R_0603_1608Metric, F.Cu at (-542.4, 158.3)
- added R321: 20k, Resistor_SMD:R_0603_1608Metric, F.Cu at (-538.0, 137.6)
- added R322: 10k, Resistor_SMD:R_0603_1608Metric, F.Cu at (-538.0, 140.6)
- added R323: 20k, Resistor_SMD:R_0603_1608Metric, F.Cu at (-538.0, 143.5)
- added R324: 200k, Resistor_SMD:R_0603_1608Metric, F.Cu at (-538.0, 146.5)
- added R325: 1M, Resistor_SMD:R_0603_1608Metric, F.Cu at (-538.0, 149.4)
- added R326: 4.7k, Resistor_SMD:R_0603_1608Metric, F.Cu at (-538.0, 152.4)
- added R327: 6.2k, Resistor_SMD:R_0603_1608Metric, F.Cu at (-538.0, 155.3)
- added R328: 4.7k, Resistor_SMD:R_0603_1608Metric, F.Cu at (-538.0, 158.3)
- added R329: 4.7k, Resistor_SMD:R_0603_1608Metric, F.Cu at (-533.6, 137.6)
- added R330: 4.7k, Resistor_SMD:R_0603_1608Metric, F.Cu at (-533.6, 140.6)
- added R331: 4.7k, Resistor_SMD:R_0603_1608Metric, F.Cu at (-533.6, 143.5)
- added R332: 4.7k, Resistor_SMD:R_0603_1608Metric, F.Cu at (-533.6, 146.5)
- added R333: 39k, Resistor_SMD:R_0603_1608Metric, F.Cu at (-533.6, 149.4)
- added R334: 22k, Resistor_SMD:R_0603_1608Metric, F.Cu at (-533.6, 152.4)
- added R335: 10k, Resistor_SMD:R_0603_1608Metric, F.Cu at (-533.6, 155.3)
- added R336: 10k, Resistor_SMD:R_0603_1608Metric, F.Cu at (-533.6, 158.3)
- added R337: 1M, Resistor_SMD:R_0603_1608Metric, F.Cu at (-913.1, 274.1)
- added R338: 4.7k, Resistor_SMD:R_0603_1608Metric, F.Cu at (-913.1, 277.0)
- added R339: 100k, Resistor_SMD:R_0603_1608Metric, F.Cu at (-913.1, 280.0)
- added R340: 3k, Resistor_SMD:R_0603_1608Metric, F.Cu at (-908.7, 274.1)
- added R341: 100k, Resistor_SMD:R_0603_1608Metric, F.Cu at (-908.7, 277.0)
- added R342: 47k, Resistor_SMD:R_0603_1608Metric, F.Cu at (-908.7, 280.0)
- added R343: 47k, Resistor_SMD:R_0603_1608Metric, F.Cu at (-904.2, 274.1)
- added R344: 1k, Resistor_SMD:R_0603_1608Metric, F.Cu at (-904.2, 277.0)
- added R345: 4.7k, Resistor_SMD:R_0603_1608Metric, F.Cu at (-904.2, 280.0)
- added R346: 220, Resistor_SMD:R_0603_1608Metric, F.Cu at (-141.3, -138.6)
- added R347: 1k, Resistor_SMD:R_0603_1608Metric, F.Cu at (-133.6, -148.9)
- added R348: 1k, Resistor_SMD:R_0603_1608Metric, F.Cu at (-133.6, -145.0)
- added R349: DNF, Capacitor_SMD:C_0402_1005Metric, F.Cu at (-133.6, -146.9)
- added R350: 4.7k, Resistor_SMD:R_0603_1608Metric, F.Cu at (-141.4, -163.2)
- added R351: 1k, Resistor_SMD:R_0603_1608Metric, F.Cu at (-141.4, -160.2)
- added R352: 100k, Resistor_SMD:R_0603_1608Metric, F.Cu at (-154.5, -32.2)
- added R353: 100k, Resistor_SMD:R_0603_1608Metric, F.Cu at (-154.5, -29.7)
- added R354: 100k, Resistor_SMD:R_0603_1608Metric, F.Cu at (-150.5, -47.2)
- added R355: 100k, Resistor_SMD:R_0603_1608Metric, F.Cu at (-150.5, -44.7)
- added R356: 100k, Resistor_SMD:R_0603_1608Metric, F.Cu at (-150.5, -42.2)
- added R357: 100k, Resistor_SMD:R_0603_1608Metric, F.Cu at (-150.5, -39.7)
- added R358: 100k, Resistor_SMD:R_0603_1608Metric, F.Cu at (-150.5, -37.2)
- added R359: 100k, Resistor_SMD:R_0603_1608Metric, F.Cu at (-150.5, -34.7)
- added R360: 100k, Resistor_SMD:R_0603_1608Metric, F.Cu at (-150.5, -32.2)
- added R361: 27, Resistor_SMD:R_0603_1608Metric, F.Cu at (-133.6, -143.0)
- added R362: 27, Resistor_SMD:R_0603_1608Metric, F.Cu at (-133.6, -141.0)
- added R363: 470, Resistor_SMD:R_0603_1608Metric, F.Cu at (-150.5, -29.7)
- added R364: 470, Resistor_SMD:R_0603_1608Metric, F.Cu at (-146.5, -47.2)
- added R365: 470, Resistor_SMD:R_0603_1608Metric, F.Cu at (-146.5, -44.7)
- added R366: 470, Resistor_SMD:R_0603_1608Metric, F.Cu at (-146.5, -42.2)
- added R367: 470, Resistor_SMD:R_0603_1608Metric, F.Cu at (-146.5, -39.7)
- added R368: 10k, Resistor_SMD:R_0805_2012Metric, F.Cu at (-50.7, -226.7)
- added R368: 470, Resistor_SMD:R_0603_1608Metric, F.Cu at (-146.5, -37.2)
- added R369: 10k, Resistor_SMD:R_0805_2012Metric, F.Cu at (-50.7, -223.8)
- added R369: 470, Resistor_SMD:R_0603_1608Metric, F.Cu at (-146.5, -34.7)
- added R370: 470, Resistor_SMD:R_0603_1608Metric, F.Cu at (-146.5, -32.2)
- added R371: 470, Resistor_SMD:R_0603_1608Metric, F.Cu at (-146.5, -29.7)
- added R372: 470, Resistor_SMD:R_0603_1608Metric, F.Cu at (-142.5, -47.2)
- added R373: 470, Resistor_SMD:R_0603_1608Metric, F.Cu at (-142.5, -44.7)
- added R374: 470, Resistor_SMD:R_0603_1608Metric, F.Cu at (-142.5, -42.2)
- added R375: 470, Resistor_SMD:R_0603_1608Metric, F.Cu at (-142.5, -39.7)
- added R376: 470, Resistor_SMD:R_0603_1608Metric, F.Cu at (-142.5, -37.2)
- added R377: 470, Resistor_SMD:R_0603_1608Metric, F.Cu at (-142.5, -34.7)
- added R378: 470, Resistor_SMD:R_0603_1608Metric, F.Cu at (-142.5, -32.2)
- added R379: 412, Resistor_SMD:R_0603_1608Metric, F.Cu at (-154.5, -34.7)
- added R380: 1.65k, Resistor_SMD:R_0603_1608Metric, F.Cu at (-154.5, -37.2)
- added R381: 10.7k, Resistor_SMD:R_0603_1608Metric, F.Cu at (-141.4, -157.3)
- added R382: 10.7k, Resistor_SMD:R_0603_1608Metric, F.Cu at (-141.4, -154.3)
- added R383: 10.7k, Resistor_SMD:R_0603_1608Metric, F.Cu at (-141.4, -151.4)
- added R384: 1.65k, Resistor_SMD:R_0603_1608Metric, F.Cu at (-137.0, -163.2)
- added R385: 1.65k, Resistor_SMD:R_0603_1608Metric, F.Cu at (-137.0, -160.2)
- added R386: 1.65k, Resistor_SMD:R_0603_1608Metric, F.Cu at (-137.0, -157.3)
- added R387: 10.7k, Resistor_SMD:R_0603_1608Metric, F.Cu at (-137.0, -154.3)
- added R388: 1.65k, Resistor_SMD:R_0603_1608Metric, F.Cu at (-137.0, -151.4)
- added R389: 10k, Resistor_SMD:R_0603_1608Metric, F.Cu at (-158.5, -34.7)
- added R390: 10k, Resistor_SMD:R_0603_1608Metric, F.Cu at (-154.5, -47.2)
- added R391: 10k, Resistor_SMD:R_0603_1608Metric, F.Cu at (-158.5, -47.2)
- added R392: 10k, Resistor_SMD:R_0603_1608Metric, F.Cu at (-141.3, -135.6)
- added R393: 10k, Resistor_SMD:R_0603_1608Metric, F.Cu at (-141.3, -132.7)
- added R394: 10k, Resistor_SMD:R_0603_1608Metric, F.Cu at (-141.3, -129.7)
- added R395: 10k, Resistor_SMD:R_0603_1608Metric, F.Cu at (-141.3, -126.8)
- added R396: 66.5k, Resistor_SMD:R_0603_1608Metric, F.Cu at (-158.5, -37.2)
- added R397: 66.5k, Resistor_SMD:R_0603_1608Metric, F.Cu at (-158.5, -29.7)
- added R398: 66.5k, Resistor_SMD:R_0603_1608Metric, F.Cu at (-158.5, -44.7)
- added R399: 28.7k, Resistor_SMD:R_0603_1608Metric, F.Cu at (-158.5, -39.7)
- added R400: 28.7k, Resistor_SMD:R_0603_1608Metric, F.Cu at (-158.5, -32.2)
- added R401: 28.7k, Resistor_SMD:R_0603_1608Metric, F.Cu at (-158.5, -42.2)
- added R402: 10k, Resistor_SMD:R_0603_1608Metric, F.Cu at (-154.5, -39.7)
- added R403: 66.5k, Resistor_SMD:R_0603_1608Metric, F.Cu at (-154.5, -42.2)
- added R404: 28.7k, Resistor_SMD:R_0603_1608Metric, F.Cu at (-154.5, -44.7)
- added R405: 10k, Resistor_SMD:R_0603_1608Metric, F.Cu at (-50.7, -232.6)
- added R406: 10k, Resistor_SMD:R_0603_1608Metric, F.Cu at (-50.7, -229.7)
- added R407: 105, Resistor_SMD:R_0603_1608Metric, F.Cu at (-79.5, -64.6)
- added R408: 20k, Resistor_SMD:R_0603_1608Metric, F.Cu at (-79.5, -62.1)
- added RV100: 100k, Potentiometer_THT:Potentiometer_Alps_RK09K_Single_Vertical, F.Cu at (-143.4, -58.2)
- added RV101: 100k, Potentiometer_THT:Potentiometer_Alps_RK09K_Single_Vertical, F.Cu at (-127.9, -72.5)
- added RV102: 100k, Potentiometer_THT:Potentiometer_Alps_RK09K_Single_Vertical, F.Cu at (-127.9, -58.2)
- added RV103: 100k, Potentiometer_THT:Potentiometer_Alps_RK09K_Single_Vertical, F.Cu at (-112.5, -72.5)
- added RV104: 100k, Potentiometer_THT:Potentiometer_Alps_RK09K_Single_Vertical, F.Cu at (-112.5, -58.2)
- added RV74: 100k, Potentiometer_THT:Potentiometer_Alps_RK09K_Single_Vertical, F.Cu at (-307.9, -392.8)
- added RV76: 100k, Potentiometer_THT:Potentiometer_Alps_RK09K_Single_Vertical, F.Cu at (-307.9, -378.5)
- added RV77: 100k, Potentiometer_THT:Potentiometer_Alps_RK09K_Single_Vertical, F.Cu at (-307.9, -364.1)
- added RV78: 100k, Potentiometer_THT:Potentiometer_Alps_RK09K_Single_Vertical, F.Cu at (-307.9, -349.8)
- added RV79: 20k, Potentiometer_SMD:Potentiometer_Bourns_TC33X_Vertical, F.Cu at (-523.9, 150.7)
- added RV80: 1M, Potentiometer_THT:Potentiometer_Alps_RK09K_Single_Vertical, F.Cu at (-547.3, 164.4)
- added RV81: 100k, Potentiometer_THT:Potentiometer_Alps_RK09K_Single_Vertical, F.Cu at (-645.3, -69.9)
- added RV82: 100k, Potentiometer_THT:Potentiometer_Alps_RK09K_Single_Vertical, F.Cu at (-645.3, -55.5)
- added RV83: 100k, Potentiometer_THT:Potentiometer_Alps_RK09K_Single_Vertical, F.Cu at (-645.3, -41.2)
- added RV84: 100k, Potentiometer_THT:Potentiometer_Alps_RK09K_Single_Vertical, F.Cu at (-645.3, -26.8)
- added RV85: 100k, Potentiometer_THT:Potentiometer_Alps_RK09K_Single_Vertical, F.Cu at (-629.9, -69.9)
- added RV86: 100k, Potentiometer_THT:Potentiometer_Alps_RK09K_Single_Vertical, F.Cu at (-629.9, -55.5)
- added RV87: 100k, Potentiometer_THT:Potentiometer_Alps_RK09K_Single_Vertical, F.Cu at (-629.9, -41.2)
- added RV88: 100k, Potentiometer_THT:Potentiometer_Alps_RK09K_Single_Vertical, F.Cu at (-629.9, -26.8)
- added RV89: 100k, Potentiometer_THT:Potentiometer_Alps_RK09K_Single_Vertical, F.Cu at (-614.4, -69.9)
- added RV90: 100k, Potentiometer_THT:Potentiometer_Alps_RK09K_Single_Vertical, F.Cu at (-614.4, -55.5)
- added RV91: 100k, Potentiometer_THT:Potentiometer_Alps_RK09K_Single_Vertical, F.Cu at (-614.4, -41.2)
- added RV92: 100k, Potentiometer_THT:Potentiometer_Alps_RK09K_Single_Vertical, F.Cu at (-614.4, -26.8)
- added RV93: 100k, Potentiometer_THT:Potentiometer_Alps_RK09K_Single_Vertical, F.Cu at (-599.0, -69.9)
- added RV94: 100k, Potentiometer_THT:Potentiometer_Alps_RK09K_Single_Vertical, F.Cu at (-599.0, -55.5)
- added RV95: 100k, Potentiometer_THT:Potentiometer_Alps_RK09K_Single_Vertical, F.Cu at (-599.0, -41.2)
- added RV96: 100k, Potentiometer_THT:Potentiometer_Alps_RK09K_Single_Vertical, F.Cu at (-599.0, -26.8)
- added RV97: 100k, Potentiometer_THT:Potentiometer_Alps_RK09K_Single_Vertical, F.Cu at (-158.8, -72.5)
- added RV98: 100k, Potentiometer_THT:Potentiometer_Alps_RK09K_Single_Vertical, F.Cu at (-158.8, -58.2)
- added RV99: 100k, Potentiometer_THT:Potentiometer_Alps_RK09K_Single_Vertical, F.Cu at (-143.4, -72.5)
- added SW1: SW_SPST, SynthProjConnectors:MTS-103-A01-T0, F.Cu at (-262.1, -79.6)
- added SW10: SW_SPDT, SynthProjConnectors:MTS-103-A01-T0, F.Cu at (975.3, 333.0)
- added SW11: SW_SPDT, SynthProjConnectors:MTS-103-A01-T0, F.Cu at (356.5, 594.7)
- added SW12: SMTS-103-A1-T0, SynthProjConnectors:MTS-103-A01-T0, F.Cu at (219.3, 615.0)
- added SW12: SW_SP3T, SynthProjConnectors:ST-0-102-A01-T000-LF, F.Cu at (356.5, 601.0)
- added SW13: SW_Push_DPDT, SynthProjConnectors:MTS-203-A1-T0, F.Cu at (45.9, 731.3)
- added SW14: SW_SPST, SynthProjConnectors:MTS-103-A01-T0, F.Cu at (-392.1, 775.5)
- added SW15: SW_Push, Button_Switch_THT:SW_PUSH_6mm_H13mm, F.Cu at (-383.1, 773.5)
- added SW16: SW_SPST, SynthProjConnectors:MTS-103-A01-T0, F.Cu at (-392.1, 783.4)
- added SW17: SW_SPDT, SynthProjConnectors:MTS-103-A01-T0, F.Cu at (-341.1, 722.9)
- added SW18: SW_SPDT, SynthProjConnectors:MTS-103-A01-T0, F.Cu at (-341.1, 729.2)
- added SW19: SW_Push, Button_Switch_THT:SW_PUSH_6mm_H13mm, F.Cu at (-383.1, 782.1)
- added SW2: SW_SPDT, SynthProjConnectors:MTS-103-A01-T0, F.Cu at (-66.1, -120.8)
- added SW20: SW_DPST, SynthProjConnectors:MTS-203-A1-T0, F.Cu at (16.3, 731.3)
- added SW21: SW_DPST, SynthProjConnectors:MTS-203-A1-T0, F.Cu at (30.1, 731.3)
- added SW22: SW_SPST, SynthProjConnectors:MTS-103-A01-T0, F.Cu at (-392.1, 791.3)
- added SW23: SW_SPST, SynthProjConnectors:MTS-103-A01-T0, F.Cu at (-392.1, 799.2)
- added SW24: SW_Push, Button_Switch_THT:SW_PUSH_6mm_H13mm, F.Cu at (-261.4, -142.3)
- added SW25: SW_Push, Button_Switch_THT:SW_PUSH_6mm_H13mm, F.Cu at (-261.4, -133.7)
- added SW26: SW_Push, Button_Switch_THT:SW_PUSH_6mm_H13mm, F.Cu at (-261.4, -125.2)
- added SW27: SW_Push, Button_Switch_THT:SW_PUSH_6mm_H13mm, F.Cu at (-261.4, -116.6)
- added SW28: SRBV141404, SynthProjConnectors:SRBV141404, F.Cu at (-339.0, 352.9)
- added SW29: SW_Push_DPDT, SynthProjConnectors:MTS-203-A1-T0, F.Cu at (32.1, 747.6)
- added SW3: SW_SPDT, SynthProjConnectors:MTS-103-A01-T0, F.Cu at (107.0, 198.2)
- added SW30: SR2612F-0112-21R0B-D8-N, SynthProjConnectors:SR2612F-0112, F.Cu at (-335.6, 328.8)
- added SW31: SW_SPST, SynthProjConnectors:MTS-103-A01-T0, F.Cu at (-384.0, 319.2)
- added SW32: SW_SPST, SynthProjConnectors:MTS-103-A01-T0, F.Cu at (-384.0, 327.1)
- added SW33: SW_SPST, SynthProjConnectors:MTS-103-A01-T0, F.Cu at (-384.0, 335.0)
- added SW34: SW_SPST, SynthProjConnectors:MTS-103-A01-T0, F.Cu at (-384.0, 342.9)
- added SW35: SW_SPST, SynthProjConnectors:MTS-103-A01-T0, F.Cu at (-384.0, 350.9)
- added SW36: SW_SPST, SynthProjConnectors:MTS-103-A01-T0, F.Cu at (-384.0, 358.8)
- added SW37: SW_SPST, SynthProjConnectors:MTS-103-A01-T0, F.Cu at (-370.1, 319.2)
- added SW38: SW_SPST, SynthProjConnectors:MTS-103-A01-T0, F.Cu at (-370.1, 327.1)
- added SW39: SW_SPST, SynthProjConnectors:MTS-103-A01-T0, F.Cu at (-370.1, 335.0)
- added SW4: SW_SPDT, SynthProjConnectors:MTS-103-A01-T0, F.Cu at (107.0, 180.0)
- added SW40: SW_SPST, SynthProjConnectors:MTS-103-A01-T0, F.Cu at (-370.1, 342.9)
- added SW41: SW_SPST, SynthProjConnectors:MTS-103-A01-T0, F.Cu at (-370.1, 350.9)
- added SW42: SW_SPST, SynthProjConnectors:MTS-103-A01-T0, F.Cu at (-370.1, 358.8)
- added SW43: SW_SPST, SynthProjConnectors:MTS-103-A01-T0, F.Cu at (-356.2, 319.2)
- added SW44: SW_SPST, SynthProjConnectors:MTS-103-A01-T0, F.Cu at (-356.2, 327.1)
- added SW45: SW_SPST, SynthProjConnectors:MTS-103-A01-T0, F.Cu at (-356.2, 335.0)
- added SW46: SW_SPST, SynthProjConnectors:MTS-103-A01-T0, F.Cu at (-356.2, 342.9)
- added SW47: SW_DPDT_x2, SynthProjConnectors:MTS-203-A1-T0, F.Cu at (16.3, 747.6)
- added SW48: SW_Push_DPDT, SynthProjConnectors:MTS-203-A1-T0, F.Cu at (47.9, 747.6)
- added SW49: SW_SPDT, SynthProjConnectors:MTS-103-A01-T0, F.Cu at (-910.6, 284.6)
- added SW5: SYNC, SynthProjConnectors:MTS-103-A01-T0, F.Cu at (107.0, 233.2)
- added SW50: SW_SPDT, SynthProjConnectors:MTS-103-A01-T0, F.Cu at (-910.6, 290.9)
- added SW51: SW_Push, Button_Switch_THT:SW_PUSH_6mm_H13mm, F.Cu at (-231.3, -195.7)
- added SW52: SW_Push, Button_Switch_THT:SW_PUSH_6mm_H13mm, F.Cu at (-231.3, -187.1)
- added SW53: SW_Push, Button_Switch_THT:SW_PUSH_6mm_H13mm, F.Cu at (-231.3, -178.6)
- added SW54: SW_Push, Button_Switch_THT:SW_PUSH_6mm_H13mm, F.Cu at (-231.3, -170.0)
- added SW55: SW_Push, Button_Switch_THT:SW_PUSH_6mm_H13mm, F.Cu at (-231.3, -161.5)
- added SW56: SW_Push, Button_Switch_THT:SW_PUSH_6mm_H13mm, F.Cu at (-220.8, -195.7)
- added SW57: SW_Push, Button_Switch_THT:SW_PUSH_6mm_H13mm, F.Cu at (-220.8, -187.1)
- added SW58: SW_Push, Button_Switch_THT:SW_PUSH_6mm_H13mm, F.Cu at (-220.8, -178.6)
- added SW6: SW_SPDT, SynthProjConnectors:MTS-103-A01-T0, F.Cu at (313.2, -472.9)
- added SW7: SW_SPDT, SynthProjConnectors:MTS-103-A01-T0, F.Cu at (313.2, -466.6)
- added SW8: SW_SPDT, SynthProjConnectors:MTS-103-A01-T0, F.Cu at (724.7, -226.0)
- added SW9: SW_SPDT, SynthProjConnectors:MTS-103-A01-T0, F.Cu at (975.3, 326.7)
- added TP1: TestPoint, TestPoint:TestPoint_Pad_D1.0mm, F.Cu at (-210.7, -177.6)
- added TP10: TestPoint, TestPoint:TestPoint_Plated_Hole_D2.0mm, F.Cu at (-266.8, -90.3)
- added TP11: TestPoint, TestPoint:TestPoint_Plated_Hole_D2.0mm, F.Cu at (-262.1, -104.3)
- added TP12: TestPoint, TestPoint:TestPoint_Plated_Hole_D2.0mm, F.Cu at (-262.1, -99.6)
- added TP13: TestPoint, TestPoint:TestPoint_Plated_Hole_D2.0mm, F.Cu at (-262.1, -95.0)
- added TP2: TestPoint, TestPoint:TestPoint_Pad_D1.0mm, F.Cu at (-210.7, -180.7)
- added TP3: TestPoint, TestPoint:TestPoint_Pad_D1.0mm, F.Cu at (-207.7, -177.6)
- added TP4: TestPoint, TestPoint:TestPoint_Pad_D1.0mm, F.Cu at (-204.6, -177.6)
- added TP5: TestPoint, TestPoint:TestPoint_Pad_D1.0mm, F.Cu at (-207.7, -180.7)
- added TP6: TestPoint, TestPoint:TestPoint_Pad_D1.0mm, F.Cu at (-204.6, -180.7)
- added TP7: TestPoint, TestPoint:TestPoint_Plated_Hole_D2.0mm, F.Cu at (-266.8, -104.3)
- added TP8: TestPoint, TestPoint:TestPoint_Plated_Hole_D2.0mm, F.Cu at (-266.8, -99.6)
- added TP9: TestPoint, TestPoint:TestPoint_Plated_Hole_D2.0mm, F.Cu at (-266.8, -95.0)
- added U23: CD4094, Package_SO:SOP-16_3.9x9.9mm_P1.27mm, F.Cu at (-789.4, 679.0)
- added U29: TL074, Package_SO:SO-14_3.9x8.65mm_P1.27mm, F.Cu at (-285.0, -351.5)
- added U32: 40106, Package_SO:SOIC-14_3.9x8.7mm_P1.27mm, F.Cu at (-552.9, 178.7)
- added U33: 4013, Package_SO:SOIC-14_3.9x8.7mm_P1.27mm, F.Cu at (-938.3, 396.0)
- added U34: 40106, Package_SO:SOIC-14_3.9x8.7mm_P1.27mm, F.Cu at (-929.9, 396.0)
- added U35: 40193, Package_SO:SOIC-16W_5.3x10.2mm_P1.27mm, F.Cu at (-552.0, 189.8)
- added U36: TL074, Package_SO:SO-14_3.9x8.65mm_P1.27mm, F.Cu at (-921.4, 396.0)
- added U37: 4042, Package_SO:SOP-16_3.9x9.9mm_P1.27mm, F.Cu at (-532.5, 189.6)
- added U38: 40193, Package_SO:SOIC-16W_5.3x10.2mm_P1.27mm, F.Cu at (-541.9, 189.8)
- added U39: CD74HC4067SM, Package_SO:SSOP-24_5.3x8.2mm_P0.65mm, F.Cu at (-641.7, -12.1)
- added U40: 6N138, Package_SO:SOP-8_6.605x9.655mm_P2.54mm, F.Cu at (-154.2, -22.8)
- added U41: NCP1117-3.3_SOT223, Package_TO_SOT_SMD:SOT-223-3_TabPin2, F.Cu at (-134.0, -135.9)
- added U42: W25Q128JVS, Package_SO:SOIC-8_5.23x5.23mm_P1.27mm, F.Cu at (-133.7, -128.4)
- added U43: RP2040, RP2040_minimal:RP2040-QFN-56, F.Cu at (-207.6, -186.8)
- added U44: MCP23017_SS, Package_SO:SSOP-28_5.3x10.2mm_P0.65mm, F.Cu at (-103.1, -32.2)
- added U45: REF3012, Package_TO_SOT_SMD:SOT-23, F.Cu at (-129.7, -147.7)
- added U46: MCP4728, Package_SO:MSOP-10_3x3mm_P0.5mm, F.Cu at (-135.2, -122.6)
- added U47: TL074, Package_SO:SO-14_3.9x8.65mm_P1.27mm, F.Cu at (-109.0, -43.4)
- added U48: CD74HC4067SM, Package_SO:SSOP-24_5.3x8.2mm_P0.65mm, F.Cu at (-103.1, -21.2)
- added U49: TL074, Package_SO:SO-14_3.9x8.65mm_P1.27mm, F.Cu at (-117.4, -43.4)
- added U51: BUF634AIDDAR, Package_SO:SOIC-8_3.9x4.9mm_P1.27mm, F.Cu at (365.3, 158.0)
- added U52: BUF634AIDDAR, Package_SO:SOIC-8_3.9x4.9mm_P1.27mm, F.Cu at (365.3, 164.5)
- added U53: TPS560200, Package_TO_SOT_SMD:SOT-23-5, F.Cu at (-79.3, -75.0)
- added U54: LM1117MP-3.3, Package_TO_SOT_SMD:SOT-223-3_TabPin2, F.Cu at (-86.4, -64.2)
- added Y1: ABLS-12.000MHZ-B4-T, RP2040_minimal:Crystal_SMD_HC49-US, F.Cu at (-204.4, -194.6)
- C1, C11, C12, C13, C14, C2, C23, C24, C25, C26, C3, C35, C36, C37, C38, C39, C4, C40, C41, C42, C47, C48, C49, C5, C50, C51, C52, C55, C58, C60: footprint Capacitor_SMD:C_0805_2012Metric_Pad1.18x1.45mm_HandSolder -> Capacitor_SMD:C_0805_2012Metric
- C10, C15, C16, C18, C19, C20, C22, C27, C28, C29, C30, C31, C32, C34, C43, C44, C45, C46, C53, C54, C56, C57, C59, C6, C7, C8, C9: footprint Capacitor_SMD:C_0805_2012Metric_Pad1.18x1.45mm_HandSolder -> Capacitor_SMD:C_0603_1608Metric
- C100: renamed from C103; footprint Capacitor_SMD:C_0805_2012Metric -> Capacitor_SMD:C_0603_1608Metric
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- renumbered C105 to C102, C106 to C103, C107 to C104, C108 to C105, C111 to C108, C114 to C111, C115 to C112, C116 to C113, C117 to C114, C123 to C120, C124 to C121, C125 to C122, C126 to C123, D35 to D34, D36 to D35, D37 to D36, D38 to D37, D39 to D38, D40 to D39, D41 to D40, D42 to D41, D43 to D42, D44 to D43, D45 to D44, D46 to D45, D47 to D46, D48 to D47, D49 to D48, D50 to D49, D51 to D50, D52 to D51, D53 to D52, D54 to D53, D55 to D54, D56 to D55, D57 to D56, D58 to D57, D59 to D58, D60 to D59, D61 to D60, D62 to D61, D63 to D62, D64 to D63, D65 to D64, D66 to D65, D67 to D66, D68 to D67, D69 to D68, D70 to D69, D71 to D70, D72 to D71, D73 to D72, D74 to D73, D75 to D74, D76 to D75, D77 to D76, D78 to D77, D79 to D78, D80 to D79, D81 to D80, D82 to D81, J14 to J1, J15 to J10, J18 to J11, J2 to J12, J3 to J13, J4 to J14, J11 to J2, J7 to J20, J8 to J21, J6 to J25, J12 to J3, J16 to J39, J13 to J4, J17 to J6, J9 to J7, J1 to J8, J10 to J9, Q26 to Q20, RV47 to RV40, RV48 to RV41, RV49 to RV42, RV50 to RV43, RV51 to RV44, RV52 to RV45, RV53 to RV46, RV54 to RV47, RV55 to RV48, RV56 to RV49, RV57 to RV50, RV58 to RV51, RV59 to RV52, RV60 to RV53, RV61 to RV54, RV62 to RV55, RV63 to RV56, RV64 to RV57, RV65 to RV58, RV66 to RV59, RV67 to RV60, RV68 to RV61, RV69 to RV62, RV70 to RV63, RV71 to RV64, RV72 to RV65, RV73 to RV66, RV74 to RV67, RV75 to RV68, RV76 to RV69, RV77 to RV70, RV78 to RV71, RV79 to RV72, RV80 to RV73, RV40 to RV75, U19 to U17, U20 to U18, U21 to U19, U22 to U20, U23 to U21, U24 to U22, U25 to U24, U26 to U25, U27 to U26, U28 to U27, U18 to U28, U29 to U30, U17 to U31
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Connections:
- net /SequencerClocking/RIN renamed Net-(D45-A)
- net /SequencerClocking/XCLK renamed /XCLK
- net Net-(D56-A) renamed /SequencerInput/Q12
- net Net-(D57-A) renamed /SequencerInput/Q4
- net Net-(D58-A) renamed /SequencerInput/Q11
- net Net-(D59-A) renamed /SequencerInput/Q5
- net Net-(D60-A) renamed /SequencerInput/Q10
- net Net-(D61-A) renamed /SequencerInput/Q6
- net Net-(D62-A) renamed /SequencerInput/Q9
- net Net-(D63-A) renamed /SequencerInput/Q7
- net Net-(D64-A) renamed /SequencerInput/Q8
- net Net-(SW25-B) renamed /PT2399Echo/Echo_ExtIn
- net Net-(U19A-Q) renamed /SequencerClocking/X2
- net XSTP renamed /SequencerClocking/XSTP
- C155 pad 1: unconnected-(C93-Pad1) -> /PT2399Echo/Echo_A
- C158 pad 2: Net-(C147-Pad2) -> Net-(C158-Pad2)
- C160 pad 1: Net-(C149-Pad1) -> Net-(C160-Pad1)
- C160 pad 2: Net-(U18B--) -> Net-(U29B--)
- C161 pad 2: unconnected-(C148-Pad2) -> /PT2399Echo/Echo_B
- C162 pad 1: Net-(C149-Pad1) -> Net-(C160-Pad1)
- D48 pad 2: Net-(D49-A) -> /SequencerClocking/FWD
- D49 pad 2: Net-(D50-A) (its old number) -> /SequencerInput/Q15
- D51 pad 2: Net-(D52-A) (its old number) -> /SequencerInput/Q14
- D53 pad 2: Net-(D54-A) (its old number) -> /SequencerInput/Q13
- D64 pad 2: Net-(D49-A) -> /SequencerClocking/FWD
- D77 pad 2: Net-(D54-A) (its old number) -> /SequencerInput/Q13
- D78 pad 2: Net-(D52-A) (its old number) -> /SequencerInput/Q14
- D79 pad 2: Net-(D50-A) (its old number) -> /SequencerInput/Q15
- D80 pad 1: Net-(D81-K) -> /SequencerInput/SBV1
- D80 pad 2: /SequencerInput/DN -> /SequencerClocking/DN
- D81 pad 1: /SequencerInput/UP -> /SequencerClocking/UP
- D81 pad 2: Net-(D81-K) -> /SequencerInput/SBV1
- R218 pad 2: Net-(D81-K) -> /SequencerInput/SBV2
- R293 pad 1: Net-(U18B-+) -> Net-(U29B-+)
- R295 pad 1: Net-(C147-Pad2) -> Net-(R295-Pad1)
- R295 pad 2: Net-(U18B-+) -> Net-(U29B-+)
- R296 pad 1: Net-(U18B--) -> Net-(U29B--)
- R297 pad 1: Net-(R194-Pad2) -> /PT2399Echo/Echo_A
- R298 pad 1: Net-(U18B-+) -> Net-(U29B-+)
- R299 pad 1: Net-(C149-Pad1) -> Net-(C160-Pad1)
- R299 pad 2: Net-(U18B--) -> Net-(U29B--)
- R301 pad 2: Net-(R194-Pad2) -> /PT2399Echo/Echo_A
- R302 pad 1: Net-(R198-Pad1) -> /PT2399Echo/Echo_B
- R304 pad 2: Net-(R198-Pad1) -> /PT2399Echo/Echo_B
- U13 pad 2: unconnected-(U13A---Pad2) -> GNDREF
- U19 pad 10: Net-(U22-UP) -> /SequencerClocking/UP
- U19 pad 4: Net-(U22-DOWN) -> /SequencerClocking/DN
- U20 pad 2: /SequencerClocking/QB -> /SequencerAnalogGenerator/QB
- U20 pad 3: /SequencerClocking/QA -> /SequencerAnalogGenerator/QA
- U20 pad 4: Net-(U22-DOWN) -> /SequencerClocking/DN
- U20 pad 5: Net-(U22-UP) -> /SequencerClocking/UP
- U20 pad 6: /SequencerClocking/QC -> /SequencerAnalogGenerator/QC
- U20 pad 7: /SequencerClocking/QD -> /SequencerAnalogGenerator/QD
- U22 pad 14: unconnected-(U24G-VDD-Pad14) -> +12V
- U22 pad 2: unconnected-(U24-Pad2) -> Net-(U23-DATA)
- U22 pad 5: Net-(D81-K) -> /SequencerInput/SBV2
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Other:
- copper layers 2 -> 4
- board text added: "80/60HP Eurorack"
- board text added: "Coarse Frequency Adjust"
- board text added: "Fine Frequency Adjust"
- board text added: "Pulse Width"

Commit message: Doing some layout
Parts:
- removed the J13 at (109.4, -140.2)
- removed the J13 at (-109.9, -150.9)
- removed the J25 at (109.4, -112.8)
- removed the J25 at (-100.8, -150.9)
- removed the J37 at (-146.8, -9.62)
- removed the J37 at (-155.7, -162.3)
- removed the J38 at (-148.5, -162.3)
- removed the J38 at (-146.8, -0.49)
- removed the SW12 at (356.5, 601.0)
- added J13: Gate, SynthProjConnectors:PJ-358, F.Cu at (301.3, 307.1)
- added J25: Master Output, SynthProjConnectors:PJ-358, F.Cu at (90.3, -266.8)
- added J37: Sequencer CV1, SynthProjConnectors:PJ-358, F.Cu at (112.5, -266.8)
- added J38: Sequencer CV1, SynthProjConnectors:PJ-358, F.Cu at (112.5, -259.4)
- added RV27: 100k, Potentiometer_THT:Potentiometer_Alps_RK09K_Single_Vertical, F.Cu at (300.4, 201.0)
- J1, J10, J11, J12, J14, J15, J16, J17, J18, J19, J2, J20, J21, J22, J23, J24, J26, J27, J28, J29, J3, J30, J31, J32, J33, J34, J35, J36, J39, J4, J5, J6, J7, J8, J9: footprint SynthProjConnectors:JINJIA CK3.5-98-LF -> SynthProjConnectors:PJ-358
- RV16, RV25, RV39, RV6: footprint Potentiometer_THT:Potentiometer_Alps_RK09K_Single_Vertical -> Potentiometer_SMD:Potentiometer_Bourns_TC33X_Vertical
- moved D82 1409.2 mm to (1101.2, -103.2)
- moved D83 1409.2 mm to (1101.2, -100.3)
- moved C135 1409.2 mm to (1142.3, -144.7)
- moved C136 1409.2 mm to (1142.3, -141.7)
- moved C137 1409.2 mm to (1142.3, -138.7)
- moved C138 1409.2 mm to (1142.3, -135.7)
- moved C139 1409.2 mm to (1142.3, -132.7)
- moved C140 1409.2 mm to (1142.3, -129.7)
- moved C141 1409.2 mm to (1096.6, -113.4)
- moved C142 1409.2 mm to (1096.6, -110.4)
- moved C143 1409.2 mm to (1096.6, -107.4)
- moved C144 1409.2 mm to (1132.7, -126.7)
- moved C145 1409.2 mm to (1137.5, -147.8)
- moved C146 1409.2 mm to (1137.5, -144.7)
- moved C147 1409.2 mm to (1096.6, -104.4)
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Other:
- board outline added: 426.4 x 110 mm
- board text added: "10HP"
- board text added: "1HP"
- board text added: "21mm between pots"
- board text added: "2HP"
- board text added: "4HP"
- board text added: "84/60HP Eurorack"
- board text added: "AD Envelope"
- board text added: "Common Small Knobs"
- board text added: "LFO"
- board text added: "Mixer"
- board text added: "S&H"
- board text added: "VCA"
- board text added: "VCF"
- board text added: "VCO1"
- board text added: "VCO2"
- board text removed: "80/60HP Eurorack"
