File: SynthProj.kicad_pcb (KiCad board)
At the start: 4 copper layers, 426.4 x 110 mm, 1058 parts, among them J1 PWM IN, J10 Mixer Ext In, J11 S&H_Out, J12 LFOA_Out, J13 Gate, J14 1V/Oct CV, J15 External Clock Input, J16 Trigger Out, J17 Gate Out, J18 Ext In, J19 External Clock Output, J2 Exp CV In, J20 ADEG1_OUT, J21 ADEG2_OUT, J22 Sequencer CV3, J23 Sequencer CV2, J24 Sequencer CV1, J25 Master Output, J26 Sequencer CV1, J27 Sequencer CV1, J28 Sequencer CV1, J29 Sequencer CV1, J3 Lin CV In, J30 Echo_DV, J31 Echo_Repeat, J32 Echo_CV_In, J33 Echo_ExtIn, J34 ADEG2_OUT, J35 Sequencer CV1, J36 Sequencer CV1, J37 Sequencer CV1, J38 Sequencer CV1, J39 Noise Out, J4 Sync, J40 Conn_01x02, J41 DIN-504D-M5, J42 USB_B, J43 Conn_01x02, J44 Jack-DC, J5 External Start, J6 S&H_In, J7 Lin CV In, J8 Exp CV In, J9 PWM IN, Q1 MMBF4393LT1G, Q10 MMBT3904-7-F, Q11 MMBT3904-7-F, Q12 MMBF4391LT1G, Q13 MMBT3904-7-F, Q14 MMBT3904-7-F, Q15 MMBT3906LT1G, Q16 MMBF5457, Q17 MMBF5457, Q18 MMBT3906LT1G, Q19 MMBF5457, Q2 MMBT3904-7-F, Q20 MMBT3904-7-F, Q21 2N3904, Q22 2N3904, Q23 2N3906, Q24 2N3906, Q25 2N3904, Q26 2N3906, Q27 2N3904, Q3 MMBT3906LT1G, Q4 MMBT3904-7-F, Q5 MMBT3906LT1G, Q6 MMBF4393LT1G, Q7 MMBT3904-7-F, Q8 MMBT3904-7-F, Q9 MMBF4391LT1G, SW1 SW_SPST, SW10 SW_SPDT, SW11 SW_SPDT, SW12 SMTS-103-A1-T0, SW13 SW_Push_DPDT, SW14 SW_SPST, SW15 SW_Push, SW16 SW_SPST, SW17 SW_SPDT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

Commit message: doing some routing - split sequencer into another project
Parts:
- removed C100, C101, C109, C110, C117, C93, C94, C95: 10nF, Capacitor_SMD:C_0603_1608Metric
- removed C102, C103, C105, C111, C112, C114, C120, C121, C123, C129, C130, C168, C169, C182, C183, C188, C189: 4.7uF, Capacitor_SMD:C_0805_2012Metric
- removed C104, C113, C122, C170, C171, C184, C185, C190, C191: 470nF, Capacitor_SMD:C_0805_2012Metric
- removed C106, C107, C115, C116, C124, C125, C173, C174, C186, C187, C192, C193: 47nF, Capacitor_SMD:C_0603_1608Metric
- removed C108, C179: 1uF, Capacitor_SMD:C_0805_2012Metric
- removed C118, C126, C127, C128, C163, C164: 1nF, Capacitor_SMD:C_0603_1608Metric
- removed C119, C165, C167, C175, C176: 100pF, Capacitor_SMD:C_0603_1608Metric
- removed C131, C133, C181: 470pF, Capacitor_SMD:C_0603_1608Metric
- removed C132, C134, C194: 100nF, Capacitor_SMD:C_0603_1608Metric
- removed C166, C172: 680pF, Capacitor_SMD:C_0603_1608Metric
- removed C177: 10pF, Capacitor_SMD:C_0603_1608Metric
- removed C178: 22pF, Capacitor_SMD:C_0603_1608Metric
- removed C180, C96, C97, C98, C99: 20nF, Capacitor_SMD:C_0603_1608Metric
- removed D34, D35, D36, D37, D38, D39, D40, D41, D42, D43, D44, D46, D47, D64, D65, D66, D67, D68, D69, D70, D71, D72, D73, D74, D75, D76, D77, D78, D79, D80, D81, D84, D85, D86, D87, D88, D89, D90, D91, D97, D98: 1N914, Diode_SMD:D_SOD-323F
- removed D45, D48, D49, D50, D51, D52, D53, D54, D55, D56, D57, D58, D59, D60, D61, D62, D63, D92, D93, D94, D95, D96, D99: LED, LED_SMD:LED_0805_2012Metric
- removed J15: External Clock Input, SynthProjConnectors:PJ-358
- removed J16: Trigger Out, SynthProjConnectors:PJ-358
- removed J17: Gate Out, SynthProjConnectors:PJ-358
- removed J19: External Clock Output, SynthProjConnectors:PJ-358
- removed J22: Sequencer CV3, SynthProjConnectors:PJ-358
- removed J23: Sequencer CV2, SynthProjConnectors:PJ-358
- removed J24: Sequencer CV1, SynthProjConnectors:PJ-358
- removed J5: External Start, SynthProjConnectors:PJ-358
- removed Q20: MMBT3904-7-F, Package_TO_SOT_SMD:SOT-23-3
- removed Q25, Q27: 2N3904, Package_TO_SOT_THT:TO-92_Inline
- removed Q26: 2N3906, Package_TO_SOT_THT:TO-92_Inline
- removed R176, R178, R179, R188, R189, R201, R215, R222, R225, R228, R315, R317, R320, R322, R335, R336: 10k, Resistor_SMD:R_0603_1608Metric
- removed R177, R190, R191, R192, R193, R207, R211, R218, R219, R223, R227, R232, R233, R235, R238, R240, R241, R243, R246, R248, R249, R251, R254, R256, R257, R259, R262, R309, R339, R341: 100k, Resistor_SMD:R_0603_1608Metric
- removed R180, R184, R212, R214, R314, R325, R337: 1M, Resistor_SMD:R_0603_1608Metric
- removed R181, R182, R183, R204: 680k, Resistor_SMD:R_0603_1608Metric
- removed R185, R186, R187, R206: 220k, Resistor_SMD:R_0603_1608Metric
- removed R194, R195, R200, R203, R224, R226, R310, R311, R318, R342, R343: 47k, Resistor_SMD:R_0603_1608Metric
- removed R196, R205, R220, R221, R344: 1k, Resistor_SMD:R_0603_1608Metric
- removed R197: 3.9k, Resistor_SMD:R_0603_1608Metric
- removed R198, R327: 6.2k, Resistor_SMD:R_0603_1608Metric
- removed R199, R308, R313, R316, R319, R321, R323: 20k, Resistor_SMD:R_0603_1608Metric
- removed R202, R216, R340: 3k, Resistor_SMD:R_0603_1608Metric
- removed R208, R231, R234, R236, R237, R239, R242, R244, R245, R247, R250, R252, R253, R255, R258, R260, R261: 2M, Resistor_SMD:R_0603_1608Metric
- removed R209, R213, R217, R306, R307, R326, R328, R329, R330, R331, R332, R338, R345: 4.7k, Resistor_SMD:R_0603_1608Metric
- removed R210: 4.7M, Resistor_SMD:R_0603_1608Metric
- removed R229, R305, R324: 200k, Resistor_SMD:R_0603_1608Metric
- removed R230: 22, Resistor_SMD:R_0603_1608Metric
- removed R312: 470k, Resistor_SMD:R_0603_1608Metric
- removed R333: 39k, Resistor_SMD:R_0603_1608Metric
- removed R334: 22k, Resistor_SMD:R_0603_1608Metric
- removed the R368 at (-50.7, -226.7)
- removed the R369 at (-50.7, -223.8)
- removed the RV27 at (300.4, 201.0)
- removed RV40, RV45, RV80: 1M, Potentiometer_THT:Potentiometer_Alps_RK09K_Single_Vertical
- removed RV41 (x2), RV42, RV43, RV44, RV46, RV47, RV48, RV49, RV50, RV51, RV52, RV53, RV54, RV55, RV56, RV57, RV58, RV59, RV60, RV61, RV62, RV63, RV64, RV65, RV66, RV67, RV68, RV69, RV70, RV71, RV72, RV73, RV81, RV82, RV83, RV84, RV85, RV86, RV87, RV88, RV89, RV90, RV91, RV92, RV93, RV94, RV95, RV96: 100k, Potentiometer_THT:Potentiometer_Alps_RK09K_Single_Vertical
- removed RV79: 20k, Potentiometer_SMD:Potentiometer_Bourns_TC33X_Vertical
- removed SW24, SW25, SW26, SW27: SW_Push, Button_Switch_THT:SW_PUSH_6mm_H13mm
- removed SW28: SRBV141404, SynthProjConnectors:SRBV141404
- removed SW29, SW48: SW_Push_DPDT, SynthProjConnectors:MTS-203-A1-T0
- removed SW30: SR2612F-0112-21R0B-D8-N, SynthProjConnectors:SR2612F-0112
- removed SW31, SW32, SW33, SW34, SW35, SW36, SW37, SW38, SW39, SW40, SW41, SW42, SW43, SW44, SW45, SW46: SW_SPST, SynthProjConnectors:MTS-103-A01-T0
- removed SW49, SW50: SW_SPDT, SynthProjConnectors:MTS-103-A01-T0
- removed SW5: SYNC, SynthProjConnectors:MTS-103-A01-T0
- removed TP10, TP11: TestPoint, TestPoint:TestPoint_Plated_Hole_D2.0mm
- removed U17, U33: 4013, Package_SO:SOIC-14_3.9x8.7mm_P1.27mm
- removed U18, U19, U22, U32, U34: 40106, Package_SO:SOIC-14_3.9x8.7mm_P1.27mm
- removed U20, U35, U38: 40193, Package_SO:SOIC-16W_5.3x10.2mm_P1.27mm
- removed U21, U25: TL082, Package_SO:SOIC-8_3.9x4.9mm_P1.27mm
- removed U23: CD4094, Package_SO:SOP-16_3.9x9.9mm_P1.27mm
- removed U24: 4514, Package_SO:SOIC-24W_7.5x15.4mm_P1.27mm
- removed U26: TL084, Package_SO:SO-14_3.9x8.65mm_P1.27mm
- removed U27: CD74HC4067M, Package_SO:SOIC-24W_7.5x15.4mm_P1.27mm
- removed U36: TL074, Package_SO:SO-14_3.9x8.65mm_P1.27mm
- removed U37: 4042, Package_SO:SOP-16_3.9x9.9mm_P1.27mm
- removed U39: CD74HC4067SM, Package_SO:SSOP-24_5.3x8.2mm_P0.65mm
- removed U51, U52: BUF634AIDDAR, Package_SO:SOIC-8_3.9x4.9mm_P1.27mm
- J1, J10, J11, J12, J13, J14, J18, J2, J20, J21, J25, J3, J30, J31, J32, J33, J34, J39, J4, J6, J7, J8, J9: footprint SynthProjConnectors:PJ-358 -> SynthProjConnectors:PJ-301
- J26: value Sequencer CV1 -> RP2040_A_in; footprint SynthProjConnectors:PJ-358 -> SynthProjConnectors:PJ-301
- J27: value Sequencer CV1 -> RP2040_B_in; footprint SynthProjConnectors:PJ-358 -> SynthProjConnectors:PJ-301
- J28: value Sequencer CV1 -> RP2040_C_in; footprint SynthProjConnectors:PJ-358 -> SynthProjConnectors:PJ-301
- J29: value Sequencer CV1 -> RP2040_D_in; footprint SynthProjConnectors:PJ-358 -> SynthProjConnectors:PJ-301
- J35: value Sequencer CV1 -> RP2040_A_out; footprint SynthProjConnectors:PJ-358 -> SynthProjConnectors:PJ-301
- J36: value Sequencer CV1 -> RP2040_B_out; footprint SynthProjConnectors:PJ-358 -> SynthProjConnectors:PJ-301
- J37: value Sequencer CV1 -> RP2040_C_out; footprint SynthProjConnectors:PJ-358 -> SynthProjConnectors:PJ-301
- J38: value Sequencer CV1 -> RP2040_D_out; footprint SynthProjConnectors:PJ-358 -> SynthProjConnectors:PJ-301
- moved C15 1091.5 mm to (50.3, 376.6)
- moved C16 1091.5 mm to (50.3, 379.7)
- moved C11 1091.5 mm to (45.5, 376.6)
- moved C12 1091.5 mm to (45.5, 379.7)
- moved C13 1091.5 mm to (45.5, 382.7)
- moved C14 1091.5 mm to (45.5, 385.7)
- moved C22 1051.1 mm to (113.9, 271.1)
- moved U5 1049.6 mm to (115.2, 266.6)
- moved R58 1029.5 mm to (111.6, 268.8), turned to 90 degrees
- moved R63 1028.2 mm to (111.5, 273.6), turned to 90 degrees
- moved R60 1027.0 mm to (113.9, 272.8)
- moved R62 1026.4 mm to (113.9, 274.4), turned to 180 degrees
- moved R48 1022.2 mm to (113.7, 262.0)
- moved R52 1020.4 mm to (113.7, 260.5), turned to 180 degrees
- moved R49 1019.3 mm to (116.0, 260.6), turned to 90 degrees
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Connections:
- C17 pad 2: X24 -> /VCO1/X29
- R41 pad 1: X24 -> /VCO1/X29
Routing:
- net Net-(Q7-C): track 0.00 -> 9.83 mm
- net Net-(C18-Pad1): track 0.00 -> 6.80 mm
- net Net-(R36-Pad2): track 0.00 -> 6.57 mm
- net Net-(Q7-E): track 0.00 -> 3.63 mm
- net Net-(U13B--): track 0.00 -> 2.66 mm
- net X13: track 0.00 -> 2.23 mm
- net X21: track 0.00 -> 2.13 mm
- net X12: track 0.00 -> 2.07 mm
- net Net-(R38-Pad2): track 0.00 -> 1.80 mm
- net Net-(U5B--): track 0.00 -> 1.53 mm
- net Net-(D2-A): track 0.00 -> 1.42 mm

Commit message: routing work...
Parts:
- removed J29: RP2040_D_in, SynthProjConnectors:PJ-301
- removed RV75: 100k, Potentiometer_THT:Potentiometer_Alps_RK09K_Single_Vertical
- J34: value ADEG2_OUT -> Echo_Out
- moved J37 418.7 mm to (129.9, 239.6)
- moved C73 408.5 mm to (244.1, 30.2), turned to 180 degrees
- moved J27 404.6 mm to (100.7, 239.5)
- moved C74 402.9 mm to (230.7, 30.4), turned to 0 degrees
- moved C83 385.0 mm to (52.2, 395.4)
- moved C84 385.0 mm to (49.1, 395.4)
- moved C82 385.0 mm to (60.6, 396.7)
- moved C81 361.5 mm to (43.7, 395.2)
- moved Q6 327.0 mm to (349.1, 304.1), turned to 180 degrees
- moved Q1 313.0 mm to (330.8, 304.1)
- moved SW2 279.1 mm to (338.5, 209.5), turned to -90 degrees
- moved J32 251.5 mm to (378.0, 156.2)
- moved J31 231.3 mm to (378.0, 174.2)
- moved J21 228.5 mm to (283.0, 240.9)
- moved J35 224.0 mm to (140.2, 169.2)
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Routing:
- net Net-(R42-Pad1): track 0.00 -> 3.66 mm
- net Net-(D2-K): track 0.00 -> 2.88 mm
- net Net-(Q7-C): track 9.83 -> 11.4 mm
Other:
- board size 426.4 x 110 mm -> 304.8 x 110 mm
- board text added: "ECHO"

Commit message: more routing...
Parts:
- moved D32 279.5 mm to (331.4, 102.5), turned to -90 degrees
- moved D33 272.7 mm to (335.7, 109.8)
- moved D31 266.7 mm to (328.9, 109.8)
- moved R166 266.4 mm to (330.8, 113.2), turned to -90 degrees
- moved U16 266.3 mm to (325.6, 115.7)
- moved R169 264.1 mm to (332.3, 108.0), turned to 180 degrees
- moved R162 257.1 mm to (333.9, 114.5)
- moved R167 256.5 mm to (327.0, 107.7), turned to 180 degrees
- moved R175 256.2 mm to (331.7, 117.0)
- moved R171 253.9 mm to (314.6, 115.5), turned to -90 degrees
- moved C90 252.7 mm to (332.3, 109.8)
- moved R168 251.3 mm to (319.8, 112.6), turned to -90 degrees
- moved C92 250.0 mm to (331.6, 118.6)
- moved C91 247.4 mm to (317.0, 109.2), turned to 180 degrees
- moved C89 246.2 mm to (325.2, 109.8)
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Routing:
- net X20: track 0.00 -> 15.3 mm
- net Net-(U4B-+): track 0.00 -> 13.3 mm
- net Net-(R83-Pad2): track 0.00 -> 10.8 mm
- net Net-(Q16-G): track 0.00 -> 8.88 mm
- net Net-(R49-Pad2): track 0.00 -> 7.78 mm
- net Net-(C22-Pad2): track 0.00 -> 7.64 mm
- net Net-(Q8-C): track 0.00 -> 6.40 mm
- net Net-(U8A-+): track 0.00 -> 6.25 mm
- net Net-(Q9-S): track 0.00 -> 5.95 mm
- net Net-(U5B--): track 1.53 -> 7.09 mm
- net Net-(U5B-+): track 0.00 -> 4.91 mm
- net Net-(D3-K): track 0.00 -> 4.57 mm
- net Net-(U8B--): track 0.00 -> 4.40 mm
- net Net-(D3-A): track 0.00 -> 4.07 mm
- net Net-(D13-K): track 0.00 -> 3.87 mm
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
Commit message: routing work...
Parts:
- removed J42: USB_B, Connector_USB:USB_B_Lumberg_2411_02_Horizontal
- added U50: BUF634AIDDAR, Package_SO:SOIC-8-1EP_3.9x4.9mm_P1.27mm_EP2.514x3.2mm_ThermalVias, F.Cu at (45.0, 118.1)
- J34: value Echo_Out -> ECHO_OUT
- J37: value RP2040_C_out -> locked
- J38: value RP2040_D_out -> locked
- moved D28 272.7 mm to (259.8, 311.5)
- moved R160 272.7 mm to (259.8, 307.6)
- moved C142 229.4 mm to (215.2, 339.8)
- moved C141 229.4 mm to (215.2, 336.8)
- moved C143 229.4 mm to (215.2, 342.8)
- moved D19 224.4 mm to (268.1, 316.1)
- moved D11 205.3 mm to (266.6, 232.0)
- moved C5 189.9 mm to (173.8, 353.9)
- moved C2 189.9 mm to (173.8, 344.8)
- moved C3 189.9 mm to (173.8, 347.8)
- moved C4 189.9 mm to (173.8, 350.9)
- moved C6 189.9 mm to (178.6, 341.8)
- moved C7 189.9 mm to (178.6, 344.8)
- moved R16 189.9 mm to (173.3, 338.8)
- moved R158 181.8 mm to (281.9, 203.0), turned to 0 degrees
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Connections:
- SW47 pad 2: Net-(SW47A-B) -> /PT2399Echo/Echo_ExtIn
- U48 pad 9: Net-(U48-I0) -> unconnected-(U48-I0-Pad9)
- U49 pad 12: /RP2040Microcontroller/VREF1.0 -> unconnected-(U49D-+-Pad12)
- U49 pad 13: Net-(U49D--) -> unconnected-(U49D---Pad13)
- U49 pad 14: Net-(U48-I0) -> unconnected-(U49-Pad14)
Routing:
- net /Mixer/X16: track 1.55 -> 41.8 mm
- net Net-(U12A--): track 0.00 -> 17.4 mm
- net X55: track 0.00 -> 13.5 mm
- net Net-(Q6-S): track 0.00 -> 10.5 mm
- net Net-(D12-A): track 0.00 -> 9.50 mm
- net Net-(Q1-G): track 0.00 -> 7.85 mm
- net X56: track 0.00 -> 7.77 mm
- net Net-(Q15-B): track 0.00 -> 7.09 mm
- net Net-(C57-Pad2): track 0.00 -> 6.90 mm
- net Net-(C34-Pad2): track 3.25 -> 9.37 mm
- net Net-(U12A-+): track 0.00 -> 6.09 mm
- net Net-(D10-K): track 0.00 -> 5.91 mm
- net Net-(U4B--): track 3.16 -> 8.94 mm
- net Net-(D20-A): track 0.00 -> 5.33 mm
- net +12V: track 0.00 -> 5.19 mm
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Other:
- board text added: "Adafruit 2{dblquote} IPS Screen"

Commit message: routing... placing... going cross eyed...
Parts:
- removed C149: 22pF, Capacitor_SMD:C_0603_1608Metric
- removed R267: 20k, Resistor_SMD:R_0603_1608Metric
- removed R271: 1k, Resistor_SMD:R_0603_1608Metric
- removed R272, R274, R352, R353, R354, R355, R356, R358: 100k, Resistor_SMD:R_0603_1608Metric
- removed R402: 10k, Resistor_SMD:R_0603_1608Metric
- removed R403: 66.5k, Resistor_SMD:R_0603_1608Metric
- removed R404: 28.7k, Resistor_SMD:R_0603_1608Metric
- removed RV102, RV103, RV97, RV98, RV99: 100k, Potentiometer_THT:Potentiometer_Alps_RK09K_Single_Vertical
- removed SW47: SW_DPDT_x2, SynthProjConnectors:MTS-203-A1-T0
- removed SW51, SW52, SW53, SW54, SW55, SW57: SW_Push, Button_Switch_THT:SW_PUSH_6mm_H13mm
- added J42: USB_B, Connector_USB:USB_B_TE_5787834_Vertical, F.Cu at (121.2, 149.3)
- added J5: Conn_01x18, Connector_FFC-FPC:Hirose_FH12-18S-0.5SH_1x18-1MP_P0.50mm_Horizontal, F.Cu at (-8.47, 100.9)
- added SW5: SW_DPDT_x2, SynthProjConnectors:MTS-203-A1-T0, F.Cu at (365.9, 231.5)
- Q21, Q22: value 2N3904 -> MMBT3904-7-F; footprint Package_TO_SOT_THT:TO-92_Inline -> Package_TO_SOT_SMD:SOT-23-3
- Q23, Q24: value 2N3906 -> MMBT3906LT1G; footprint Package_TO_SOT_THT:TO-92_Inline -> Package_TO_SOT_SMD:SOT-23-3
- moved C135 315.3 mm to (190.1, 358.3)
- moved C136 315.3 mm to (190.1, 361.3)
- moved C137 315.3 mm to (190.1, 364.3)
- moved C138 315.3 mm to (190.1, 367.3)
- moved C139 284.8 mm to (220.4, 362.7)
- moved C140 284.8 mm to (220.4, 365.7)
- moved R279 174.4 mm to (371.6, 180.1), turned to -90 degrees
- moved C151 171.0 mm to (373.1, 180.0), turned to -90 degrees
- moved R263 169.5 mm to (369.1, 185.6), turned to 180 degrees
- moved R264 166.8 mm to (372.2, 184.0), turned to 180 degrees
- moved R266 164.9 mm to (371.5, 186.3), turned to -90 degrees
- moved R268 162.5 mm to (373.1, 186.3), turned to 90 degrees
- moved R302 162.2 mm to (374.6, 218.1), turned to 180 degrees
- moved U28 157.0 mm to (379.7, 183.4), turned to 180 degrees
- moved R303 156.8 mm to (383.8, 198.2), turned to 180 degrees
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- renumbered RV101 to RV40, RV104 to RV41, RV100 to RV42
Connections:
- C148 pad 2: Net-(SW47A-C) -> /PT2399Echo/Echo_ExtIn
- C156 pad 1: Net-(SW47B-B) -> Net-(U28A--)
- C158 pad 1: Net-(SW47B-B) -> Net-(U28A--)
- J33 pad T: /PT2399Echo/Echo_ExtIn -> Net-(SW5A-A)
- J34 pad T: /PT2399Echo/EchoOut -> Net-(SW5B-A)
- SW11 pad 3: GNDREF -> unconnected-(SW11-C-Pad3)
- U28 pad 1: Net-(SW47B-C) -> Net-(U28A--)
- U48 pad 2: Net-(U48-I7) -> unconnected-(U48-I7-Pad2)
- U48 pad 23: Net-(U48-I8) -> unconnected-(U48-I8-Pad23)
- U48 pad 3: Net-(U48-I6) -> unconnected-(U48-I6-Pad3)
- U48 pad 4: Net-(U48-I5) -> unconnected-(U48-I5-Pad4)
- U48 pad 5: Net-(U48-I4) -> unconnected-(U48-I4-Pad5)
Routing:
- net Net-(C30-Pad1): track 0.00 -> 15.0 mm
- net Net-(U6A--): track 0.00 -> 12.2 mm
- net X91: track 0.00 -> 10.6 mm
- net Net-(Q10-C): track 0.00 -> 9.99 mm
- net Net-(U31-LPF2-OUT): track 0.00 -> 9.67 mm
- net /VCO1/X18: track 0.00 -> 9.24 mm
- net Net-(U28D--): track 0.00 -> 9.05 mm
- net Net-(U31-LPF1-IN): track 0.00 -> 8.71 mm
- net Net-(U31-LPF2-IN): track 0.00 -> 6.83 mm
- net /Mixer/MXO: track 0.00 -> 6.26 mm
- net Net-(R76-Pad1): track 0.00 -> 5.98 mm
- net Net-(Q10-E): track 0.00 -> 5.95 mm
- net Net-(U31-LPF1-OUT): track 0.00 -> 5.53 mm
- net Net-(Q19-D): track 0.00 -> 5.53 mm
- net Net-(U16A--): track 0.00 -> 5.21 mm
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Other:
- board text added: "60HP Eurorack"
- board text removed: "84/60HP Eurorack"
