File: SynthProj.kicad_pcb (KiCad board)
At the start: 4 copper layers, 304.8 x 110 mm, 649 parts, among them J1 PWM IN, J10 Mixer Ext In, J11 S&H_Out, J12 LFOA_Out, J13 Gate, J14 1V/Oct CV, J18 Ext In, J2 Exp CV In, J20 ADEG1_OUT, J21 ADEG2_OUT, J25 Master Output, J26 RP2040_A_in, J27 RP2040_B_in, J28 RP2040_C_in, J3 Lin CV In, J30 Echo_DV, J31 Echo_Repeat, J32 Echo_CV_In, J33 Echo_ExtIn, J34 ECHO_OUT, J35 RP2040_A_out, J36 RP2040_B_out, J37 locked, J38 locked, J39 Noise Out, J4 Sync, J40 Conn_01x02, J41 DIN-504D-M5, J42 USB_B, J43 Conn_01x02, J44 Jack-DC, J5 Conn_01x18, J6 S&H_In, J7 Lin CV In, J8 Exp CV In, J9 PWM IN, Q1 MMBF4393LT1G, Q10 MMBT3904-7-F, Q11 MMBT3904-7-F, Q12 MMBF4391LT1G, Q13 MMBT3904-7-F, Q14 MMBT3904-7-F, Q15 MMBT3906LT1G, Q16 MMBF5457, Q17 MMBF5457, Q18 MMBT3906LT1G, Q19 MMBF5457, Q2 MMBT3904-7-F, Q21 MMBT3904-7-F, Q22 MMBT3904-7-F, Q23 MMBT3906LT1G, Q24 MMBT3906LT1G, Q3 MMBT3906LT1G, Q4 MMBT3904-7-F, Q5 MMBT3906LT1G, Q6 MMBF4393LT1G, Q7 MMBT3904-7-F, Q8 MMBT3904-7-F, Q9 MMBF4391LT1G, SW1 SW_SPST, SW10 SW_SPDT, SW11 SW_SPDT, SW12 SMTS-103-A1-T0, SW13 SW_Push_DPDT, SW14 SW_SPST, SW15 SW_Push, SW16 SW_SPST, SW17 SW_SPDT, SW18 SW_SPDT, SW19 SW_Push, SW2 SW_SPDT, SW20 SW_DPST, SW21 SW_DPST, SW22 SW_SPST, SW23 SW_SPST, SW3 SW_SPDT, SW4 SW_SPDT, SW5 SW_DPDT_x2, SW56 SW_Push, SW58 SW_Push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

Commit message: work
Parts:
- moved D32 153.1 mm to (301.8, 354.6)
- moved R270 59.3 mm to (389.8, 186.1)
- moved R269 59.3 mm to (392.9, 186.1)
- moved C147 58.9 mm to (390.1, 184.3)
- moved J34 55.9 mm to (337.8, 241.0), turned to 90 degrees
- moved R11 32.5 mm to (359.2, 183.5)
- moved SW5 30.2 mm to (338.0, 220.1), turned to 90 degrees
- moved C89 25.5 mm to (299.3, 219.2)
- moved C90 25.5 mm to (306.6, 220.6)
- moved C92 25.5 mm to (305.8, 227.1)
- moved D33 25.5 mm to (310.0, 218.7)
- moved R169 25.5 mm to (306.7, 218.8)
- moved RV39 25.5 mm to (293.7, 232.0)
- moved C91 25.5 mm to (291.1, 218.6)
- moved D31 25.5 mm to (302.9, 216.4)
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Routing:
- net Net-(Q19-G): track 4.34 -> 0.00 mm
- net Net-(U31-REF): track 3.20 -> 0.00 mm
- net -12V: track 4.61 -> 3.20 mm

Commit message: lots of routes, added vco3, lfo2.
Parts:
- removed RV41: 100k, Potentiometer_THT:Potentiometer_Alps_RK09K_Single_Vertical
- added C100: 1nF, Capacitor_SMD:C_0603_1608Metric, F.Cu at (184.5, 104.3)
- added C101: 100pF, Capacitor_SMD:C_0603_1608Metric, F.Cu at (187.0, 104.3)
- added C102: 5n, Capacitor_SMD:C_0603_1608Metric, F.Cu at (189.5, 104.3)
- added C103: 4.7pF, Capacitor_SMD:C_0603_1608Metric, F.Cu at (192.0, 104.3)
- added C104: 1nF, Capacitor_SMD:C_0603_1608Metric, F.Cu at (194.5, 104.3)
- added C105: 4.7pF, Capacitor_SMD:C_0603_1608Metric, F.Cu at (197.0, 104.3)
- added C106: 22nF, Capacitor_SMD:C_0603_1608Metric, F.Cu at (363.2, 266.2)
- added C107: 10pF, Capacitor_SMD:C_0603_1608Metric, F.Cu at (360.7, 266.2)
- added C108: 4.7uF, Capacitor_SMD:C_0805_2012Metric, F.Cu at (320.7, 318.9)
- added C109: 4.7uF, Capacitor_SMD:C_0805_2012Metric, F.Cu at (317.7, 318.9)
- added C110: 470nF, Capacitor_SMD:C_0805_2012Metric, F.Cu at (314.7, 318.9)
- added C111: 470nF, Capacitor_SMD:C_0805_2012Metric, F.Cu at (311.7, 318.9)
- added C112: 47nF, Capacitor_SMD:C_0603_1608Metric, F.Cu at (358.2, 266.2)
- added C113: 47nF, Capacitor_SMD:C_0603_1608Metric, F.Cu at (355.6, 266.2)
- added C114: 100nF, Capacitor_SMD:C_0603_1608Metric, F.Cu at (164.1, 42.2)
- added C93: 100nF, Capacitor_SMD:C_0603_1608Metric, F.Cu at (94.5, 257.9)
- added C94: 4.7uF, Capacitor_SMD:C_0805_2012Metric, F.Cu at (179.7, 84.0)
- added C95: 4.7uF, Capacitor_SMD:C_0805_2012Metric, F.Cu at (182.7, 84.0)
- added C96: 470nF, Capacitor_SMD:C_0805_2012Metric, F.Cu at (185.7, 84.0)
- added C97: 470nF, Capacitor_SMD:C_0805_2012Metric, F.Cu at (188.7, 84.0)
- added C98: 47nF, Capacitor_SMD:C_0603_1608Metric, F.Cu at (179.5, 104.3)
- added C99: 47nF, Capacitor_SMD:C_0603_1608Metric, F.Cu at (182.0, 104.3)
- added D34: 1N914, Diode_SMD:D_SOD-323F, F.Cu at (214.9, 90.5)
- added D35: 1N914, Diode_SMD:D_SOD-323F, F.Cu at (217.9, 90.5)
- added D36: 1N914, Diode_SMD:D_SOD-323F, F.Cu at (335.3, 266.3)
- added D37: 1N914, Diode_SMD:D_SOD-323F, F.Cu at (332.3, 266.3)
- added D38: LED, LED_SMD:LED_0805_2012Metric, F.Cu at (208.4, 70.7)
- added J17: PWM IN, SynthProjConnectors:PJ-301-BM, F.Cu at (219.2, 227.8)
- added J19: Exp CV In, SynthProjConnectors:PJ-301-BM, F.Cu at (219.2, 240.0)
- added J22: Lin CV In, SynthProjConnectors:PJ-301-BM, F.Cu at (205.5, 240.0)
- added J23: Sync, SynthProjConnectors:PJ-301-BM, F.Cu at (205.5, 227.8)
- added J24: Sync, SynthProjConnectors:PJ-301-BM, F.Cu at (178.0, 227.8)
- added J323.25: LFO2_Out, SynthProjConnectors:PJ-301-BM, F.Cu at (303.0, 240.3)
- added Q20: MMBT3904-7-F, Package_TO_SOT_SMD:SOT-23-3, F.Cu at (203.0, 95.3)
- added Q25: MMBT3904-7-F, Package_TO_SOT_SMD:SOT-23-3, F.Cu at (207.5, 95.3)
- added Q26: MMBF4391LT1G, Package_TO_SOT_SMD:SOT-23-3, F.Cu at (211.9, 95.3)
- added Q27: MMBT3904-7-F, Package_TO_SOT_SMD:SOT-23-3, F.Cu at (209.1, 75.5)
- added R176: 470k, Resistor_SMD:R_0603_1608Metric, F.Cu at (97.0, 257.9)
- added R177: 4.7M, Resistor_SMD:R_0603_1608Metric, F.Cu at (199.5, 104.3)
- added R178: 100k, Resistor_SMD:R_0603_1608Metric, F.Cu at (179.5, 100.3)
- added R179: 39k, Resistor_SMD:R_0603_1608Metric, F.Cu at (182.0, 100.3)
- added R180: 100k, Resistor_SMD:R_0603_1608Metric, F.Cu at (184.5, 100.3)
- added R181: 100k, Resistor_SMD:R_0603_1608Metric, F.Cu at (187.0, 100.3)
- added R182: 100k, Resistor_SMD:R_0603_1608Metric, F.Cu at (189.5, 100.3)
- added R183: 2k, Resistor_SMD:R_0603_1608Metric, F.Cu at (192.0, 100.3)
- added R184: 36k, Resistor_SMD:R_0603_1608Metric, F.Cu at (194.5, 100.3)
- added R185: 475, Resistor_SMD:R_0603_1608Metric, F.Cu at (197.0, 100.3)
- added R186: 100k, Resistor_SMD:R_0603_1608Metric, F.Cu at (199.5, 100.3)
- added R187: 1M, Resistor_SMD:R_0603_1608Metric, F.Cu at (179.5, 96.3)
- added R188: 100k, Resistor_SMD:R_0603_1608Metric, F.Cu at (182.0, 96.3)
- added R189: 4.7k, Resistor_SMD:R_0603_1608Metric, F.Cu at (184.5, 96.3)
- added R190: 1k, Resistor_SMD:R_0603_1608Metric, F.Cu at (187.0, 96.3)
- added R191: 10k, Resistor_SMD:R_0603_1608Metric, F.Cu at (189.5, 96.3)
- added R192: 1.2M, Resistor_SMD:R_0603_1608Metric, F.Cu at (192.0, 96.3)
- added R193: 10k, Resistor_SMD:R_0603_1608Metric, F.Cu at (194.5, 96.3)
- added R194: 10k, Resistor_SMD:R_0603_1608Metric, F.Cu at (197.0, 96.3)
- added R195: 9.1k, Resistor_SMD:R_0603_1608Metric, F.Cu at (199.5, 96.3)
- added R196: 47k, Resistor_SMD:R_0603_1608Metric, F.Cu at (179.5, 92.3)
- added R197: 10k, Resistor_SMD:R_0603_1608Metric, F.Cu at (182.0, 92.3)
- added R198: 2k, Resistor_SMD:R_0603_1608Metric, F.Cu at (184.5, 92.3)
- added R199: 110k, Resistor_SMD:R_0603_1608Metric, F.Cu at (187.0, 92.3)
- added R200: 1M, Resistor_SMD:R_0603_1608Metric, F.Cu at (189.5, 92.3)
- added R201: 20k, Resistor_SMD:R_0603_1608Metric, F.Cu at (192.0, 92.3)
- added R202: 100k, Resistor_SMD:R_0603_1608Metric, F.Cu at (194.5, 92.3)
- added R203: 3k, Resistor_SMD:R_0603_1608Metric, F.Cu at (197.0, 92.3)
- added R204: 18k, Resistor_SMD:R_0603_1608Metric, F.Cu at (199.5, 92.3)
- added R205: 22k, Resistor_SMD:R_0603_1608Metric, F.Cu at (179.5, 88.3)
- added R206: 20k, Resistor_SMD:R_0603_1608Metric, F.Cu at (182.0, 88.3)
- added R207: 1M, Resistor_SMD:R_0603_1608Metric, F.Cu at (184.5, 88.3)
- added R208: 47k, Resistor_SMD:R_0603_1608Metric, F.Cu at (187.0, 88.3)
- added R209: 4.7k, Resistor_SMD:R_0603_1608Metric, F.Cu at (189.5, 88.3)
- added R210: 3.3k, Resistor_SMD:R_0603_1608Metric, F.Cu at (192.0, 88.3)
- added R211: 1k, Resistor_SMD:R_0603_1608Metric, F.Cu at (353.1, 266.2)
- added R212: 100k, Resistor_SMD:R_0603_1608Metric, F.Cu at (350.6, 266.2)
- added R213: 3M, Resistor_SMD:R_0603_1608Metric, F.Cu at (363.2, 270.2)
- added R214: 220, Resistor_SMD:R_0603_1608Metric, F.Cu at (360.7, 270.2)
- added R215: 3.9k, Resistor_SMD:R_0603_1608Metric, F.Cu at (358.2, 270.2)
- added R216: 100k, Resistor_SMD:R_0603_1608Metric, F.Cu at (355.6, 270.2)
- added R217: 2.2k, Resistor_SMD:R_0603_1608Metric, F.Cu at (353.1, 270.2)
- added R218: 130k, Resistor_SMD:R_0603_1608Metric, F.Cu at (350.6, 270.2)
- added R219: 9.1k, Resistor_SMD:R_0603_1608Metric, F.Cu at (363.2, 274.2)
- added R220: 10k, Resistor_SMD:R_0603_1608Metric, F.Cu at (360.7, 274.2)
- added R221: 270k, Resistor_SMD:R_0603_1608Metric, F.Cu at (358.2, 274.2)
- added R222: 470k, Resistor_SMD:R_0603_1608Metric, F.Cu at (164.1, 44.7)
- added RV3: 100k, Potentiometer_THT:Potentiometer_Alps_RK09K_Single_Vertical, F.Cu at (118.0, 229.0)
- added RV43: 100k, Potentiometer_THT:Potentiometer_Alps_RK09K_Single_Vertical, F.Cu at (204.0, 181.5)
- added RV44: 100k, Potentiometer_THT:Potentiometer_Alps_RK09K_Single_Vertical, F.Cu at (204.0, 162.5)
- added RV45: 100, Potentiometer_SMD:Potentiometer_Bourns_TC33X_Vertical, F.Cu at (192.6, 83.1)
- added RV46: 100k, Potentiometer_SMD:Potentiometer_Bourns_TC33X_Vertical, F.Cu at (197.4, 83.1)
- added RV47: 100k, Potentiometer_THT:Potentiometer_Alps_RK09K_Single_Vertical, F.Cu at (204.0, 219.5)
- added RV48: 10k, Potentiometer_THT:Potentiometer_Alps_RK09K_Single_Vertical, F.Cu at (300.5, 200.5)
- added RV49: 100k, Potentiometer_THT:Potentiometer_Alps_RK09K_Single_Vertical, F.Cu at (300.5, 219.5)
- added RV50: 100k, Potentiometer_THT:Potentiometer_Alps_RK09K_Single_Vertical, F.Cu at (237.5, 181.5)
- added SW24: SW_SPDT, SynthProjConnectors:SMTS-102, F.Cu at (206.5, 194.8)
- added SW25: SW_SPDT, SynthProjConnectors:SMTS-102, F.Cu at (206.5, 202.2)
- added SW26: SW_SPDT, SynthProjConnectors:SMTS-102, F.Cu at (313.1, 187.5)
- added SW27: SMTS-103-A1-T0, SynthProjConnectors:SMTS-102, F.Cu at (313.1, 215.5)
- added SW28: SW_Push_DPDT, SynthProjConnectors:SMTS-202, F.Cu at (313.0, 203.5)
- added SW29: SW_SPDT, SynthProjConnectors:SMTS-102, F.Cu at (206.5, 187.5)
- added U17: TL072, Package_SO:SO-8_3.9x4.9mm_P1.27mm, F.Cu at (204.0, 102.1)
- added U18: TL072, Package_SO:SO-8_3.9x4.9mm_P1.27mm, F.Cu at (210.5, 102.1)
- added U19: TL072, Package_SO:SO-8_3.9x4.9mm_P1.27mm, F.Cu at (216.9, 102.1)
- added U20: TL072, Package_SO:SO-8_3.9x4.9mm_P1.27mm, F.Cu at (313.1, 195.8)
- J1, J10, J11, J13, J14, J18, J2, J20, J21, J25, J26, J27, J28, J3, J30, J31, J32, J33, J34, J35, J36, J37, J38, J39, J4, J6, J7, J8, J9: footprint SynthProjConnectors:PJ-301 -> SynthProjConnectors:PJ-301-BM
- J12: value LFOA_Out -> LFO1_Out; footprint SynthProjConnectors:PJ-301 -> SynthProjConnectors:PJ-301-BM
- SW1, SW10, SW11, SW12, SW14, SW16, SW17, SW18, SW2, SW22, SW23, SW3, SW4, SW6, SW7, SW8, SW9: footprint SynthProjConnectors:MTS-103-A01-T0 -> SynthProjConnectors:SMTS-102
- SW13, SW20, SW21, SW5: footprint SynthProjConnectors:MTS-203-A1-T0 -> SynthProjConnectors:SMTS-202
- moved J5 152.9 mm to (115.4, 190.6)
- moved C158 131.1 mm to (395.6, 165.5), turned to 90 degrees
- moved R292 122.4 mm to (352.4, 242.3), turned to 180 degrees
- moved R169 115.2 mm to (296.7, 333.6)
- moved R301 102.2 mm to (386.2, 204.4), turned to -90 degrees
- moved C141 95.1 mm to (303.1, 300.5)
- moved C6 95.1 mm to (266.5, 305.5)
- moved C142 95.1 mm to (303.1, 303.5)
- moved C143 95.1 mm to (303.1, 306.6)
- moved C80 95.1 mm to (209.1, 303.6)
- moved C12 95.1 mm to (218.4, 299.5)
- moved C13 95.1 mm to (218.4, 302.5)
- moved C14 95.1 mm to (218.4, 305.5)
- moved C16 95.1 mm to (223.2, 299.5)
- moved C24 95.1 mm to (226.8, 305.9)
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Connections:
- C29 pad 2: /VCO1/X29 -> /VCO2/X37
- J12 pad T: LFOA -> LFO1A
- J4 pad T: /VCO1/X29 -> /VCO3/X37
- R75 pad 1: /VCO1/X29 -> /VCO2/X37
- RV27 pad 2: LFOA -> LFO1A
- RV40 pad 2: Net-(U48-I5) -> Net-(U48-I1)
- RV42 pad 2: Net-(U48-I4) -> Net-(U48-I3)
Routing:
- net /Mixer/X16: track 41.8 -> 1.55 mm
- net Net-(U13B--): track 0.00 -> 25.4 mm
- net Net-(Q2-C): track 0.00 -> 20.7 mm
- net Net-(C62-Pad2): track 0.00 -> 20.2 mm
- net Net-(Q12-S): track 0.00 -> 17.3 mm
- net Net-(U6A--): track 12.2 -> 28.4 mm
- net Net-(R131-Pad1): track 0.00 -> 15.1 mm
- net Net-(C61-Pad2): track 0.00 -> 14.9 mm
- net Net-(U13A-+): track 0.00 -> 14.5 mm
- net Net-(U12A--): track 17.4 -> 3.20 mm
- net Net-(U12B--): track 0.00 -> 13.6 mm
- net Net-(R150-Pad1): track 0.00 -> 12.6 mm
- net Net-(Q2-E): track 0.00 -> 10.8 mm
- net Net-(Q6-S): track 15.0 -> 4.52 mm
- net Net-(U31-LPF2-OUT): track 9.67 -> 0.00 mm
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Other:
- board text added: "LFO 1"
- board text added: "LFO 2"
- board text added: "VCO3"
- board text removed: "LFO"

Commit message: more and more routing
Parts:
- removed D10: 1N914, Diode_SMD:D_SOD-323F
- added RV51: 100k, Potentiometer_THT:Potentiometer_Alps_RK09K_Single_Vertical, F.Cu at (346.0, 162.5)
- moved C93 268.1 mm to (360.6, 225.6), turned to -90 degrees
- moved R176 263.3 mm to (358.2, 224.8), turned to 0 degrees
- moved D38 209.5 mm to (304.2, 257.0)
- moved Q27 209.5 mm to (304.9, 261.8)
- moved R16 171.7 mm to (366.7, 167.1)
- moved C112 164.4 mm to (210.5, 338.5)
- moved C113 152.8 mm to (219.1, 334.7)
- moved R147 140.7 mm to (270.8, 262.3)
- moved R298 99.2 mm to (358.6, 179.1)
- moved C161 98.1 mm to (356.9, 179.0), turned to -90 degrees
- moved R221 96.8 mm to (320.9, 184.8), turned to 180 degrees
- moved R213 90.0 mm to (303.8, 202.5), turned to 0 degrees
- moved C107 89.2 mm to (320.9, 186.3), turned to 0 degrees
- moved R220 88.2 mm to (316.1, 198.1), turned to 0 degrees
- moved R218 88.1 mm to (316.7, 188.9), turned to 90 degrees
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- renumbered J323.25 to J16, RV3 to RV41
Connections:
- C148 pad 2: /PT2399Echo/Echo_ExtIn -> Net-(C148-Pad2)
- C223 pad 1: GNDD -> GNDREF
- C224 pad 1: GNDD -> GNDREF
- C225 pad 1: GNDD -> GNDREF
- C226 pad 1: GNDD -> GNDREF
- C227 pad 1: GNDD -> GNDREF
- C228 pad 1: GNDD -> GNDREF
- C229 pad 1: GNDD -> GNDREF
- C93 pad 2: /Mixer/Mixer_EchoIn -> /EchoOut
- J16 pad T: /LFO1/LFOA -> LFO2A
- R407 pad 2: GNDD -> Net-(U53-FB)
- R408 pad 1: GNDD -> Net-(U53-FB)
- R408 pad 2: GNDD -> GNDREF
- RV3 pad 1: AD1A -> AD1
- RV49 pad 2: /LFO1/LFOA -> LFO2A
- SW24 pad 1: /VCO3/KBV -> KBV
- SW24 pad 3: /VCO3/AD2A -> AD2A
- SW25 pad 1: /VCO3/SAH -> S&H
- SW25 pad 3: /VCO3/LFOA -> LFO2A
- SW4 pad 3: LFOA -> LFO1A
- SW5 pad 3: unconnected-(SW5A-C-Pad3) -> /VCA/Main_Out
- SW5 pad 6: unconnected-(SW5B-C-Pad6) -> /EchoOut
- SW7 pad 3: LFOA -> LFO1A
- U53 pad 2: GNDD -> GNDREF
- U53 pad 5: GNDD -> Net-(U53-FB)
- U54 pad 1: GNDD -> GNDREF
Routing:
- net Net-(C62-Pad2): track 20.2 -> 0.00 mm
- net Net-(U13B--): track 25.4 -> 6.83 mm
- net Net-(R131-Pad1): track 15.1 -> 0.00 mm
- net Net-(C61-Pad2): track 14.9 -> 0.05 mm
- net Net-(U13A-+): track 14.5 -> 0.00 mm
- net Net-(Q2-C): track 20.7 -> 8.01 mm
- net Net-(Q2-E): track 10.8 -> 2.11 mm
- net Net-(U1A--): track 8.67 -> 0.00 mm
- net Net-(Q1-G): track 7.85 -> 0.00 mm
- net Net-(R14-Pad1): track 5.98 -> 0.00 mm
- net Net-(U16C-+): track 5.47 -> 0.00 mm
- net Net-(D1-A): track 5.47 -> 0.00 mm
- net Net-(D6-K): track 5.29 -> 0.00 mm
- net Net-(R18-Pad1): track 5.01 -> 0.00 mm
- net Net-(U16D--): track 4.88 -> 0.00 mm
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
Commit message: my back hurts im routing so much
Parts:
- moved C94 257.8 mm to (174.7, 341.8)
- moved C95 257.8 mm to (177.7, 341.8)
- moved C96 257.8 mm to (180.7, 341.8)
- moved C97 257.8 mm to (183.7, 341.8)
- moved C99 193.6 mm to (154.8, 296.0)
- moved C98 185.8 mm to (228.4, 283.5)
- moved C114 161.7 mm to (240.1, 185.0)
- moved R222 157.5 mm to (238.6, 183.5)
- moved R205 136.9 mm to (217.5, 219.7)
- moved R206 136.9 mm to (220.0, 219.7)
- moved R208 131.1 mm to (214.0, 216.6)
- moved R202 127.7 mm to (196.4, 220.0)
- moved Q26 125.5 mm to (193.9, 219.5), turned to -90 degrees
- moved R180 123.5 mm to (215.9, 219.7)
- moved D35 120.4 mm to (191.0, 207.9), turned to 0 degrees
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Routing:
- net X27: track 1.92 -> 0.00 mm
- net Net-(U11--): track 1.41 -> 0.00 mm
