File: RP2040Microcontroller.kicad_sch (KiCad schematic)
At the start: 117 parts, among them J15 Micro_SD_Card, J41 DIN-504D-M5, J42 USB_B, J5 Conn_01x18, SW56 SW_Push, SW58 SW_Push, U40 6N138, U44 MCP23017_SS, U45 REF3012, U46 MCP4728, U47 TL074, U48 CD74HC4067SM, U49 TL074

Commit message: routing microcontroller
Parts:
- removed D? (x16): LED, LED_THT:LED_D3.0mm, symbol Device:LED
- removed R? (x16): 470, Resistor_SMD:R_0603_1608Metric, symbol Device:R_US
- removed R? (x2): 100k, Resistor_SMD:R_0603_1608Metric, symbol Device:R_US
- removed RV? (x3): 100k, Potentiometer_THT:Potentiometer_Alps_RK09K_Single_Vertical, symbol SynthProj-rescue:R_POT_US-Device
- removed SW58: SW_Push, Button_Switch_THT:SW_PUSH_6mm_H13mm, symbol Switch:SW_Push
- removed U44: MCP23017_SS, Package_SO:SSOP-28_5.3x10.2mm_P0.65mm, symbol Interface_Expansion:MCP23017_SS
- removed U48: CD74HC4067SM, Package_SO:SSOP-24_5.3x8.2mm_P0.65mm, symbol 74xx:CD74HC4067SM
- removed unit 4 of U49
- added D10, D39, D40, D41, D42, D43, D44, D45: LED_Dual_KAK, LED_THT:LED_D3.0mm-3, symbol Device:LED_Dual_KAK
- added R? (x5): 100k, Resistor_SMD:R_0603_1608Metric, symbol Device:R_US
- added R? (x16): 330, Resistor_SMD:R_0805_2012Metric, symbol Device:R_US
- added RV?: 100k, Potentiometer_THT:Potentiometer_Alps_RK09K_Single_Vertical, symbol SynthProj-rescue:R_POT_US-Device
- added SW30: RotaryEncoder_Switch, Rotary_Encoder:RotaryEncoder_Alps_EC11E-Switch_Vertical_H20mm, symbol Device:RotaryEncoder_Switch
- added SW31, SW32: SW_Push, Button_Switch_THT:SW_PUSH_6mm_H13mm, symbol Switch:SW_Push
- added U21: PCA9685PW, Package_SO:TSSOP-28_4.4x9.7mm_P0.65mm, symbol Driver_LED:PCA9685PW
- added U22: MCP4922-ESL, Package_SO:SOIC-14_3.9x8.7mm_P1.27mm, symbol Analog_DAC:MCP4922-ESL
Connections:
- net GNDD is gone; now on net GNDREF: C?.2, C?.2, C?.2, C?.2, C?.2, C?.2, C?.2, C?.2, C?.2, C?.2, C?.2, C?.2, C?.2, C?.2, C?.2, C?.2, C?.2, C?.2, J42.4 (GND), J42.5 (Shield), J?.2 (Pin_2), R?.2, SW56.2, U40.5 (GND), U46.10 (VSS), U?.1 (GND), U?.19 (TESTEN), U?.4 (GND), U?.57 (GND)
- net +3V3: now also R?.1, R?.1, R?.2, R?.2, RV?.3, SW30.S1, U21.28 (VDD), U22.1 (VDD), U22.11 (VrefB), U22.13 (VrefA)
- net +5V: now also D10.2 (A), D39.2 (A), D40.2 (A), D41.2 (A), D42.2 (A), D43.2 (A), D44.2 (A), D45.2 (A)
- net GNDREF: now also R?.2, RV?.1, SW30.C, SW31.2, SW32.2, U21.14 (VSS), U22.12 (AVSS)
- net GPIO13: now also R?.2, SW30.A
- net GPIO14: now also R?.2, SW30.B
- net GPIO15: now also R?.1, SW30.S2
- net GPIO18: now also R?.1, SW31.1
- net GPIO20: now also R?.1, SW32.1
- net GPIO29_ADC3: now also RV?.2
- net GPIO6: now also U21.27 (SDA)
- net GPIO7: now also U21.26 (SCL)
- net at C?.2: now also U22.10 (VoutB); no longer U46.9 (VOUTD)
- net at C?.2: now also U22.14 (VoutA); no longer U46.8 (VOUTC)
- net VOUT_A renamed DIGILFO_OUT_A
- net VOUT_B renamed DIGILFO_OUT_B
- net VOUT_C renamed DIGIVCO_OUT_A
- net VOUT_D renamed DIGIVCO_OUT_B
- new net: D43.1 (K1), R?.1
- new net: D43.3 (K2), R?.1
- new net: D44.1 (K1), R?.1
- new net: D44.3 (K2), R?.1
- new net: R?.2, U21.10 (LED4)
- new net: R?.2, U21.11 (LED5)
- new net: R?.2, U21.12 (LED6)
- new net: R?.2, U21.13 (LED7)
- new net: R?.2, U21.15 (LED8)
- new net: R?.2, U21.16 (LED9)
- new net: R?.2, U21.17 (LED10)
- new net: R?.2, U21.18 (LED11)
- new net: R?.2, U21.19 (LED12)
- new net: R?.2, U21.20 (LED13)
- new net: R?.2, U21.21 (LED14)
- new net: R?.2, U21.22 (LED15)
- new net: R?.2, U21.6 (LED0)
- new net: R?.2, U21.7 (LED1)
- new net: R?.2, U21.8 (LED2)
- new net: R?.2, U21.9 (LED3)
- new net: D41.1 (K1), R?.1
- new net: D41.3 (K2), R?.1
- new net: D40.1 (K1), R?.1
- new net: D42.3 (K2), R?.1
- new net: D10.3 (K2), R?.1
- new net: D39.1 (K1), R?.1
- new net: D39.3 (K2), R?.1
- new net: D45.3 (K2), R?.1
- new net: D45.1 (K1), R?.1
- new net: D42.1 (K1), R?.1
- new net: D40.3 (K2), R?.1
- new net: D10.1 (K1), R?.1
Other:
- note added: "2 Fast SPI DAC Outputs"
- note added: "2 Slo I2C DAC Output"
- note added: "3 ADC Input"
- note added: "Encoder Data"
- note added: "Potentiometer Input"
- note added: "Push Rotary Encoder Input"
- note removed: "8 LEDS for the potentiometers"
- note removed: "8 LEDS for the pushbuttons"
- note removed: "Analog Mux Data"
- note removed: "Potentiometer Inputs"
- note removed: "Quad ADC Input"
- note removed: "Quad I2C DAC Output"
- moved on the sheet: C?, D?, J15, J41, J5, J?, R?, SW56, TP?, U40, U45, U47A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
