File: RP2040Microcontroller.kicad_sch (KiCad schematic)
At the start: 112 parts, among them J15 Micro_SD_Card, J41 DIN-504D-M5, J42 USB_B, J5 Conn_01x18, SW30 RotaryEncoder_Switch, SW31 SW_Push, SW32 SW_Push, SW56 SW_Push, U21 PCA9685PW, U22 MCP4922-ESL, U40 6N138, U45 REF3012, U46 MCP4728, U47 TL074, U49 TL074

Commit message: more and more and more and more and more routing
Parts:
- removed C?: 10uF, Capacitor_SMD:C_0805_2012Metric, symbol Device:C
- removed J15: Micro_SD_Card, symbol Connector:Micro_SD_Card
- removed R?: 66.5k, Resistor_SMD:R_0603_1608Metric, symbol Device:R_US
- removed R?: 10k, Resistor_SMD:R_0603_1608Metric, symbol Device:R_US
- removed R?: 1k, Resistor_SMD:R_0603_1608Metric, symbol Device:R
- removed R?: 28.7k, Resistor_SMD:R_0603_1608Metric, symbol Device:R_US
- removed unit 3 of U47
- removed U?: NCP1117-3.3_SOT223, Package_TO_SOT_SMD:SOT-223-3_TabPin2, symbol Regulator_Linear:NCP1117-3.3_SOT223
Connections:
- net GNDREF: now also U21.1 (A0), U21.2 (A1), U21.24 (A5), U21.3 (A2), U21.4 (A3), U21.5 (A4)
- net XOUT: now also C?.1, Y?.2
Other:
- note added: "2 ADC Input"
- note removed: "3 ADC Input"
- moved on the sheet: R?, SW31, SW32, SW56, TP?, U45
