File: PT2399Echo.kicad_sch (KiCad schematic)
At the start: 80 parts, among them Q21 MMBT3904-7-F, Q22 MMBT3904-7-F, Q23 MMBT3906LT1G, Q24 MMBT3906LT1G, U28 TL074, U29 TL074, U30 LM13700, U31 PT2399

Commit message: created manufacturing files
Parts:
- R? (x2), RV? (x5): value 100k -> 50k
Changed lines of the file:
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@@
       (effects (font (size 1.27 1.27)))
     )
-    (property "Value" "100k" (at 49.53 83.82 90)
+    (property "Value" "50k" (at 49.53 83.82 90)
       (effects (font (size 1.27 1.27)))
     )
@@
       (effects (font (size 1.27 1.27)) (justify right))
     )
-    (property "Value" "100k" (at 184.9882 121.793 0)
+    (property "Value" "50k" (at 184.9882 121.793 0)
       (effects (font (size 1.27 1.27)) (justify right))
     )
@@
       (effects (font (size 1.27 1.27)) (justify right))
     )
-    (property "Value" "100k" (at 99.8982 159.893 0)
+    (property "Value" "50k" (at 99.8982 159.893 0)
       (effects (font (size 1.27 1.27)) (justify right))
     )
@@
       (effects (font (size 1.27 1.27)))
     )
-    (property "Value" "100k" (at 49.53 97.79 90)
+    (property "Value" "50k" (at 49.53 97.79 90)
       (effects (font (size 1.27 1.27)))
     )
@@
       (effects (font (size 1.27 1.27)) (justify right))
     )
-    (property "Value" "100k" (at 170.6118 109.347 0)
+    (property "Value" "50k" (at 170.6118 109.347 0)
       (effects (font (size 1.27 1.27)) (justify right))
     )
@@
       (effects (font (size 1.27 1.27)) (justify right))
     )
-    (property "Value" "100k" (at 60.5282 119.253 0)
+    (property "Value" "50k" (at 60.5282 119.253 0)
       (effects (font (size 1.27 1.27)) (justify right))
     )
@@
       (effects (font (size 1.27 1.27)) (justify right))
     )
-    (property "Value" "100k" (at 30.0482 87.503 0)
+    (property "Value" "50k" (at 30.0482 87.503 0)
       (effects (font (size 1.27 1.27)) (justify right))
     )
