File: WhiteNoiseGenerator.kicad_sch (KiCad schematic)
At the start: 22 parts, among them Q13 MMBT3904-7-F, U12 TL072

Commit message: more work...
Parts:
- C49, C50, C51, C52, C55, C58, C60: footprint Capacitor_SMD:C_0805_2012Metric_Pad1.18x1.45mm_HandSolder -> Capacitor_SMD:C_0805_2012Metric
- C53, C54, C56, C57, C59: footprint Capacitor_SMD:C_0805_2012Metric_Pad1.18x1.45mm_HandSolder -> Capacitor_SMD:C_0603_1608Metric
- R116, R117, R118, R119, R120, R121, R122: footprint Resistor_SMD:R_0805_2012Metric_Pad1.20x1.40mm_HandSolder -> Resistor_SMD:R_0603_1608Metric
Changed lines of the file:
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@@
       (effects (font (size 1.27 1.27)))
     )
-    (property "Footprint" "Capacitor_SMD:C_0805_2012Metric_Pad1.18x1.45mm_HandSolder" (at 79.0448 154.94 0)
+    (property "Footprint" "Capacitor_SMD:C_0805_2012Metric" (at 79.0448 154.94 0)
       (effects (font (size 1.27 1.27)) hide)
     )
@@
       (effects (font (size 1.27 1.27)))
     )
-    (property "Footprint" "Capacitor_SMD:C_0805_2012Metric_Pad1.18x1.45mm_HandSolder" (at 85.3948 154.94 0)
+    (property "Footprint" "Capacitor_SMD:C_0805_2012Metric" (at 85.3948 154.94 0)
       (effects (font (size 1.27 1.27)) hide)
     )
@@
       (effects (font (size 1.27 1.27)))
     )
-    (property "Footprint" "Capacitor_SMD:C_0805_2012Metric_Pad1.18x1.45mm_HandSolder" (at 91.7448 154.94 0)
+    (property "Footprint" "Capacitor_SMD:C_0603_1608Metric" (at 91.7448 154.94 0)
       (effects (font (size 1.27 1.27)) hide)
     )
@@
       (effects (font (size 1.27 1.27)))
     )
-    (property "Footprint" "Capacitor_SMD:C_0805_2012Metric_Pad1.18x1.45mm_HandSolder" (at 79.0448 162.56 0)
+    (property "Footprint" "Capacitor_SMD:C_0805_2012Metric" (at 79.0448 162.56 0)
       (effects (font (size 1.27 1.27)) hide)
     )
@@
       (effects (font (size 1.27 1.27)))
     )
-    (property "Footprint" "Capacitor_SMD:C_0805_2012Metric_Pad1.18x1.45mm_HandSolder" (at 85.3948 162.56 0)
+    (property "Footprint" "Capacitor_SMD:C_0805_2012Metric" (at 85.3948 162.56 0)
       (effects (font (size 1.27 1.27)) hide)
     )
@@
       (effects (font (size 1.27 1.27)))
     )
-    (property "Footprint" "Capacitor_SMD:C_0805_2012Metric_Pad1.18x1.45mm_HandSolder" (at 91.7448 162.56 0)
+    (property "Footprint" "Capacitor_SMD:C_0603_1608Metric" (at 91.7448 162.56 0)
       (effects (font (size 1.27 1.27)) hide)
     )
@@
       (effects (font (size 1.27 1.27)))
     )
-    (property "Footprint" "Resistor_SMD:R_0805_2012Metric_Pad1.20x1.40mm_HandSolder" (at 110.744 73.406 90)
+    (property "Footprint" "Resistor_SMD:R_0603_1608Metric" (at 110.744 73.406 90)
       (effects (font (size 1.27 1.27)) hide)
     )
@@
       (effects (font (size 1.27 1.27)))
     )
-    (property "Footprint" "Capacitor_SMD:C_0805_2012Metric_Pad1.18x1.45mm_HandSolder" (at 121.92 80.3148 0)
+    (property "Footprint" "Capacitor_SMD:C_0603_1608Metric" (at 121.92 80.3148 0)
       (effects (font (size 1.27 1.27)) hide)
     )
@@
       (effects (font (size 1.27 1.27)))
     )
-    (property "Footprint" "Resistor_SMD:R_0805_2012Metric_Pad1.20x1.40mm_HandSolder" (at 139.954 66.294 90)
+    (property "Footprint" "Resistor_SMD:R_0603_1608Metric" (at 139.954 66.294 90)
       (effects (font (size 1.27 1.27)) hide)
     )
@@
       (effects (font (size 1.27 1.27)))
     )
-    (property "Footprint" "Resistor_SMD:R_0805_2012Metric_Pad1.20x1.40mm_HandSolder" (at 138.684 91.694 90)
+    (property "Footprint" "Resistor_SMD:R_0603_1608Metric" (at 138.684 91.694 90)
       (effects (font (size 1.27 1.27)) hide)
     )
@@
       (effects (font (size 1.27 1.27)))
     )
-    (property "Footprint" "Capacitor_SMD:C_0805_2012Metric_Pad1.18x1.45mm_HandSolder" (at 142.24 100.6348 0)
+    (property "Footprint" "Capacitor_SMD:C_0603_1608Metric" (at 142.24 100.6348 0)
       (effects (font (size 1.27 1.27)) hide)
     )
@@
       (effects (font (size 1.27 1.27)))
     )
-    (property "Footprint" "Capacitor_SMD:C_0805_2012Metric_Pad1.18x1.45mm_HandSolder" (at 158.75 82.8548 0)
+    (property "Footprint" "Capacitor_SMD:C_0805_2012Metric" (at 158.75 82.8548 0)
       (effects (font (size 1.27 1.27)) hide)
     )
@@
       (effects (font (size 1.27 1.27)))
     )
-    (property "Footprint" "Capacitor_SMD:C_0805_2012Metric_Pad1.18x1.45mm_HandSolder" (at 190.5 85.3948 0)
+    (property "Footprint" "Capacitor_SMD:C_0805_2012Metric" (at 190.5 85.3948 0)
       (effects (font (size 1.27 1.27)) hide)
     )
@@
       (effects (font (size 1.27 1.27)))
     )
-    (property "Footprint" "Resistor_SMD:R_0805_2012Metric_Pad1.20x1.40mm_HandSolder" (at 171.704 92.964 90)
+    (property "Footprint" "Resistor_SMD:R_0603_1608Metric" (at 171.704 92.964 90)
       (effects (font (size 1.27 1.27)) hide)
     )
@@
       (effects (font (size 1.27 1.27)))
     )
-    (property "Footprint" "Capacitor_SMD:C_0805_2012Metric_Pad1.18x1.45mm_HandSolder" (at 175.26 101.9048 0)
+    (property "Footprint" "Capacitor_SMD:C_0603_1608Metric" (at 175.26 101.9048 0)
       (effects (font (size 1.27 1.27)) hide)
     )
@@
       (effects (font (size 1.27 1.27)))
     )
-    (property "Footprint" "Resistor_SMD:R_0805_2012Metric_Pad1.20x1.40mm_HandSolder" (at 128.524 107.696 90)
+    (property "Footprint" "Resistor_SMD:R_0603_1608Metric" (at 128.524 107.696 90)
       (effects (font (size 1.27 1.27)) hide)
     )
@@
       (effects (font (size 1.27 1.27)))
     )
-    (property "Footprint" "Capacitor_SMD:C_0805_2012Metric_Pad1.18x1.45mm_HandSolder" (at 96.8248 81.28 0)
+    (property "Footprint" "Capacitor_SMD:C_0805_2012Metric" (at 96.8248 81.28 0)
       (effects (font (size 1.27 1.27)) hide)
     )
@@
       (effects (font (size 1.27 1.27)))
     )
-    (property "Footprint" "Resistor_SMD:R_0805_2012Metric_Pad1.20x1.40mm_HandSolder" (at 110.744 65.786 90)
+    (property "Footprint" "Resistor_SMD:R_0603_1608Metric" (at 110.744 65.786 90)
       (effects (font (size 1.27 1.27)) hide)
     )
@@
       (effects (font (size 1.27 1.27)))
     )
-    (property "Footprint" "Resistor_SMD:R_0805_2012Metric_Pad1.20x1.40mm_HandSolder" (at 175.514 68.834 90)
-      (effects (font (size 1.27 1.27)) hide)
-    )
+    (property "Footprint" "Resistor_SMD:R_0603_1608Metric" (at 175.514 68.834 90)
+      (effects (font (size 1.27 1.27)) hide)
+    )

Commit message: Doing some layout
Parts:
- RV25: footprint Potentiometer_THT:Potentiometer_Alps_RK09K_Single_Vertical -> Potentiometer_SMD:Potentiometer_Bourns_TC33X_Vertical
Changed lines of the file:
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@@
       (effects (font (size 1.27 1.27)) (justify right))
     )
-    (property "Footprint" "Potentiometer_THT:Potentiometer_Alps_RK09K_Single_Vertical" (at 160.02 113.03 0)
+    (property "Footprint" "Potentiometer_SMD:Potentiometer_Bourns_TC33X_Vertical" (at 160.02 113.03 0)
       (effects (font (size 1.27 1.27)) hide)
     )

Commit message: routing work...
Parts:
- added unit 3 of U12
Connections:
- net +12V: now also U12.8 (V+)
- net -12V: now also U12.4 (V-)
Changed lines of the file:
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@@
     (effects (font (size 1.27 1.27)) (justify left))
-  )
-  (symbol (lib_id "power:+12V") (at 60.96 153.67 0) (unit 1)
-    (in_bom yes) (on_board yes) (dnp no)
-    (property "Reference" "#PWR0152" (at 60.96 157.48 0)
-      (effects (font (size 1.27 1.27)) hide)
-    )
-    (property "Value" "+12V" (at 61.341 149.2758 0)
-      (effects (font (size 1.27 1.27)))
-    )
-    (property "Footprint" "" (at 60.96 153.67 0)
-      (effects (font (size 1.27 1.27)) hide)
-    )
-    (property "Datasheet" "" (at 60.96 153.67 0)
-      (effects (font (size 1.27 1.27)) hide)
-    )
-    (pin "1")
-    (instances
-      (project "SynthProj"
-        (path "/9021c97e-351f-4ed9-b393-50257df6a463/00000000-0000-0000-0000-000066016bf3"
-          (reference "#PWR0152") (unit 1)
-        )
-        (path "/9021c97e-351f-4ed9-b393-50257df6a463/00000000-0000-0000-0000-0000659a4e2e"
-          (reference "#PWR?") (unit 1)
-        )
-      )
-    )
-  )
-  (symbol (lib_id "power:-12V") (at 60.96 168.91 180) (unit 1)
-    (in_bom yes) (on_board yes) (dnp no)
-    (property "Reference" "#PWR0153" (at 60.96 171.45 0)
-      (effects (font (size 1.27 1.27)) hide)
-    )
-    (property "Value" "-12V" (at 60.579 173.3042 0)
-      (effects (font (size 1.27 1.27)))
-    )
-    (property "Footprint" "" (at 60.96 168.91 0)
-      (effects (font (size 1.27 1.27)) hide)
-    )
-    (property "Datasheet" "" (at 60.96 168.91 0)
-      (effects (font (size 1.27 1.27)) hide)
-    )
-    (pin "1")
-    (instances
-      (project "SynthProj"
-        (path "/9021c97e-351f-4ed9-b393-50257df6a463/00000000-0000-0000-0000-000066016bf3"
-          (reference "#PWR0153") (unit 1)
-        )
-        (path "/9021c97e-351f-4ed9-b393-50257df6a463/00000000-0000-0000-0000-0000659a4e2e"
-          (reference "#PWR?") (unit 1)
-        )
-      )
-    )
   )
   (symbol (lib_id "power:+12V") (at 80.01 154.94 0) (unit 1)
@@
         )
       )
+    )
+  )
+  (symbol (lib_id "power:+12V") (at 107.315 155.575 0) (unit 1)
+    (in_bom yes) (on_board yes) (dnp no)
+    (property "Reference" "#PWR0171" (at 107.315 159.385 0)
+      (effects (font (size 1.27 1.27)) hide)
+    )
+    (property "Value" "+12V" (at 107.696 151.1808 0)
+      (effects (font (size 1.27 1.27)))
+    )
+    (property "Footprint" "" (at 107.315 155.575 0)
+      (effects (font (size 1.27 1.27)) hide)
+    )
+    (property "Datasheet" "" (at 107.315 155.575 0)
+      (effects (font (size 1.27 1.27)) hide)
+    )
+    (pin "1")
+    (instances
+      (project "SynthProj"
+        (path "/9021c97e-351f-4ed9-b393-50257df6a463/00000000-0000-0000-0000-000066b08086"
+          (reference "#PWR0171") (unit 1)
+        )
+        (path "/9021c97e-351f-4ed9-b393-50257df6a463/00000000-0000-0000-0000-000066016bf3"
+          (reference "#PWR016") (unit 1)
+        )
+      )
+    )
+  )
+  (symbol (lib_id "Amplifier_Operational:TL072") (at 109.855 163.195 0) (unit 3)
+    (in_bom yes) (on_board yes) (dnp no)
+    (property "Reference" "U12" (at 108.7882 162.0266 0)
+      (effects (font (size 1.27 1.27)) (justify left))
+    )
+    (property "Value" "TL072" (at 108.7882 164.338 0)
+      (effects (font (size 1.27 1.27)) (justify left))
+    )
+    (property "Footprint" "Package_SO:SO-8_3.9x4.9mm_P1.27mm" (at 109.855 163.195 0)
+      (effects (font (size 1.27 1.27)) hide)
+    )
+    (property "Datasheet" "http://www.ti.com/lit/ds/symlink/tl071.pdf" (at 109.855 163.195 0)
+      (effects (font (size 1.27 1.27)) hide)
+    )
+    (pin "2")
+    (pin "5")
+    (pin "1")
+    (pin "6")
+    (pin "3")
+    (pin "8")
+    (pin "7")
+    (pin "4")
+    (instances
+      (project "SynthProj"
+        (path "/9021c97e-351f-4ed9-b393-50257df6a463/00000000-0000-0000-0000-000066b08086"
+          (reference "U12") (unit 3)
+        )
+        (path "/9021c97e-351f-4ed9-b393-50257df6a463/00000000-0000-0000-0000-000066016bf3"
+          (reference "U12") (unit 3)
+        )
+      )
+    )
+  )
+  (symbol (lib_id "power:-12V") (at 107.315 170.815 180) (unit 1)
+    (in_bom yes) (on_board yes) (dnp no)
+    (property "Reference" "#PWR0172" (at 107.315 173.355 0)
+      (effects (font (size 1.27 1.27)) hide)
+    )
+    (property "Value" "-12V" (at 106.934 175.2092 0)
+      (effects (font (size 1.27 1.27)))
+    )
+    (property "Footprint" "" (at 107.315 170.815 0)
+      (effects (font (size 1.27 1.27)) hide)
+    )
+    (property "Datasheet" "" (at 107.315 170.815 0)
+      (effects (font (size 1.27 1.27)) hide)
+    )
+    (pin "1")
+    (instances
+      (project "SynthProj"
+        (path "/9021c97e-351f-4ed9-b393-50257df6a463/00000000-0000-0000-0000-000066b08086"
+          (reference "#PWR0172") (unit 1)
+        )
+        (path "/9021c97e-351f-4ed9-b393-50257df6a463/00000000-0000-0000-0000-000066016bf3"
+          (reference "#PWR017") (unit 1)
+        )
+      )

Commit message: more and more and more and more and more routing
Parts:
- removed C49, C50: 4.7uF, Capacitor_SMD:C_0805_2012Metric, symbol Device:C
- removed C53, C54: 47nF, Capacitor_SMD:C_0603_1608Metric, symbol Device:C
Changed lines of the file:
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@@
   (junction (at 97.79 88.9) (diameter 0) (color 0 0 0 0)
   )
-  (junction (at 86.36 154.94) (diameter 0) (color 0 0 0 0)
-  )
   (junction (at 148.59 92.71) (diameter 0) (color 0 0 0 0)
   )
@@
   (junction (at 111.76 69.85) (diameter 0) (color 0 0 0 0)
   )
-  (junction (at 86.36 170.18) (diameter 0) (color 0 0 0 0)
-  )
   (junction (at 160.02 107.95) (diameter 0) (color 0 0 0 0)
   )
-  (junction (at 80.01 162.56) (diameter 0) (color 0 0 0 0)
-  )
   (junction (at 86.36 162.56) (diameter 0) (color 0 0 0 0)
   )
   (junction (at 180.34 86.36) (diameter 0) (color 0 0 0 0)
   )
-  (junction (at 80.01 154.94) (diameter 0) (color 0 0 0 0)
-  )
   (junction (at 129.54 101.6) (diameter 0) (color 0 0 0 0)
   )
@@
   (junction (at 180.34 93.98) (diameter 0) (color 0 0 0 0)
   )
-  (junction (at 92.71 162.56) (diameter 0) (color 0 0 0 0)
-  )
-  (junction (at 80.01 170.18) (diameter 0) (color 0 0 0 0)
-  )
   (junction (at 160.02 102.87) (diameter 0) (color 0 0 0 0)
   )
@@
     (stroke (width 0) (type default))
   )
-  (wire (pts (xy 86.36 170.18) (xy 92.71 170.18))
-    (stroke (width 0) (type default))
-  )
   (wire (pts (xy 125.73 81.28) (xy 121.92 81.28))
     (stroke (width 0) (type default))
@@
     (stroke (width 0) (type default))
   )
-  (wire (pts (xy 86.36 154.94) (xy 92.71 154.94))
-    (stroke (width 0) (type default))
-  )
   (wire (pts (xy 129.54 101.6) (xy 129.54 92.71))
     (stroke (width 0) (type default))
@@
     (stroke (width 0) (type default))
   )
-  (wire (pts (xy 76.2 162.56) (xy 80.01 162.56))
-    (stroke (width 0) (type default))
-  )
-  (wire (pts (xy 80.01 162.56) (xy 86.36 162.56))
-    (stroke (width 0) (type default))
-  )
-  (wire (pts (xy 86.36 162.56) (xy 92.71 162.56))
+  (wire (pts (xy 76.2 162.56) (xy 86.36 162.56))
     (stroke (width 0) (type default))
   )
@@
     )
   )
-  (symbol (lib_id "Device:C") (at 80.01 158.75 180) (unit 1)
-    (in_bom yes) (on_board yes) (dnp no)
-    (property "Reference" "C49" (at 86.4108 158.75 90)
-      (effects (font (size 1.27 1.27)))
-    )
-    (property "Value" "4.7uF" (at 84.0994 158.75 90)
-      (effects (font (size 1.27 1.27)))
-    )
-    (property "Footprint" "Capacitor_SMD:C_0805_2012Metric" (at 79.0448 154.94 0)
-      (effects (font (size 1.27 1.27)) hide)
-    )
-    (property "Datasheet" "~" (at 80.01 158.75 0)
+  (symbol (lib_id "Device:C") (at 86.36 158.75 180) (unit 1)
+    (in_bom yes) (on_board yes) (dnp no)
+    (property "Reference" "C51" (at 92.7608 158.75 90)
+      (effects (font (size 1.27 1.27)))
+    )
+    (property "Value" "470nF" (at 90.4494 158.75 90)
+      (effects (font (size 1.27 1.27)))
+    )
+    (property "Footprint" "Capacitor_SMD:C_0805_2012Metric" (at 85.3948 154.94 0)
+      (effects (font (size 1.27 1.27)) hide)
+    )
+    (property "Datasheet" "~" (at 86.36 158.75 0)
       (effects (font (size 1.27 1.27)) hide)
     )
@@
       (project "SynthProj"
         (path "/9021c97e-351f-4ed9-b393-50257df6a463/00000000-0000-0000-0000-000066016bf3"
-          (reference "C49") (unit 1)
+          (reference "C51") (unit 1)
         )
         (path "/9021c97e-351f-4ed9-b393-50257df6a463/00000000-0000-0000-0000-0000659a4e2e"
@@
     )
   )
-  (symbol (lib_id "Device:C") (at 86.36 158.75 180) (unit 1)
-    (in_bom yes) (on_board yes) (dnp no)
-    (property "Reference" "C51" (at 92.7608 158.75 90)
-      (effects (font (size 1.27 1.27)))
-    )
-    (property "Value" "470nF" (at 90.4494 158.75 90)
-      (effects (font (size 1.27 1.27)))
-    )
-    (property "Footprint" "Capacitor_SMD:C_0805_2012Metric" (at 85.3948 154.94 0)
-      (effects (font (size 1.27 1.27)) hide)
-    )
-    (property "Datasheet" "~" (at 86.36 158.75 0)
-      (effects (font (size 1.27 1.27)) hide)
-    )
+  (symbol (lib_id "Device:C") (at 86.36 166.37 180) (unit 1)
+    (in_bom yes) (on_board yes) (dnp no)
+    (property "Reference" "C52" (at 92.7608 166.37 90)
+      (effects (font (size 1.27 1.27)))
+    )
+    (property "Value" "470nF" (at 90.4494 166.37 90)
+      (effects (font (size 1.27 1.27)))
+    )
+    (property "Footprint" "Capacitor_SMD:C_0805_2012Metric" (at 85.3948 162.56 0)
+      (effects (font (size 1.27 1.27)) hide)
+    )
+    (property "Datasheet" "~" (at 86.36 166.37 0)
+      (effects (font (size 1.27 1.27)) hide)
+    )
+    (pin "1")
     (pin "2")
-    (pin "1")
-    (instances
-      (project "SynthProj"
-        (path "/9021c97e-351f-4ed9-b393-50257df6a463/00000000-0000-0000-0000-000066016bf3"
-          (reference "C51") (unit 1)
-        )
-        (path "/9021c97e-351f-4ed9-b393-50257df6a463/00000000-0000-0000-0000-0000659a4e2e"
-          (reference "C?") (unit 1)
-        )
-      )
-    )
-  )
-  (symbol (lib_id "Device:C") (at 92.71 158.75 180) (unit 1)
-    (in_bom yes) (on_board yes) (dnp no)
-    (property "Reference" "C53" (at 99.1108 158.75 90)
-      (effects (font (size 1.27 1.27)))
-    )
-    (property "Value" "47nF" (at 96.7994 158.75 90)
-      (effects (font (size 1.27 1.27)))
-    )
-    (property "Footprint" "Capacitor_SMD:C_0603_1608Metric" (at 91.7448 154.94 0)
-      (effects (font (size 1.27 1.27)) hide)
-    )
-    (property "Datasheet" "~" (at 92.71 158.75 0)
-      (effects (font (size 1.27 1.27)) hide)
-    )
-    (pin "1")
-    (pin "2")
-    (instances
-      (project "SynthProj"
-        (path "/9021c97e-351f-4ed9-b393-50257df6a463/00000000-0000-0000-0000-000066016bf3"
-          (reference "C53") (unit 1)
-        )
-        (path "/9021c97e-351f-4ed9-b393-50257df6a463/00000000-0000-0000-0000-0000659a4e2e"
-          (reference "C?") (unit 1)
-        )
-      )
-    )
-  )
-  (symbol (lib_id "Device:C") (at 80.01 166.37 180) (unit 1)
-    (in_bom yes) (on_board yes) (dnp no)
-    (property "Reference" "C50" (at 86.4108 166.37 90)
-      (effects (font (size 1.27 1.27)))
-    )
-    (property "Value" "4.7uF" (at 84.0994 166.37 90)
-      (effects (font (size 1.27 1.27)))
-    )
-    (property "Footprint" "Capacitor_SMD:C_0805_2012Metric" (at 79.0448 162.56 0)
-      (effects (font (size 1.27 1.27)) hide)
-    )
-    (property "Datasheet" "~" (at 80.01 166.37 0)
-      (effects (font (size 1.27 1.27)) hide)
-    )
-    (pin "2")
-    (pin "1")
-    (instances
-      (project "SynthProj"
-        (path "/9021c97e-351f-4ed9-b393-50257df6a463/00000000-0000-0000-0000-000066016bf3"
-          (reference "C50") (unit 1)
-        )
-        (path "/9021c97e-351f-4ed9-b393-50257df6a463/00000000-0000-0000-0000-0000659a4e2e"
-          (reference "C?") (unit 1)
-        )
-      )
-    )
-  )
-  (symbol (lib_id "Device:C") (at 86.36 166.37 180) (unit 1)
-    (in_bom yes) (on_board yes) (dnp no)
-    (property "Reference" "C52" (at 92.7608 166.37 90)
-      (effects (font (size 1.27 1.27)))
-    )
-    (property "Value" "470nF" (at 90.4494 166.37 90)
-      (effects (font (size 1.27 1.27)))
-    )
-    (property "Footprint" "Capacitor_SMD:C_0805_2012Metric" (at 85.3948 162.56 0)
-      (effects (font (size 1.27 1.27)) hide)
-    )
-    (property "Datasheet" "~" (at 86.36 166.37 0)
-      (effects (font (size 1.27 1.27)) hide)
-    )
-    (pin "1")
-    (pin "2")
     (instances
       (project "SynthProj"
@@
         )
         (path "/9021c97e-351f-4ed9-b393-50257df6a463/00000000-0000-0000-0000-0000659a4e2e"
-          (reference "C?") (unit 1)
-        )
-      )
-    )
-  )
-  (symbol (lib_id "Device:C") (at 92.71 166.37 180) (unit 1)
-    (in_bom yes) (on_board yes) (dnp no)
-    (property "Reference" "C54" (at 99.1108 166.37 90)
-      (effects (font (size 1.27 1.27)))
-    )
-    (property "Value" "47nF" (at 96.7994 166.37 90)
-      (effects (font (size 1.27 1.27)))
-    )
-    (property "Footprint" "Capacitor_SMD:C_0603_1608Metric" (at 91.7448 162.56 0)
-      (effects (font (size 1.27 1.27)) hide)
-    )
-    (property "Datasheet" "~" (at 92.71 166.37 0)
-      (effects (font (size 1.27 1.27)) hide)
-    )
-    (pin "2")
-    (pin "1")
-    (instances
-      (project "SynthProj"
-        (path "/9021c97e-351f-4ed9-b393-50257df6a463/00000000-0000-0000-0000-000066016bf3"
-          (reference "C54") (unit 1)
-        )
-        (path "/9021c97e-351f-4ed9-b393-50257df6a463/00000000-0000-0000-0000-0000659a4e2e"
