File: AD_Envelope.kicad_sch (KiCad schematic)
At the start: 87 parts, among them Q15 MMBT3906LT1G, Q18 MMBT3906LT1G, SW14 SW_SPST, SW15 SW_Push, SW16 SW_SPST, SW17 SW_SPDT, SW18 SW_SPDT, SW19 SW_Push, SW20 SW_DPST, SW21 SW_DPST, SW22 SW_SPST, SW23 SW_SPST, U14 TL072, U15 TL074

Commit message: created manufacturing files
Parts:
- R155, R156: value 1k -> 50k
- RV28, RV29, RV30, RV31, RV32, RV33: value 1M -> 50k
- RV34, RV35: value 100k -> 50k
Connections:
- net X56: now also RV31.1; no longer RV31.3
- net X61: now also RV31.3; no longer RV31.1
Other:
- note added: "Might have to fidle with this value to match the 50k pots"
- moved on the sheet: RV31
Changed lines of the file:
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@@
     (stroke (width 0) (type default))
   )
+  (arc (start 145.415 121.92) (mid 146.4458 127.635) (end 145.415 133.35)
+    (stroke (width 0) (type default))
+    (fill (type none))
+  )
+  (circle (center 143.51 137.16) (radius 4.066)
+    (stroke (width 0) (type default))
+    (fill (type none))
+  )
   (text "Gate Ind" (at 114.3 80.01 0)
     (effects (font (size 1.27 1.27)) (justify left bottom))
@@
     (effects (font (size 1.27 1.27)) (justify left bottom))
   )
+  (text "Might have to fidle with this value to match the 50k pots"
+    (at 120.015 121.285 0)
+    (effects (font (size 1.27 1.27)) (justify left bottom))
+  )
   (text "Repeat" (at 43.18 86.36 0)
     (effects (font (size 1.27 1.27)) (justify left bottom))
@@
       (effects (font (size 1.27 1.27)))
     )
-    (property "Value" "1k" (at 151.13 47.9044 90)
+    (property "Value" "50k" (at 151.13 47.9044 90)
       (effects (font (size 1.27 1.27)))
     )
@@
       (effects (font (size 1.27 1.27)) (justify right))
     )
-    (property "Value" "1M" (at 195.453 52.5018 0)
+    (property "Value" "50k" (at 195.453 52.5018 0)
       (effects (font (size 1.27 1.27)) (justify right))
     )
@@
       (effects (font (size 1.27 1.27)) (justify right))
     )
-    (property "Value" "1M" (at 195.453 34.7218 0)
+    (property "Value" "50k" (at 195.453 34.7218 0)
       (effects (font (size 1.27 1.27)) (justify right))
     )
@@
       (effects (font (size 1.27 1.27)) (justify right))
     )
-    (property "Value" "100k" (at 226.8982 53.213 0)
+    (property "Value" "50k" (at 226.8982 53.213 0)
       (effects (font (size 1.27 1.27)) (justify right))
     )
@@
       (effects (font (size 1.27 1.27)) (justify right))
     )
-    (property "Value" "1M" (at 64.643 99.4918 0)
+    (property "Value" "50k" (at 64.643 99.4918 0)
       (effects (font (size 1.27 1.27)) (justify right))
     )
@@
       (effects (font (size 1.27 1.27)) (justify right))
     )
-    (property "Value" "1M" (at 143.383 100.7618 0)
+    (property "Value" "50k" (at 143.383 100.7618 0)
       (effects (font (size 1.27 1.27)) (justify right))
     )
@@
       (effects (font (size 1.27 1.27)))
     )
-    (property "Value" "1k" (at 143.51 140.0556 90)
+    (property "Value" "50k" (at 143.51 140.0556 90)
       (effects (font (size 1.27 1.27)))
     )
@@
     )
   )
-  (symbol (lib_id "SynthProj-rescue:R_POT_US-Device") (at 189.23 147.32 90) (unit 1)
+  (symbol (lib_id "SynthProj-rescue:R_POT_US-Device") (at 189.23 147.32 270) (mirror x) (unit 1)
     (in_bom yes) (on_board yes) (dnp no)
-    (property "Reference" "RV31" (at 188.0616 149.0218 0)
+    (property "Reference" "RV31" (at 190.3984 149.0218 0)
       (effects (font (size 1.27 1.27)) (justify right))
     )
-    (property "Value" "1M" (at 190.373 149.0218 0)
+    (property "Value" "50k" (at 188.087 149.0218 0)
       (effects (font (size 1.27 1.27)) (justify right))
     )
@@
       (effects (font (size 1.27 1.27)) (justify right))
     )
-    (property "Value" "1M" (at 190.373 131.2418 0)
+    (property "Value" "50k" (at 190.373 131.2418 0)
       (effects (font (size 1.27 1.27)) (justify right))
     )
@@
       (effects (font (size 1.27 1.27)) (justify right))
     )
-    (property "Value" "100k" (at 221.8182 149.733 0)
+    (property "Value" "50k" (at 221.8182 149.733 0)
       (effects (font (size 1.27 1.27)) (justify right))
     )
