File: LFO.kicad_sch (KiCad schematic)
At the start: 29 parts, among them Q14 MMBT3904-7-F, SW11 SW_SPDT, SW12 SW_SP3T, SW13 SW_Push_DPDT, U12 TL072, U13 TL072

Commit message: more work...
Parts:
- C61, C66, C67: footprint Capacitor_SMD:C_0805_2012Metric_Pad1.18x1.45mm_HandSolder -> Capacitor_SMD:C_0603_1608Metric
- C62, C63, C64, C65: footprint Capacitor_SMD:C_0805_2012Metric_Pad1.18x1.45mm_HandSolder -> Capacitor_SMD:C_0805_2012Metric
- R123, R124, R125, R126, R127, R128, R129, R130, R131, R132, R133: footprint Resistor_SMD:R_0805_2012Metric_Pad1.20x1.40mm_HandSolder -> Resistor_SMD:R_0603_1608Metric
Changed lines of the file:
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@@
       (effects (font (size 1.27 1.27)))
     )
-    (property "Footprint" "Capacitor_SMD:C_0805_2012Metric_Pad1.18x1.45mm_HandSolder" (at 253.0348 63.5 0)
+    (property "Footprint" "Capacitor_SMD:C_0805_2012Metric" (at 253.0348 63.5 0)
       (effects (font (size 1.27 1.27)) hide)
     )
@@
       (effects (font (size 1.27 1.27)))
     )
-    (property "Footprint" "Capacitor_SMD:C_0805_2012Metric_Pad1.18x1.45mm_HandSolder" (at 259.3848 63.5 0)
+    (property "Footprint" "Capacitor_SMD:C_0805_2012Metric" (at 259.3848 63.5 0)
       (effects (font (size 1.27 1.27)) hide)
     )
@@
       (effects (font (size 1.27 1.27)))
     )
-    (property "Footprint" "Capacitor_SMD:C_0805_2012Metric_Pad1.18x1.45mm_HandSolder" (at 265.7348 63.5 0)
+    (property "Footprint" "Capacitor_SMD:C_0603_1608Metric" (at 265.7348 63.5 0)
       (effects (font (size 1.27 1.27)) hide)
     )
@@
       (effects (font (size 1.27 1.27)))
     )
-    (property "Footprint" "Capacitor_SMD:C_0805_2012Metric_Pad1.18x1.45mm_HandSolder" (at 253.0348 71.12 0)
+    (property "Footprint" "Capacitor_SMD:C_0805_2012Metric" (at 253.0348 71.12 0)
       (effects (font (size 1.27 1.27)) hide)
     )
@@
       (effects (font (size 1.27 1.27)))
     )
-    (property "Footprint" "Capacitor_SMD:C_0805_2012Metric_Pad1.18x1.45mm_HandSolder" (at 259.3848 71.12 0)
+    (property "Footprint" "Capacitor_SMD:C_0805_2012Metric" (at 259.3848 71.12 0)
       (effects (font (size 1.27 1.27)) hide)
     )
@@
       (effects (font (size 1.27 1.27)))
     )
-    (property "Footprint" "Capacitor_SMD:C_0805_2012Metric_Pad1.18x1.45mm_HandSolder" (at 265.7348 71.12 0)
+    (property "Footprint" "Capacitor_SMD:C_0603_1608Metric" (at 265.7348 71.12 0)
       (effects (font (size 1.27 1.27)) hide)
     )
@@
       (effects (font (size 1.27 1.27)))
     )
-    (property "Footprint" "Resistor_SMD:R_0805_2012Metric_Pad1.20x1.40mm_HandSolder" (at 98.044 109.474 90)
+    (property "Footprint" "Resistor_SMD:R_0603_1608Metric" (at 98.044 109.474 90)
       (effects (font (size 1.27 1.27)) hide)
     )
@@
       (effects (font (size 1.27 1.27)))
     )
-    (property "Footprint" "Resistor_SMD:R_0805_2012Metric_Pad1.20x1.40mm_HandSolder" (at 129.286 82.804 90)
+    (property "Footprint" "Resistor_SMD:R_0603_1608Metric" (at 129.286 82.804 90)
       (effects (font (size 1.27 1.27)) hide)
     )
@@
       (effects (font (size 1.27 1.27)))
     )
-    (property "Footprint" "Resistor_SMD:R_0805_2012Metric_Pad1.20x1.40mm_HandSolder" (at 158.496 108.204 90)
+    (property "Footprint" "Resistor_SMD:R_0603_1608Metric" (at 158.496 108.204 90)
       (effects (font (size 1.27 1.27)) hide)
     )
@@
       (effects (font (size 1.27 1.27)))
     )
-    (property "Footprint" "Resistor_SMD:R_0805_2012Metric_Pad1.20x1.40mm_HandSolder" (at 166.116 117.856 90)
+    (property "Footprint" "Resistor_SMD:R_0603_1608Metric" (at 166.116 117.856 90)
       (effects (font (size 1.27 1.27)) hide)
     )
@@
       (effects (font (size 1.27 1.27)))
     )
-    (property "Footprint" "Resistor_SMD:R_0805_2012Metric_Pad1.20x1.40mm_HandSolder" (at 166.116 128.016 90)
+    (property "Footprint" "Resistor_SMD:R_0603_1608Metric" (at 166.116 128.016 90)
       (effects (font (size 1.27 1.27)) hide)
     )
@@
       (effects (font (size 1.27 1.27)))
     )
-    (property "Footprint" "Capacitor_SMD:C_0805_2012Metric_Pad1.18x1.45mm_HandSolder" (at 205.74 108.2548 0)
+    (property "Footprint" "Capacitor_SMD:C_0603_1608Metric" (at 205.74 108.2548 0)
       (effects (font (size 1.27 1.27)) hide)
     )
@@
       (effects (font (size 1.27 1.27)))
     )
-    (property "Footprint" "Resistor_SMD:R_0805_2012Metric_Pad1.20x1.40mm_HandSolder" (at 201.676 103.886 90)
+    (property "Footprint" "Resistor_SMD:R_0603_1608Metric" (at 201.676 103.886 90)
       (effects (font (size 1.27 1.27)) hide)
     )
@@
       (effects (font (size 1.27 1.27)))
     )
-    (property "Footprint" "Resistor_SMD:R_0805_2012Metric_Pad1.20x1.40mm_HandSolder" (at 98.044 122.174 90)
+    (property "Footprint" "Resistor_SMD:R_0603_1608Metric" (at 98.044 122.174 90)
       (effects (font (size 1.27 1.27)) hide)
     )
@@
       (effects (font (size 1.27 1.27)))
     )
-    (property "Footprint" "Resistor_SMD:R_0805_2012Metric_Pad1.20x1.40mm_HandSolder" (at 98.044 133.604 90)
+    (property "Footprint" "Resistor_SMD:R_0603_1608Metric" (at 98.044 133.604 90)
       (effects (font (size 1.27 1.27)) hide)
     )
@@
       (effects (font (size 1.27 1.27)))
     )
-    (property "Footprint" "Resistor_SMD:R_0805_2012Metric_Pad1.20x1.40mm_HandSolder" (at 98.044 143.764 90)
+    (property "Footprint" "Resistor_SMD:R_0603_1608Metric" (at 98.044 143.764 90)
       (effects (font (size 1.27 1.27)) hide)
     )
@@
       (effects (font (size 1.27 1.27)))
     )
-    (property "Footprint" "Resistor_SMD:R_0805_2012Metric_Pad1.20x1.40mm_HandSolder" (at 181.356 82.296 90)
+    (property "Footprint" "Resistor_SMD:R_0603_1608Metric" (at 181.356 82.296 90)
       (effects (font (size 1.27 1.27)) hide)
     )
@@
       (effects (font (size 1.27 1.27)))
     )
-    (property "Footprint" "Resistor_SMD:R_0805_2012Metric_Pad1.20x1.40mm_HandSolder" (at 188.976 82.296 90)
-      (effects (font (size 1.27 1.27)) hide)
-    )
+    (property "Footprint" "Resistor_SMD:R_0603_1608Metric" (at 188.976 82.296 90)
+      (effects (font (size 1.27 1.27)) hide)
+    )

Commit message: finishing schematic 1.0
Parts:
- removed SW12: SW_SP3T, SynthProjConnectors:ST-0-102-A01-T000-LF, symbol Switch:SW_SP3T
- added C61: 22nF, Capacitor_SMD:C_0603_1608Metric, symbol Device:C
- added SW12: SMTS-103-A1-T0, SynthProjConnectors:MTS-103-A01-T0, symbol Switch:SW_SPDT
- RV27: value 10k -> 100k
- SW11: footprint SynthProjConnectors:ST-0-102-A01-T000-LF -> SynthProjConnectors:MTS-103-A01-T0
- SW13: footprint (none) -> SynthProjConnectors:MTS-203-A1-T0
- renumbered C61 to C62, C62 to C63, C63 to C64, C64 to C65, C65 to C66, C66 to C67, C67 to C68
Connections:
- net GNDREF: now also U13.2 (-)
- net at D6.1 (K): now also SW12.1 (A)
- net at D7.2 (A): now also SW12.3 (C)
- net at R123.2, R124.2, R125.2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: now also C61.1
- net at R128.2, R129.2, R130.2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: now also C61.2
- net at SW13.1 (A): now also SW12.2 (B)
Other:
- note added: "Falling"
- note added: "Ramp"
- note added: "Ramp Shape"
- note added: "Ramp/Square Select"
- note added: "Rising"
- note added: "SPDT On-Off-On SMTS-103-A1-T0"
- note added: "Square"
- note added: "Triangle"

Commit message: routing work...
Parts:
- removed U12: TL072, Package_SO:SO-8_3.9x4.9mm_P1.27mm, symbol Amplifier_Operational:TL072
- added unit 3 of U13
Connections:
- net +12V: now also U13.8 (V+)
- net -12V: now also U13.4 (V-)
- net GNDREF: no longer SW11.3 (C)
Other:
- note added: "Hi"
- note added: "Low"
- note added: "Range"
Changed lines of the file:
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@@
-    (stroke (width 0) (type default))
-  )
-  (wire (pts (xy 132.08 124.46) (xy 134.62 124.46))
     (stroke (width 0) (type default))
   )
@@
     (effects (font (size 1.27 1.27)) (justify left bottom))
   )
+  (text "Hi" (at 76.835 123.19 0)
+    (effects (font (size 1.27 1.27)) (justify left bottom))
+  )
   (text "Falling" (at 96.52 61.595 0)
     (effects (font (size 1.27 1.27)) (justify left bottom))
@@
     (effects (font (size 1.27 1.27)) (justify left bottom))
   )
+  (text "Low" (at 76.835 129.54 0)
+    (effects (font (size 1.27 1.27)) (justify left bottom))
+  )
   (text "SPDT On-Off-On \nSMTS-103-A1-T0" (at 123.825 56.515 0)
     (effects (font (size 1.27 1.27)) (justify left bottom))
   )
+  (text "Range" (at 68.58 115.57 0)
+    (effects (font (size 1.27 1.27)) (justify left bottom))
+  )
   (text "Ramp Shape" (at 126.365 49.53 0)
     (effects (font (size 1.27 1.27)) (justify left bottom))
@@
   (hierarchical_label "LFOA" (shape output) (at 219.71 50.8 0) (fields_autoplaced)
     (effects (font (size 1.27 1.27)) (justify left))
-  )
-  (symbol (lib_id "power:+12V") (at 238.76 63.5 0) (unit 1)
-    (in_bom yes) (on_board yes) (dnp no)
-    (property "Reference" "#PWR0171" (at 238.76 67.31 0)
-      (effects (font (size 1.27 1.27)) hide)
-    )
-    (property "Value" "+12V" (at 239.141 59.1058 0)
-      (effects (font (size 1.27 1.27)))
-    )
-    (property "Footprint" "" (at 238.76 63.5 0)
-      (effects (font (size 1.27 1.27)) hide)
-    )
-    (property "Datasheet" "" (at 238.76 63.5 0)
-      (effects (font (size 1.27 1.27)) hide)
-    )
-    (pin "1")
-    (instances
-      (project "SynthProj"
-        (path "/9021c97e-351f-4ed9-b393-50257df6a463/00000000-0000-0000-0000-000066b08086"
-          (reference "#PWR0171") (unit 1)
-        )
-      )
-    )
-  )
-  (symbol (lib_id "power:-12V") (at 238.76 78.74 180) (unit 1)
-    (in_bom yes) (on_board yes) (dnp no)
-    (property "Reference" "#PWR0172" (at 238.76 81.28 0)
-      (effects (font (size 1.27 1.27)) hide)
-    )
-    (property "Value" "-12V" (at 238.379 83.1342 0)
-      (effects (font (size 1.27 1.27)))
-    )
-    (property "Footprint" "" (at 238.76 78.74 0)
-      (effects (font (size 1.27 1.27)) hide)
-    )
-    (property "Datasheet" "" (at 238.76 78.74 0)
-      (effects (font (size 1.27 1.27)) hide)
-    )
-    (pin "1")
-    (instances
-      (project "SynthProj"
-        (path "/9021c97e-351f-4ed9-b393-50257df6a463/00000000-0000-0000-0000-000066b08086"
-          (reference "#PWR0172") (unit 1)
-        )
-      )
-    )
   )
   (symbol (lib_id "power:+12V") (at 254 63.5 0) (unit 1)
@@
     )
   )
-  (symbol (lib_id "Amplifier_Operational:TL072") (at 241.3 71.12 0) (unit 3)
-    (in_bom yes) (on_board yes) (dnp no)
-    (property "Reference" "U12" (at 240.2332 69.9516 0)
-      (effects (font (size 1.27 1.27)) (justify left))
-    )
-    (property "Value" "TL072" (at 240.2332 72.263 0)
-      (effects (font (size 1.27 1.27)) (justify left))
-    )
-    (property "Footprint" "Package_SO:SO-8_3.9x4.9mm_P1.27mm" (at 241.3 71.12 0)
-      (effects (font (size 1.27 1.27)) hide)
-    )
-    (property "Datasheet" "http://www.ti.com/lit/ds/symlink/tl071.pdf" (at 241.3 71.12 0)
-      (effects (font (size 1.27 1.27)) hide)
-    )
-    (pin "2")
-    (pin "5")
-    (pin "1")
-    (pin "6")
-    (pin "3")
-    (pin "8")
-    (pin "7")
-    (pin "4")
-    (instances
-      (project "SynthProj"
-        (path "/9021c97e-351f-4ed9-b393-50257df6a463/00000000-0000-0000-0000-000066b08086"
-          (reference "U12") (unit 3)
-        )
-      )
-    )
-  )
   (symbol (lib_id "power:+12V") (at 128.27 76.2 0) (unit 1)
     (in_bom yes) (on_board yes) (dnp no)
@@
     )
   )
-  (symbol (lib_id "power:GNDREF") (at 76.2 128.27 0) (unit 1)
-    (in_bom yes) (on_board yes) (dnp no)
-    (property "Reference" "#PWR0163" (at 76.2 134.62 0)
-      (effects (font (size 1.27 1.27)) hide)
-    )
-    (property "Value" "GNDREF" (at 76.327 132.6642 0)
-      (effects (font (size 1.27 1.27)))
-    )
-    (property "Footprint" "" (at 76.2 128.27 0)
-      (effects (font (size 1.27 1.27)) hide)
-    )
-    (property "Datasheet" "" (at 76.2 128.27 0)
-      (effects (font (size 1.27 1.27)) hide)
-    )
-    (pin "1")
-    (instances
-      (project "SynthProj"
-        (path "/9021c97e-351f-4ed9-b393-50257df6a463/00000000-0000-0000-0000-000066b08086"
-          (reference "#PWR0163") (unit 1)
-        )
-        (path "/9021c97e-351f-4ed9-b393-50257df6a463/00000000-0000-0000-0000-0000659a4e2e"
-          (reference "#PWR?") (unit 1)
-        )
-      )
-    )
-  )
-  (symbol (lib_id "power:GNDREF") (at 132.08 124.46 0) (unit 1)
-    (in_bom yes) (on_board yes) (dnp no)
-    (property "Reference" "#PWR0167" (at 132.08 130.81 0)
-      (effects (font (size 1.27 1.27)) hide)
-    )
-    (property "Value" "GNDREF" (at 132.207 128.8542 0)
-      (effects (font (size 1.27 1.27)))
-    )
-    (property "Footprint" "" (at 132.08 124.46 0)
-      (effects (font (size 1.27 1.27)) hide)
-    )
-    (property "Datasheet" "" (at 132.08 124.46 0)
+  (symbol (lib_id "power:GNDREF") (at 134.62 124.46 0) (unit 1)
+    (in_bom yes) (on_board yes) (dnp no)
+    (property "Reference" "#PWR0167" (at 134.62 130.81 0)
+      (effects (font (size 1.27 1.27)) hide)
+    )
+    (property "Value" "GNDREF" (at 134.747 128.8542 0)
+      (effects (font (size 1.27 1.27)) hide)
+    )
+    (property "Footprint" "" (at 134.62 124.46 0)
+      (effects (font (size 1.27 1.27)) hide)
+    )
+    (property "Datasheet" "" (at 134.62 124.46 0)
       (effects (font (size 1.27 1.27)) hide)
     )
@@
     )
   )
+  (symbol (lib_id "power:-12V") (at 229.87 78.74 180) (unit 1)
+    (in_bom yes) (on_board yes) (dnp no)
+    (property "Reference" "#PWR0200" (at 229.87 81.28 0)
+      (effects (font (size 1.27 1.27)) hide)
+    )
+    (property "Value" "-12V" (at 229.489 83.1342 0)
+      (effects (font (size 1.27 1.27)))
+    )
+    (property "Footprint" "" (at 229.87 78.74 0)
+      (effects (font (size 1.27 1.27)) hide)
+    )
+    (property "Datasheet" "" (at 229.87 78.74 0)
+      (effects (font (size 1.27 1.27)) hide)
+    )
+    (pin "1")
+    (instances
+      (project "SynthProj"
+        (path "/9021c97e-351f-4ed9-b393-50257df6a463/00000000-0000-0000-0000-00006620617f"
+          (reference "#PWR0200") (unit 1)
+        )
+        (path "/9021c97e-351f-4ed9-b393-50257df6a463/00000000-0000-0000-0000-0000659a4e2e"
+          (reference "#PWR?") (unit 1)
+        )
+        (path "/9021c97e-351f-4ed9-b393-50257df6a463/00000000-0000-0000-0000-000066b08086"
+          (reference "#PWR015") (unit 1)
+        )
+      )
+    )
+  )
+  (symbol (lib_id "Amplifier_Operational:TL072") (at 232.41 71.12 0) (unit 3)
+    (in_bom yes) (on_board yes) (dnp no)
+    (property "Reference" "U13" (at 231.3432 69.9516 0)
+      (effects (font (size 1.27 1.27)) (justify left))
+    )
+    (property "Value" "TL072" (at 231.3432 72.263 0)
+      (effects (font (size 1.27 1.27)) (justify left))
+    )
+    (property "Footprint" "Package_SO:SOP-8_3.9x4.9mm_P1.27mm" (at 232.41 71.12 0)
+      (effects (font (size 1.27 1.27)) hide)
+    )
+    (property "Datasheet" "http://www.ti.com/lit/ds/symlink/tl071.pdf" (at 232.41 71.12 0)
+      (effects (font (size 1.27 1.27)) hide)
+    )
+    (pin "8")
+    (pin "2")
+    (pin "5")
+    (pin "6")
+    (pin "7")
+    (pin "4")
+    (pin "1")
+    (pin "3")
+    (instances
+      (project "SynthProj"
+        (path "/9021c97e-351f-4ed9-b393-50257df6a463/00000000-0000-0000-0000-00006620617f"
+          (reference "U13") (unit 3)
+        )
+        (path "/9021c97e-351f-4ed9-b393-50257df6a463/00000000-0000-0000-0000-0000659a4e2e"
+          (reference "U?") (unit 3)
+        )
+        (path "/9021c97e-351f-4ed9-b393-50257df6a463/00000000-0000-0000-0000-000066b08086"
+          (reference "U13") (unit 3)
+        )
+      )
+    )
+  )
   (symbol (lib_id "Switch:SW_SPDT") (at 133.35 64.77 0) (mirror y) (unit 1)
     (in_bom yes) (on_board yes) (dnp no)
@@
         )
       )
+    )
+  )
+  (symbol (lib_id "power:+12V") (at 229.87 63.5 0) (unit 1)
+    (in_bom yes) (on_board yes) (dnp no)
+    (property "Reference" "#PWR0199" (at 229.87 67.31 0)
+      (effects (font (size 1.27 1.27)) hide)
+    )
+    (property "Value" "+12V" (at 230.251 59.1058 0)
+      (effects (font (size 1.27 1.27)))
+    )
+    (property "Footprint" "" (at 229.87 63.5 0)
+      (effects (font (size 1.27 1.27)) hide)
+    )
+    (property "Datasheet" "" (at 229.87 63.5 0)
+      (effects (font (size 1.27 1.27)) hide)
+    )
+    (pin "1")
+    (instances
+      (project "SynthProj"
+        (path "/9021c97e-351f-4ed9-b393-50257df6a463/00000000-0000-0000-0000-00006620617f"
+          (reference "#PWR0199") (unit 1)
+        )
+        (path "/9021c97e-351f-4ed9-b393-50257df6a463/00000000-0000-0000-0000-0000659a4e2e"
+          (reference "#PWR?") (unit 1)
+        )
+        (path "/9021c97e-351f-4ed9-b393-50257df6a463/00000000-0000-0000-0000-000066b08086"
+          (reference "#PWR05") (unit 1)
+        )
+      )

Commit message: lots of routes, added vco3, lfo2.
Parts:
- SW11, SW12: footprint SynthProjConnectors:MTS-103-A01-T0 -> SynthProjConnectors:SMTS-102
- SW13: footprint SynthProjConnectors:MTS-203-A1-T0 -> SynthProjConnectors:SMTS-202

Commit message: more work
Parts:
- D8: footprint LED_SMD:LED_0805_2012Metric -> LED_THT:LED_D3.0mm
Changed lines of the file:
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@@
       (effects (font (size 1.27 1.27)) (justify right))
     )
-    (property "Footprint" "LED_SMD:LED_0805_2012Metric" (at 128.27 105.41 0)
+    (property "Footprint" "LED_THT:LED_D3.0mm" (at 128.27 105.41 0)
       (effects (font (size 1.27 1.27)) hide)
     )
