File: LFO.kicad_sch (KiCad schematic)
At the start: 29 parts, among them Q14 MMBT3904-7-F, SW11 SW_SPDT, SW12 SMTS-103-A1-T0, SW13 SW_Push_DPDT, U13 TL072

Commit message: more and more and more and more and more routing
Parts:
- removed C63, C64: 4.7uF, Capacitor_SMD:C_0805_2012Metric, symbol Device:C
- removed C67, C68: 47nF, Capacitor_SMD:C_0603_1608Metric, symbol Device:C
Changed lines of the file:
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@@
   (junction (at 194.31 109.22) (diameter 0) (color 0 0 0 0)
   )
-  (junction (at 260.35 63.5) (diameter 0) (color 0 0 0 0)
-  )
   (junction (at 260.35 71.12) (diameter 0) (color 0 0 0 0)
   )
   (junction (at 81.28 110.49) (diameter 0) (color 0 0 0 0)
   )
-  (junction (at 254 71.12) (diameter 0) (color 0 0 0 0)
-  )
   (junction (at 194.31 127) (diameter 0) (color 0 0 0 0)
   )
@@
   (junction (at 214.63 102.87) (diameter 0) (color 0 0 0 0)
   )
-  (junction (at 254 78.74) (diameter 0) (color 0 0 0 0)
-  )
   (junction (at 204.47 43.18) (diameter 0) (color 0 0 0 0)
   )
   (junction (at 177.8 67.31) (diameter 0) (color 0 0 0 0)
   )
-  (junction (at 260.35 78.74) (diameter 0) (color 0 0 0 0)
-  )
   (junction (at 199.39 67.31) (diameter 0) (color 0 0 0 0)
   )
@@
   (junction (at 185.42 81.28) (diameter 0) (color 0 0 0 0)
   )
-  (junction (at 266.7 71.12) (diameter 0) (color 0 0 0 0)
-  )
   (junction (at 132.08 129.54) (diameter 0) (color 0 0 0 0)
   )
-  (junction (at 254 63.5) (diameter 0) (color 0 0 0 0)
-  )
   (junction (at 157.48 116.84) (diameter 0) (color 0 0 0 0)
   )
@@
     (stroke (width 0) (type default))
   )
-  (wire (pts (xy 250.19 71.12) (xy 254 71.12))
+  (wire (pts (xy 250.19 71.12) (xy 260.35 71.12))
     (stroke (width 0) (type default))
   )
@@
     (stroke (width 0) (type default))
   )
-  (wire (pts (xy 260.35 71.12) (xy 266.7 71.12))
-    (stroke (width 0) (type default))
-  )
   (wire (pts (xy 143.51 86.36) (xy 143.51 74.93))
     (stroke (width 0) (type default))
@@
     (stroke (width 0) (type default))
   )
-  (wire (pts (xy 260.35 63.5) (xy 266.7 63.5))
-    (stroke (width 0) (type default))
-  )
   (wire (pts (xy 157.48 127) (xy 162.56 127))
     (stroke (width 0) (type default))
@@
     (stroke (width 0) (type default))
   )
-  (wire (pts (xy 254 71.12) (xy 260.35 71.12))
-    (stroke (width 0) (type default))
-  )
   (wire (pts (xy 157.48 127) (xy 157.48 137.795))
     (stroke (width 0) (type default))
@@
   )
   (wire (pts (xy 162.56 116.84) (xy 157.48 116.84))
-    (stroke (width 0) (type default))
-  )
-  (wire (pts (xy 260.35 78.74) (xy 266.7 78.74))
     (stroke (width 0) (type default))
   )
@@
         (path "/9021c97e-351f-4ed9-b393-50257df6a463/ecb6a5e5-382b-482a-961b-02eec3fee7f6"
           (reference "#PWR0254") (unit 1)
-        )
-      )
-    )
-  )
-  (symbol (lib_id "Device:C") (at 254 67.31 180) (unit 1)
-    (in_bom yes) (on_board yes) (dnp no)
-    (property "Reference" "C63" (at 260.4008 67.31 90)
-      (effects (font (size 1.27 1.27)))
-    )
-    (property "Value" "4.7uF" (at 258.0894 67.31 90)
-      (effects (font (size 1.27 1.27)))
-    )
-    (property "Footprint" "Capacitor_SMD:C_0805_2012Metric" (at 253.0348 63.5 0)
-      (effects (font (size 1.27 1.27)) hide)
-    )
-    (property "Datasheet" "~" (at 254 67.31 0)
-      (effects (font (size 1.27 1.27)) hide)
-    )
-    (pin "1")
-    (pin "2")
-    (instances
-      (project "SynthProj"
-        (path "/9021c97e-351f-4ed9-b393-50257df6a463/00000000-0000-0000-0000-000066b08086"
-          (reference "C63") (unit 1)
-        )
-        (path "/9021c97e-351f-4ed9-b393-50257df6a463/ecb6a5e5-382b-482a-961b-02eec3fee7f6"
-          (reference "C108") (unit 1)
         )
       )
@@
     )
   )
-  (symbol (lib_id "Device:C") (at 266.7 67.31 180) (unit 1)
-    (in_bom yes) (on_board yes) (dnp no)
-    (property "Reference" "C67" (at 273.1008 67.31 90)
-      (effects (font (size 1.27 1.27)))
-    )
-    (property "Value" "47nF" (at 270.7894 67.31 90)
-      (effects (font (size 1.27 1.27)))
-    )
-    (property "Footprint" "Capacitor_SMD:C_0603_1608Metric" (at 265.7348 63.5 0)
-      (effects (font (size 1.27 1.27)) hide)
-    )
-    (property "Datasheet" "~" (at 266.7 67.31 0)
-      (effects (font (size 1.27 1.27)) hide)
-    )
-    (pin "1")
-    (pin "2")
-    (instances
-      (project "SynthProj"
-        (path "/9021c97e-351f-4ed9-b393-50257df6a463/00000000-0000-0000-0000-000066b08086"
-          (reference "C67") (unit 1)
-        )
-        (path "/9021c97e-351f-4ed9-b393-50257df6a463/00000000-0000-0000-0000-0000659a4e2e"
-          (reference "C?") (unit 1)
-        )
-        (path "/9021c97e-351f-4ed9-b393-50257df6a463/ecb6a5e5-382b-482a-961b-02eec3fee7f6"
-          (reference "C112") (unit 1)
-        )
-      )
-    )
-  )
-  (symbol (lib_id "Device:C") (at 254 74.93 180) (unit 1)
-    (in_bom yes) (on_board yes) (dnp no)
-    (property "Reference" "C64" (at 260.4008 74.93 90)
-      (effects (font (size 1.27 1.27)))
-    )
-    (property "Value" "4.7uF" (at 258.0894 74.93 90)
-      (effects (font (size 1.27 1.27)))
-    )
-    (property "Footprint" "Capacitor_SMD:C_0805_2012Metric" (at 253.0348 71.12 0)
-      (effects (font (size 1.27 1.27)) hide)
-    )
-    (property "Datasheet" "~" (at 254 74.93 0)
-      (effects (font (size 1.27 1.27)) hide)
-    )
-    (pin "1")
-    (pin "2")
-    (instances
-      (project "SynthProj"
-        (path "/9021c97e-351f-4ed9-b393-50257df6a463/00000000-0000-0000-0000-000066b08086"
-          (reference "C64") (unit 1)
-        )
-        (path "/9021c97e-351f-4ed9-b393-50257df6a463/ecb6a5e5-382b-482a-961b-02eec3fee7f6"
-          (reference "C109") (unit 1)
-        )
-      )
-    )
-  )
   (symbol (lib_id "Device:C") (at 260.35 74.93 180) (unit 1)
     (in_bom yes) (on_board yes) (dnp no)
@@
         )
       )
-    )
-  )
-  (symbol (lib_id "Device:C") (at 266.7 74.93 180) (unit 1)
-    (in_bom yes) (on_board yes) (dnp no)
-    (property "Reference" "C68" (at 273.1008 74.93 90)
-      (effects (font (size 1.27 1.27)))
-    )
-    (property "Value" "47nF" (at 270.7894 74.93 90)
-      (effects (font (size 1.27 1.27)))
-    )
-    (property "Footprint" "Capacitor_SMD:C_0603_1608Metric" (at 265.7348 71.12 0)
-      (effects (font (size 1.27 1.27)) hide)
-    )
-    (property "Datasheet" "~" (at 266.7 74.93 0)
-      (effects (font (size 1.27 1.27)) hide)
-    )
-    (pin "1")
-    (pin "2")
-    (instances
-      (project "SynthProj"
-        (path "/9021c97e-351f-4ed9-b393-50257df6a463/00000000-0000-0000-0000-000066b08086"
-          (reference "C68") (unit 1)
-        )
-        (path "/9021c97e-351f-4ed9-b393-50257df6a463/ecb6a5e5-382b-482a-961b-02eec3fee7f6"
-          (reference "C113") (unit 1)
-        )
-      )

Commit message: created manufacturing files
Parts:
- RV26: value 10k -> 50k
- RV27: value 100k -> 50k
Changed lines of the file:
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@@
       (effects (font (size 1.27 1.27)))
     )
-    (property "Value" "10k" (at 49.4284 134.62 90)
+    (property "Value" "50k" (at 49.4284 134.62 90)
       (effects (font (size 1.27 1.27)))
     )
@@
       (effects (font (size 1.27 1.27)))
     )
-    (property "Value" "100k" (at 200.5584 50.8 90)
+    (property "Value" "50k" (at 200.5584 50.8 90)
       (effects (font (size 1.27 1.27)))
     )
