File: Mixer.kicad_sch (KiCad schematic)
At the start: 23 parts, among them J33 Noise Out, SW10 SW_SPDT, SW9 SW_SPDT, U11 TL071

Commit message: more work...
Parts:
- C39, C40, C41, C42, C47, C48: footprint Capacitor_SMD:C_0805_2012Metric_Pad1.18x1.45mm_HandSolder -> Capacitor_SMD:C_0805_2012Metric
- C43, C44, C45, C46: footprint Capacitor_SMD:C_0805_2012Metric_Pad1.18x1.45mm_HandSolder -> Capacitor_SMD:C_0603_1608Metric
- R111, R112, R113, R114, R115: footprint Resistor_SMD:R_0805_2012Metric_Pad1.20x1.40mm_HandSolder -> Resistor_SMD:R_0603_1608Metric
Changed lines of the file:
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@@
       (effects (font (size 1.27 1.27)) (justify left))
     )
-    (property "Footprint" "Capacitor_SMD:C_0805_2012Metric_Pad1.18x1.45mm_HandSolder" (at 149.86 70.8152 0)
+    (property "Footprint" "Capacitor_SMD:C_0603_1608Metric" (at 149.86 70.8152 0)
       (effects (font (size 1.27 1.27)) hide)
     )
@@
       (effects (font (size 1.27 1.27)))
     )
-    (property "Footprint" "Resistor_SMD:R_0805_2012Metric_Pad1.20x1.40mm_HandSolder" (at 161.036 70.866 90)
+    (property "Footprint" "Resistor_SMD:R_0603_1608Metric" (at 161.036 70.866 90)
       (effects (font (size 1.27 1.27)) hide)
     )
@@
       (effects (font (size 1.27 1.27)) (justify left))
     )
-    (property "Footprint" "Capacitor_SMD:C_0805_2012Metric_Pad1.18x1.45mm_HandSolder" (at 149.86 89.8652 0)
+    (property "Footprint" "Capacitor_SMD:C_0603_1608Metric" (at 149.86 89.8652 0)
       (effects (font (size 1.27 1.27)) hide)
     )
@@
       (effects (font (size 1.27 1.27)))
     )
-    (property "Footprint" "Resistor_SMD:R_0805_2012Metric_Pad1.20x1.40mm_HandSolder" (at 161.036 89.916 90)
+    (property "Footprint" "Resistor_SMD:R_0603_1608Metric" (at 161.036 89.916 90)
       (effects (font (size 1.27 1.27)) hide)
     )
@@
       (effects (font (size 1.27 1.27)) (justify left))
     )
-    (property "Footprint" "Capacitor_SMD:C_0805_2012Metric_Pad1.18x1.45mm_HandSolder" (at 149.86 110.1852 0)
+    (property "Footprint" "Capacitor_SMD:C_0805_2012Metric" (at 149.86 110.1852 0)
       (effects (font (size 1.27 1.27)) hide)
     )
@@
       (effects (font (size 1.27 1.27)))
     )
-    (property "Footprint" "Resistor_SMD:R_0805_2012Metric_Pad1.20x1.40mm_HandSolder" (at 161.036 110.236 90)
+    (property "Footprint" "Resistor_SMD:R_0603_1608Metric" (at 161.036 110.236 90)
       (effects (font (size 1.27 1.27)) hide)
     )
@@
       (effects (font (size 1.27 1.27)) (justify left))
     )
-    (property "Footprint" "Capacitor_SMD:C_0805_2012Metric_Pad1.18x1.45mm_HandSolder" (at 149.86 129.2352 0)
+    (property "Footprint" "Capacitor_SMD:C_0805_2012Metric" (at 149.86 129.2352 0)
       (effects (font (size 1.27 1.27)) hide)
     )
@@
       (effects (font (size 1.27 1.27)))
     )
-    (property "Footprint" "Resistor_SMD:R_0805_2012Metric_Pad1.20x1.40mm_HandSolder" (at 161.036 129.286 90)
+    (property "Footprint" "Resistor_SMD:R_0603_1608Metric" (at 161.036 129.286 90)
       (effects (font (size 1.27 1.27)) hide)
     )
@@
       (effects (font (size 1.27 1.27)))
     )
-    (property "Footprint" "Resistor_SMD:R_0805_2012Metric_Pad1.20x1.40mm_HandSolder" (at 188.976 89.916 90)
+    (property "Footprint" "Resistor_SMD:R_0603_1608Metric" (at 188.976 89.916 90)
       (effects (font (size 1.27 1.27)) hide)
     )
@@
       (effects (font (size 1.27 1.27)))
     )
-    (property "Footprint" "Capacitor_SMD:C_0805_2012Metric_Pad1.18x1.45mm_HandSolder" (at 85.3948 148.59 0)
+    (property "Footprint" "Capacitor_SMD:C_0805_2012Metric" (at 85.3948 148.59 0)
       (effects (font (size 1.27 1.27)) hide)
     )
@@
       (effects (font (size 1.27 1.27)))
     )
-    (property "Footprint" "Capacitor_SMD:C_0805_2012Metric_Pad1.18x1.45mm_HandSolder" (at 91.7448 148.59 0)
+    (property "Footprint" "Capacitor_SMD:C_0805_2012Metric" (at 91.7448 148.59 0)
       (effects (font (size 1.27 1.27)) hide)
     )
@@
       (effects (font (size 1.27 1.27)))
     )
-    (property "Footprint" "Capacitor_SMD:C_0805_2012Metric_Pad1.18x1.45mm_HandSolder" (at 98.0948 148.59 0)
+    (property "Footprint" "Capacitor_SMD:C_0603_1608Metric" (at 98.0948 148.59 0)
       (effects (font (size 1.27 1.27)) hide)
     )
@@
       (effects (font (size 1.27 1.27)))
     )
-    (property "Footprint" "Capacitor_SMD:C_0805_2012Metric_Pad1.18x1.45mm_HandSolder" (at 85.3948 156.21 0)
+    (property "Footprint" "Capacitor_SMD:C_0805_2012Metric" (at 85.3948 156.21 0)
       (effects (font (size 1.27 1.27)) hide)
     )
@@
       (effects (font (size 1.27 1.27)))
     )
-    (property "Footprint" "Capacitor_SMD:C_0805_2012Metric_Pad1.18x1.45mm_HandSolder" (at 91.7448 156.21 0)
+    (property "Footprint" "Capacitor_SMD:C_0805_2012Metric" (at 91.7448 156.21 0)
       (effects (font (size 1.27 1.27)) hide)
     )
@@
       (effects (font (size 1.27 1.27)))
     )
-    (property "Footprint" "Capacitor_SMD:C_0805_2012Metric_Pad1.18x1.45mm_HandSolder" (at 98.0948 156.21 0)
-      (effects (font (size 1.27 1.27)) hide)
-    )
+    (property "Footprint" "Capacitor_SMD:C_0603_1608Metric" (at 98.0948 156.21 0)
+      (effects (font (size 1.27 1.27)) hide)
+    )

Commit message: finishing schematic 1.0
Parts:
- SW10, SW9: footprint SynthProjConnectors:ST-0-102-A01-T000-LF -> SynthProjConnectors:MTS-103-A01-T0
- renumbered J33 to J39
Changed lines of the file:
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@@
       (effects (font (size 1.27 1.27)))
     )
-    (property "Footprint" "SynthProjConnectors:ST-0-102-A01-T000-LF" (at 111.76 66.04 0)
+    (property "Footprint" "SynthProjConnectors:MTS-103-A01-T0" (at 111.76 66.04 0)
       (effects (font (size 1.27 1.27)) hide)
     )
@@
   (symbol (lib_id "power:GNDREF") (at 179.07 64.77 0) (unit 1)
     (in_bom yes) (on_board yes) (dnp no)
-    (property "Reference" "#PWR0143" (at 179.07 71.12 0)
+    (property "Reference" "#PWR0149" (at 179.07 71.12 0)
       (effects (font (size 1.27 1.27)) hide)
     )
@@
       (project "SynthProj"
         (path "/9021c97e-351f-4ed9-b393-50257df6a463/00000000-0000-0000-0000-00006611e0f5"
-          (reference "#PWR0143") (unit 1)
+          (reference "#PWR0149") (unit 1)
         )
       )
@@
   (symbol (lib_id "power:GNDREF") (at 128.27 73.66 0) (unit 1)
     (in_bom yes) (on_board yes) (dnp no)
-    (property "Reference" "#PWR0139" (at 128.27 80.01 0)
+    (property "Reference" "#PWR0145" (at 128.27 80.01 0)
       (effects (font (size 1.27 1.27)) hide)
     )
@@
       (project "SynthProj"
         (path "/9021c97e-351f-4ed9-b393-50257df6a463/00000000-0000-0000-0000-00006611e0f5"
-          (reference "#PWR0139") (unit 1)
+          (reference "#PWR0145") (unit 1)
         )
       )
@@
       (effects (font (size 1.27 1.27)))
     )
-    (property "Footprint" "SynthProjConnectors:ST-0-102-A01-T000-LF" (at 111.76 85.09 0)
+    (property "Footprint" "SynthProjConnectors:MTS-103-A01-T0" (at 111.76 85.09 0)
       (effects (font (size 1.27 1.27)) hide)
     )
@@
   (symbol (lib_id "power:GNDREF") (at 128.27 95.25 0) (unit 1)
     (in_bom yes) (on_board yes) (dnp no)
-    (property "Reference" "#PWR0140" (at 128.27 101.6 0)
+    (property "Reference" "#PWR0146" (at 128.27 101.6 0)
       (effects (font (size 1.27 1.27)) hide)
     )
@@
       (project "SynthProj"
         (path "/9021c97e-351f-4ed9-b393-50257df6a463/00000000-0000-0000-0000-00006611e0f5"
-          (reference "#PWR0140") (unit 1)
+          (reference "#PWR0146") (unit 1)
         )
       )
@@
   (symbol (lib_id "power:GNDREF") (at 128.27 113.03 0) (unit 1)
     (in_bom yes) (on_board yes) (dnp no)
-    (property "Reference" "#PWR0141" (at 128.27 119.38 0)
+    (property "Reference" "#PWR0147" (at 128.27 119.38 0)
       (effects (font (size 1.27 1.27)) hide)
     )
@@
       (project "SynthProj"
         (path "/9021c97e-351f-4ed9-b393-50257df6a463/00000000-0000-0000-0000-00006611e0f5"
-          (reference "#PWR0141") (unit 1)
+          (reference "#PWR0147") (unit 1)
         )
       )
@@
   (symbol (lib_id "power:GNDREF") (at 128.27 132.08 0) (unit 1)
     (in_bom yes) (on_board yes) (dnp no)
-    (property "Reference" "#PWR0142" (at 128.27 138.43 0)
+    (property "Reference" "#PWR0148" (at 128.27 138.43 0)
       (effects (font (size 1.27 1.27)) hide)
     )
@@
       (project "SynthProj"
         (path "/9021c97e-351f-4ed9-b393-50257df6a463/00000000-0000-0000-0000-00006611e0f5"
-          (reference "#PWR0142") (unit 1)
+          (reference "#PWR0148") (unit 1)
         )
       )
@@
   (symbol (lib_id "power:+12V") (at 184.15 59.69 0) (unit 1)
     (in_bom yes) (on_board yes) (dnp no)
-    (property "Reference" "#PWR0144" (at 184.15 63.5 0)
+    (property "Reference" "#PWR0150" (at 184.15 63.5 0)
       (effects (font (size 1.27 1.27)) hide)
     )
@@
       (project "SynthProj"
         (path "/9021c97e-351f-4ed9-b393-50257df6a463/00000000-0000-0000-0000-00006611e0f5"
-          (reference "#PWR0144") (unit 1)
+          (reference "#PWR0150") (unit 1)
         )
       )
@@
   (symbol (lib_id "power:-12V") (at 184.15 74.93 180) (unit 1)
     (in_bom yes) (on_board yes) (dnp no)
-    (property "Reference" "#PWR0145" (at 184.15 77.47 0)
+    (property "Reference" "#PWR0151" (at 184.15 77.47 0)
       (effects (font (size 1.27 1.27)) hide)
     )
@@
       (project "SynthProj"
         (path "/9021c97e-351f-4ed9-b393-50257df6a463/00000000-0000-0000-0000-00006611e0f5"
-          (reference "#PWR0145") (unit 1)
+          (reference "#PWR0151") (unit 1)
         )
       )
@@
   (symbol (lib_id "SynthProj-rescue:AudioJack2-Connector") (at 102.87 99.06 0) (unit 1)
     (in_bom yes) (on_board yes) (dnp no)
-    (property "Reference" "J33" (at 103.6828 90.805 0)
+    (property "Reference" "J39" (at 103.6828 90.805 0)
       (effects (font (size 1.27 1.27)))
     )
@@
       (project "SynthProj"
         (path "/9021c97e-351f-4ed9-b393-50257df6a463/00000000-0000-0000-0000-00006611e0f5"
-          (reference "J33") (unit 1)
+          (reference "J39") (unit 1)
         )
         (path "/9021c97e-351f-4ed9-b393-50257df6a463/00000000-0000-0000-0000-0000659a4e2e"
@@
   (symbol (lib_id "power:GNDREF") (at 107.95 96.52 90) (unit 1)
     (in_bom yes) (on_board yes) (dnp no)
-    (property "Reference" "#PWR0138" (at 114.3 96.52 0)
+    (property "Reference" "#PWR0144" (at 114.3 96.52 0)
       (effects (font (size 1.27 1.27)) hide)
     )
@@
       (project "SynthProj"
         (path "/9021c97e-351f-4ed9-b393-50257df6a463/00000000-0000-0000-0000-00006611e0f5"
-          (reference "#PWR0138") (unit 1)
+          (reference "#PWR0144") (unit 1)
         )
         (path "/9021c97e-351f-4ed9-b393-50257df6a463/00000000-0000-0000-0000-0000659a4e2e"
@@
   (symbol (lib_id "power:+12V") (at 86.36 148.59 0) (unit 1)
     (in_bom yes) (on_board yes) (dnp no)
-    (property "Reference" "#PWR0136" (at 86.36 152.4 0)
+    (property "Reference" "#PWR0142" (at 86.36 152.4 0)
       (effects (font (size 1.27 1.27)) hide)
     )
@@
       (project "SynthProj"
         (path "/9021c97e-351f-4ed9-b393-50257df6a463/00000000-0000-0000-0000-00006611e0f5"
-          (reference "#PWR0136") (unit 1)
+          (reference "#PWR0142") (unit 1)
         )
       )
@@
   (symbol (lib_id "power:-12V") (at 86.36 163.83 180) (unit 1)
     (in_bom yes) (on_board yes) (dnp no)
-    (property "Reference" "#PWR0137" (at 86.36 166.37 0)
+    (property "Reference" "#PWR0143" (at 86.36 166.37 0)
       (effects (font (size 1.27 1.27)) hide)
     )
@@
       (project "SynthProj"
         (path "/9021c97e-351f-4ed9-b393-50257df6a463/00000000-0000-0000-0000-00006611e0f5"
-          (reference "#PWR0137") (unit 1)
+          (reference "#PWR0143") (unit 1)
         )
       )
@@
   (symbol (lib_id "power:GNDREF") (at 82.55 156.21 270) (unit 1)
     (in_bom yes) (on_board yes) (dnp no)
-    (property "Reference" "#PWR0135" (at 76.2 156.21 0)
+    (property "Reference" "#PWR0141" (at 76.2 156.21 0)
       (effects (font (size 1.27 1.27)) hide)
     )
@@
       (project "SynthProj"
         (path "/9021c97e-351f-4ed9-b393-50257df6a463/00000000-0000-0000-0000-00006611e0f5"
-          (reference "#PWR0135") (unit 1)
-        )
-      )
+          (reference "#PWR0141") (unit 1)
+        )
+      )

Commit message: Doing some layout
Parts:
- J39: footprint SynthProjConnectors:JINJIA CK3.5-98-LF -> SynthProjConnectors:PJ-358
Other:
- note added: "Ramp"
- note added: "Square"
Changed lines of the file:
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@@
     (stroke (width 0) (type default))
   )
+  (text "Ramp" (at 100.33 87.63 0)
+    (effects (font (size 1.27 1.27)) (justify left bottom))
+  )
   (text "To VCF" (at 210.82 64.77 0)
     (effects (font (size 1.27 1.27)) (justify left bottom))
   )
   (text "From VCO1" (at 81.28 62.23 0)
+    (effects (font (size 1.27 1.27)) (justify left bottom))
+  )
+  (text "Ramp" (at 100.965 68.58 0)
+    (effects (font (size 1.27 1.27)) (justify left bottom))
+  )
+  (text "Square" (at 100.33 82.55 0)
+    (effects (font (size 1.27 1.27)) (justify left bottom))
+  )
+  (text "Square" (at 100.965 63.5 0)
     (effects (font (size 1.27 1.27)) (justify left bottom))
   )
@@
       (effects (font (size 1.27 1.27)))
     )
-    (property "Footprint" "SynthProjConnectors:JINJIA CK3.5-98-LF" (at 102.87 99.06 0)
-      (effects (font (size 1.27 1.27)) hide)
-    )
+    (property "Footprint" "SynthProjConnectors:PJ-358" (at 102.87 99.06 0)
+      (effects (font (size 1.27 1.27)) hide)
+    )

Commit message: doing some routing - split sequencer into another project
Parts:
- J39: footprint SynthProjConnectors:PJ-358 -> SynthProjConnectors:PJ-301
Changed lines of the file:
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@@
       (effects (font (size 1.27 1.27)))
     )
-    (property "Footprint" "SynthProjConnectors:PJ-358" (at 102.87 99.06 0)
+    (property "Footprint" "SynthProjConnectors:PJ-301" (at 102.87 99.06 0)
       (effects (font (size 1.27 1.27)) hide)
     )

Commit message: work
Parts:
- added C93: 100nF, Capacitor_SMD:C_0603_1608Metric, symbol Device:C
- added R176: 470k, Resistor_SMD:R_0603_1608Metric, symbol Device:R_US
Connections:
- net at R111.1, R112.1, R113.1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: now also R176.1
- new net: C93.1, R176.2
- new net Mixer_EchoIn: C93.2
Changed lines of the file:
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@@
   (junction (at 201.93 67.31) (diameter 0) (color 0 0 0 0)
   )
+  (junction (at 172.72 128.27) (diameter 0) (color 0 0 0 0)
+  )
   (junction (at 86.36 156.21) (diameter 0) (color 0 0 0 0)
   )
@@
     (stroke (width 0) (type default))
   )
+  (wire (pts (xy 172.72 146.05) (xy 172.72 128.27))
+    (stroke (width 0) (type default))
+  )
   (wire (pts (xy 106.68 82.55) (xy 93.98 82.55))
     (stroke (width 0) (type default))
@@
     (stroke (width 0) (type default))
   )
+  (wire (pts (xy 165.735 146.05) (xy 172.72 146.05))
+    (stroke (width 0) (type default))
+  )
   (wire (pts (xy 106.68 63.5) (xy 93.98 63.5))
     (stroke (width 0) (type default))
@@
   )
   (wire (pts (xy 128.27 102.87) (xy 128.27 105.41))
+    (stroke (width 0) (type default))
+  )
+  (wire (pts (xy 123.19 146.05) (xy 150.495 146.05))
     (stroke (width 0) (type default))
   )
@@
     )
   )
+  (hierarchical_label "Mixer_EchoIn" (shape input) (at 123.19 146.05 180) (fields_autoplaced)
+    (effects (font (size 1.27 1.27)) (justify right))
+  )
   (hierarchical_label "X38" (shape input) (at 93.98 102.87 180) (fields_autoplaced)
     (effects (font (size 1.27 1.27)) (justify right))
@@
         )
       )
+    )
+  )
+  (symbol (lib_id "Device:C") (at 154.305 146.05 270) (unit 1)
+    (in_bom yes) (on_board yes) (dnp no)
+    (property "Reference" "C93" (at 155.4734 148.971 0)
+      (effects (font (size 1.27 1.27)) (justify left))
+    )
+    (property "Value" "100nF" (at 153.162 148.971 0)
+      (effects (font (size 1.27 1.27)) (justify left))
+    )
+    (property "Footprint" "Capacitor_SMD:C_0603_1608Metric" (at 150.495 147.0152 0)
+      (effects (font (size 1.27 1.27)) hide)
+    )
+    (property "Datasheet" "~" (at 154.305 146.05 0)
+      (effects (font (size 1.27 1.27)) hide)
+    )
+    (pin "2")
+    (pin "1")
+    (instances
+      (project "SynthProj"
+        (path "/9021c97e-351f-4ed9-b393-50257df6a463/00000000-0000-0000-0000-00006611e0f5"
+          (reference "C93") (unit 1)
+        )
+        (path "/9021c97e-351f-4ed9-b393-50257df6a463/00000000-0000-0000-0000-0000659a4e2e"
+          (reference "C?") (unit 1)
+        )
+      )
+    )
+  )
+  (symbol (lib_id "Device:R_US") (at 161.925 146.05 270) (unit 1)
+    (in_bom yes) (on_board yes) (dnp no)
+    (property "Reference" "R176" (at 161.925 140.843 90)
+      (effects (font (size 1.27 1.27)))
+    )
+    (property "Value" "470k" (at 161.925 143.1544 90)
+      (effects (font (size 1.27 1.27)))
+    )
+    (property "Footprint" "Resistor_SMD:R_0603_1608Metric" (at 161.671 147.066 90)
+      (effects (font (size 1.27 1.27)) hide)
+    )
+    (property "Datasheet" "~" (at 161.925 146.05 0)
+      (effects (font (size 1.27 1.27)) hide)
+    )
+    (pin "2")
+    (pin "1")
+    (instances
+      (project "SynthProj"
+        (path "/9021c97e-351f-4ed9-b393-50257df6a463/00000000-0000-0000-0000-00006611e0f5"
+          (reference "R176") (unit 1)
+        )
+        (path "/9021c97e-351f-4ed9-b393-50257df6a463/00000000-0000-0000-0000-0000659a4e2e"
+          (reference "R?") (unit 1)
+        )
+      )
