File: Sample&Hold.kicad_sch (KiCad schematic)
At the start: 31 parts, among them U16 TL064

Commit message: more work...
Parts:
- C84, C85, C86, C87, C88: footprint Capacitor_SMD:C_0805_2012Metric_Pad1.18x1.45mm_HandSolder -> Capacitor_SMD:C_0805_2012Metric
- C89, C90, C91: footprint Capacitor_SMD:C_0805_2012Metric_Pad1.18x1.45mm_HandSolder -> Capacitor_SMD:C_0603_1608Metric
- R162, R163, R164, R165, R166, R167, R168, R169, R170, R171, R172, R173, R174, R175: footprint Resistor_SMD:R_0805_2012Metric_Pad1.20x1.40mm_HandSolder -> Resistor_SMD:R_0603_1608Metric
Changed lines of the file:
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@@
       (effects (font (size 1.27 1.27)))
     )
-    (property "Footprint" "Capacitor_SMD:C_0805_2012Metric_Pad1.18x1.45mm_HandSolder" (at 71.4248 138.43 0)
+    (property "Footprint" "Capacitor_SMD:C_0805_2012Metric" (at 71.4248 138.43 0)
       (effects (font (size 1.27 1.27)) hide)
     )
@@
       (effects (font (size 1.27 1.27)))
     )
-    (property "Footprint" "Capacitor_SMD:C_0805_2012Metric_Pad1.18x1.45mm_HandSolder" (at 77.7748 138.43 0)
+    (property "Footprint" "Capacitor_SMD:C_0805_2012Metric" (at 77.7748 138.43 0)
       (effects (font (size 1.27 1.27)) hide)
     )
@@
       (effects (font (size 1.27 1.27)))
     )
-    (property "Footprint" "Capacitor_SMD:C_0805_2012Metric_Pad1.18x1.45mm_HandSolder" (at 71.4248 146.05 0)
+    (property "Footprint" "Capacitor_SMD:C_0805_2012Metric" (at 71.4248 146.05 0)
       (effects (font (size 1.27 1.27)) hide)
     )
@@
       (effects (font (size 1.27 1.27)))
     )
-    (property "Footprint" "Capacitor_SMD:C_0805_2012Metric_Pad1.18x1.45mm_HandSolder" (at 77.7748 146.05 0)
+    (property "Footprint" "Capacitor_SMD:C_0805_2012Metric" (at 77.7748 146.05 0)
       (effects (font (size 1.27 1.27)) hide)
     )
@@
       (effects (font (size 1.27 1.27)))
     )
-    (property "Footprint" "Resistor_SMD:R_0805_2012Metric_Pad1.20x1.40mm_HandSolder" (at 87.376 60.706 90)
+    (property "Footprint" "Resistor_SMD:R_0603_1608Metric" (at 87.376 60.706 90)
       (effects (font (size 1.27 1.27)) hide)
     )
@@
       (effects (font (size 1.27 1.27)))
     )
-    (property "Footprint" "Resistor_SMD:R_0805_2012Metric_Pad1.20x1.40mm_HandSolder" (at 94.234 63.246 90)
+    (property "Footprint" "Resistor_SMD:R_0603_1608Metric" (at 94.234 63.246 90)
       (effects (font (size 1.27 1.27)) hide)
     )
@@
       (effects (font (size 1.27 1.27)))
     )
-    (property "Footprint" "Resistor_SMD:R_0805_2012Metric_Pad1.20x1.40mm_HandSolder" (at 115.316 74.676 90)
+    (property "Footprint" "Resistor_SMD:R_0603_1608Metric" (at 115.316 74.676 90)
       (effects (font (size 1.27 1.27)) hide)
     )
@@
       (effects (font (size 1.27 1.27)))
     )
-    (property "Footprint" "Resistor_SMD:R_0805_2012Metric_Pad1.20x1.40mm_HandSolder" (at 91.186 84.836 90)
+    (property "Footprint" "Resistor_SMD:R_0603_1608Metric" (at 91.186 84.836 90)
       (effects (font (size 1.27 1.27)) hide)
     )
@@
       (effects (font (size 1.27 1.27)))
     )
-    (property "Footprint" "Resistor_SMD:R_0805_2012Metric_Pad1.20x1.40mm_HandSolder" (at 144.526 74.676 90)
+    (property "Footprint" "Resistor_SMD:R_0603_1608Metric" (at 144.526 74.676 90)
       (effects (font (size 1.27 1.27)) hide)
     )
@@
       (effects (font (size 1.27 1.27)))
     )
-    (property "Footprint" "Resistor_SMD:R_0805_2012Metric_Pad1.20x1.40mm_HandSolder" (at 151.384 81.026 90)
+    (property "Footprint" "Resistor_SMD:R_0603_1608Metric" (at 151.384 81.026 90)
       (effects (font (size 1.27 1.27)) hide)
     )
@@
       (effects (font (size 1.27 1.27)))
     )
-    (property "Footprint" "Capacitor_SMD:C_0805_2012Metric_Pad1.18x1.45mm_HandSolder" (at 128.27 104.4448 0)
+    (property "Footprint" "Capacitor_SMD:C_0603_1608Metric" (at 128.27 104.4448 0)
       (effects (font (size 1.27 1.27)) hide)
     )
@@
       (effects (font (size 1.27 1.27)))
     )
-    (property "Footprint" "Resistor_SMD:R_0805_2012Metric_Pad1.20x1.40mm_HandSolder" (at 133.604 112.776 90)
+    (property "Footprint" "Resistor_SMD:R_0603_1608Metric" (at 133.604 112.776 90)
       (effects (font (size 1.27 1.27)) hide)
     )
@@
       (effects (font (size 1.27 1.27)))
     )
-    (property "Footprint" "Resistor_SMD:R_0805_2012Metric_Pad1.20x1.40mm_HandSolder" (at 97.536 93.726 90)
+    (property "Footprint" "Resistor_SMD:R_0603_1608Metric" (at 97.536 93.726 90)
       (effects (font (size 1.27 1.27)) hide)
     )
@@
       (effects (font (size 1.27 1.27)))
     )
-    (property "Footprint" "Resistor_SMD:R_0805_2012Metric_Pad1.20x1.40mm_HandSolder" (at 75.946 93.726 90)
+    (property "Footprint" "Resistor_SMD:R_0603_1608Metric" (at 75.946 93.726 90)
       (effects (font (size 1.27 1.27)) hide)
     )
@@
       (effects (font (size 1.27 1.27)))
     )
-    (property "Footprint" "Capacitor_SMD:C_0805_2012Metric_Pad1.18x1.45mm_HandSolder" (at 86.36 106.9848 0)
+    (property "Footprint" "Capacitor_SMD:C_0805_2012Metric" (at 86.36 106.9848 0)
       (effects (font (size 1.27 1.27)) hide)
     )
@@
       (effects (font (size 1.27 1.27)))
     )
-    (property "Footprint" "Resistor_SMD:R_0805_2012Metric_Pad1.20x1.40mm_HandSolder" (at 97.536 119.126 90)
+    (property "Footprint" "Resistor_SMD:R_0603_1608Metric" (at 97.536 119.126 90)
       (effects (font (size 1.27 1.27)) hide)
     )
@@
       (effects (font (size 1.27 1.27)))
     )
-    (property "Footprint" "Capacitor_SMD:C_0805_2012Metric_Pad1.18x1.45mm_HandSolder" (at 164.1348 64.77 0)
+    (property "Footprint" "Capacitor_SMD:C_0603_1608Metric" (at 164.1348 64.77 0)
       (effects (font (size 1.27 1.27)) hide)
     )
@@
       (effects (font (size 1.27 1.27)))
     )
-    (property "Footprint" "Resistor_SMD:R_0805_2012Metric_Pad1.20x1.40mm_HandSolder" (at 188.976 51.816 90)
+    (property "Footprint" "Resistor_SMD:R_0603_1608Metric" (at 188.976 51.816 90)
       (effects (font (size 1.27 1.27)) hide)
     )
@@
       (effects (font (size 1.27 1.27)))
     )
-    (property "Footprint" "Resistor_SMD:R_0805_2012Metric_Pad1.20x1.40mm_HandSolder" (at 190.246 77.216 90)
+    (property "Footprint" "Resistor_SMD:R_0603_1608Metric" (at 190.246 77.216 90)
       (effects (font (size 1.27 1.27)) hide)
     )
@@
       (effects (font (size 1.27 1.27)))
     )
-    (property "Footprint" "Resistor_SMD:R_0805_2012Metric_Pad1.20x1.40mm_HandSolder" (at 197.866 101.346 90)
+    (property "Footprint" "Resistor_SMD:R_0603_1608Metric" (at 197.866 101.346 90)
       (effects (font (size 1.27 1.27)) hide)
     )
@@
       (effects (font (size 1.27 1.27)))
     )
-    (property "Footprint" "Capacitor_SMD:C_0805_2012Metric_Pad1.18x1.45mm_HandSolder" (at 204.1652 109.22 0)
+    (property "Footprint" "Capacitor_SMD:C_0603_1608Metric" (at 204.1652 109.22 0)
       (effects (font (size 1.27 1.27)) hide)
     )
@@
       (effects (font (size 1.27 1.27)))
     )
-    (property "Footprint" "Resistor_SMD:R_0805_2012Metric_Pad1.20x1.40mm_HandSolder" (at 117.094 135.636 90)
-      (effects (font (size 1.27 1.27)) hide)
-    )
+    (property "Footprint" "Resistor_SMD:R_0603_1608Metric" (at 117.094 135.636 90)
+      (effects (font (size 1.27 1.27)) hide)
+    )

Commit message: finishing schematic 1.0
Parts:
- renumbered C84 to C85, C85 to C86, C86 to C87, C87 to C88, C88 to C89, C89 to C90, C90 to C91, C91 to C92

Commit message: Doing some layout
Parts:
- RV39: footprint Potentiometer_THT:Potentiometer_Alps_RK09K_Single_Vertical -> Potentiometer_SMD:Potentiometer_Bourns_TC33X_Vertical
Other:
- note added: "Sample Rate"
Changed lines of the file:
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@@
+    (effects (font (size 1.27 1.27)) (justify left bottom))
+  )
+  (text "Sample Rate" (at 104.775 129.54 0)
     (effects (font (size 1.27 1.27)) (justify left bottom))
   )
@@
       (effects (font (size 1.27 1.27)) (justify right))
     )
-    (property "Footprint" "Potentiometer_THT:Potentiometer_Alps_RK09K_Single_Vertical" (at 205.74 50.8 0)
-      (effects (font (size 1.27 1.27)) hide)
-    )
+    (property "Footprint" "Potentiometer_SMD:Potentiometer_Bourns_TC33X_Vertical" (at 205.74 50.8 0)
+      (effects (font (size 1.27 1.27)) hide)
+    )

Commit message: more work
Parts:
- D32: footprint LED_SMD:LED_0805_2012Metric -> LED_THT:LED_D3.0mm
Changed lines of the file:
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@@
       (effects (font (size 1.27 1.27)) (justify right))
     )
-    (property "Footprint" "LED_SMD:LED_0805_2012Metric" (at 118.11 144.78 0)
+    (property "Footprint" "LED_THT:LED_D3.0mm" (at 118.11 144.78 0)
       (effects (font (size 1.27 1.27)) hide)
     )

Commit message: more and more and more and more and more routing
Parts:
- removed C85, C86: 4.7uF, Capacitor_SMD:C_0805_2012Metric, symbol Device:C
Changed lines of the file:
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@@
   (junction (at 165.1 62.23) (diameter 0) (color 0 0 0 0)
   )
-  (junction (at 72.39 153.67) (diameter 0) (color 0 0 0 0)
-  )
   (junction (at 179.07 100.33) (diameter 0) (color 0 0 0 0)
   )
@@
   (junction (at 203.2 100.33) (diameter 0) (color 0 0 0 0)
   )
-  (junction (at 72.39 138.43) (diameter 0) (color 0 0 0 0)
-  )
   (junction (at 236.22 102.87) (diameter 0) (color 0 0 0 0)
   )
@@
   (junction (at 118.11 123.19) (diameter 0) (color 0 0 0 0)
   )
-  (junction (at 72.39 146.05) (diameter 0) (color 0 0 0 0)
-  )
   (junction (at 128.27 62.23) (diameter 0) (color 0 0 0 0)
   )
@@
     (stroke (width 0) (type default))
   )
-  (wire (pts (xy 72.39 146.05) (xy 78.74 146.05))
-    (stroke (width 0) (type default))
-  )
   (wire (pts (xy 128.27 73.66) (xy 128.27 62.23))
     (stroke (width 0) (type default))
@@
     (stroke (width 0) (type default))
   )
-  (wire (pts (xy 68.58 146.05) (xy 72.39 146.05))
+  (wire (pts (xy 68.58 146.05) (xy 78.74 146.05))
     (stroke (width 0) (type default))
   )
@@
         (path "/9021c97e-351f-4ed9-b393-50257df6a463/00000000-0000-0000-0000-0000659a4e2e"
           (reference "#PWR?") (unit 1)
-        )
-      )
-    )
-  )
-  (symbol (lib_id "Device:C") (at 72.39 142.24 180) (unit 1)
-    (in_bom yes) (on_board yes) (dnp no)
-    (property "Reference" "C85" (at 78.7908 142.24 90)
-      (effects (font (size 1.27 1.27)))
-    )
-    (property "Value" "4.7uF" (at 76.4794 142.24 90)
-      (effects (font (size 1.27 1.27)))
-    )
-    (property "Footprint" "Capacitor_SMD:C_0805_2012Metric" (at 71.4248 138.43 0)
-      (effects (font (size 1.27 1.27)) hide)
-    )
-    (property "Datasheet" "~" (at 72.39 142.24 0)
-      (effects (font (size 1.27 1.27)) hide)
-    )
-    (pin "1")
-    (pin "2")
-    (instances
-      (project "SynthProj"
-        (path "/9021c97e-351f-4ed9-b393-50257df6a463/00000000-0000-0000-0000-00006579d07e"
-          (reference "C85") (unit 1)
-        )
-        (path "/9021c97e-351f-4ed9-b393-50257df6a463/00000000-0000-0000-0000-0000659a4e2e"
-          (reference "C?") (unit 1)
         )
       )
@@
         )
       )
-    )
-  )
-  (symbol (lib_id "Device:C") (at 72.39 149.86 180) (unit 1)
-    (in_bom yes) (on_board yes) (dnp no)
-    (property "Reference" "C86" (at 78.7908 149.86 90)
-      (effects (font (size 1.27 1.27)))
-    )
-    (property "Value" "4.7uF" (at 76.4794 149.86 90)
-      (effects (font (size 1.27 1.27)))
-    )
-    (property "Footprint" "Capacitor_SMD:C_0805_2012Metric" (at 71.4248 146.05 0)
-      (effects (font (size 1.27 1.27)) hide)
-    )
-    (property "Datasheet" "~" (at 72.39 149.86 0)
-      (effects (font (size 1.27 1.27)) hide)
-    )
-    (pin "1")
-    (pin "2")
-    (instances
-      (project "SynthProj"
-        (path "/9021c97e-351f-4ed9-b393-50257df6a463/00000000-0000-0000-0000-00006579d07e"
-          (reference "C86") (unit 1)
-        )
-      )

Commit message: created manufacturing files
Parts:
- removed C92: 100nF, Capacitor_SMD:C_0603_1608Metric, symbol Device:C
- added C79: 10uF, Capacitor_SMD:C_0805_2012Metric, symbol Device:C
- R163, R165: value 100k -> 2k
- R167: value 4.7k -> 50k
- RV36: value 100k -> 50k
- RV37, RV38: value 1M -> 50k
Connections:
- net GNDREF: now also C79.1
- net at R175.1, U16.10 (+): now also C79.2
Changed lines of the file:
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@@
       (effects (font (size 1.27 1.27)) (justify right))
     )
-    (property "Value" "100k" (at 74.4982 60.833 0)
+    (property "Value" "50k" (at 74.4982 60.833 0)
       (effects (font (size 1.27 1.27)) (justify right))
     )
@@
       (effects (font (size 1.27 1.27)))
     )
-    (property "Value" "100k" (at 87.63 56.7944 90)
+    (property "Value" "2k" (at 87.63 56.7944 90)
       (effects (font (size 1.27 1.27)))
     )
@@
       (effects (font (size 1.27 1.27)))
     )
-    (property "Value" "100k" (at 98.1456 63.5 90)
+    (property "Value" "2k" (at 98.1456 63.5 90)
       (effects (font (size 1.27 1.27)))
     )
@@
     )
     (property "Datasheet" "~" (at 95.25 63.5 0)
+      (effects (font (size 1.27 1.27)) hide)
+    )
+    (property "Field4" "" (at 95.25 63.5 90)
       (effects (font (size 1.27 1.27)) hide)
     )
@@
       (effects (font (size 1.27 1.27)))
     )
-    (property "Value" "4.7k" (at 97.79 115.2144 90)
+    (property "Value" "50k" (at 97.79 115.2144 90)
       (effects (font (size 1.27 1.27)))
     )
@@
       (effects (font (size 1.27 1.27)) (justify right))
     )
-    (property "Value" "1M" (at 108.077 121.4882 0)
+    (property "Value" "50k" (at 108.077 121.4882 0)
       (effects (font (size 1.27 1.27)) (justify right))
     )
@@
       (effects (font (size 1.27 1.27)) (justify right))
     )
-    (property "Value" "1M" (at 183.007 98.6282 0)
+    (property "Value" "50k" (at 183.007 98.6282 0)
       (effects (font (size 1.27 1.27)) (justify right))
     )
@@
     )
   )
-  (symbol (lib_id "Device:C") (at 203.2 105.41 0) (unit 1)
-    (in_bom yes) (on_board yes) (dnp no)
-    (property "Reference" "C92" (at 196.7992 105.41 90)
-      (effects (font (size 1.27 1.27)))
-    )
-    (property "Value" "100nF" (at 199.1106 105.41 90)
-      (effects (font (size 1.27 1.27)))
-    )
-    (property "Footprint" "Capacitor_SMD:C_0603_1608Metric" (at 204.1652 109.22 0)
-      (effects (font (size 1.27 1.27)) hide)
-    )
-    (property "Datasheet" "~" (at 203.2 105.41 0)
-      (effects (font (size 1.27 1.27)) hide)
-    )
-    (pin "2")
-    (pin "1")
-    (instances
-      (project "SynthProj"
-        (path "/9021c97e-351f-4ed9-b393-50257df6a463/00000000-0000-0000-0000-00006579d07e"
-          (reference "C92") (unit 1)
-        )
-        (path "/9021c97e-351f-4ed9-b393-50257df6a463/00000000-0000-0000-0000-0000659a4e2e"
-          (reference "C?") (unit 1)
-        )
-      )
-    )
-  )
   (symbol (lib_id "power:GNDREF") (at 203.2 111.76 0) (unit 1)
     (in_bom yes) (on_board yes) (dnp no)
@@
         )
       )
+    )
+  )
+  (symbol (lib_id "Device:C") (at 203.2 105.41 180) (unit 1)
+    (in_bom yes) (on_board yes) (dnp no)
+    (property "Reference" "C79" (at 209.6008 105.41 90)
+      (effects (font (size 1.27 1.27)))
+    )
+    (property "Value" "10uF" (at 207.2894 105.41 90)
+      (effects (font (size 1.27 1.27)))
+    )
+    (property "Footprint" "Capacitor_SMD:C_0805_2012Metric" (at 202.2348 101.6 0)
+      (effects (font (size 1.27 1.27)) hide)
+    )
+    (property "Datasheet" "~" (at 203.2 105.41 0)
+      (effects (font (size 1.27 1.27)) hide)
+    )
+    (pin "1")
+    (pin "2")
+    (instances
+      (project "SynthProj"
+        (path "/9021c97e-351f-4ed9-b393-50257df6a463/00000000-0000-0000-0000-00006579d07e"
+          (reference "C79") (unit 1)
+        )
+        (path "/9021c97e-351f-4ed9-b393-50257df6a463/00000000-0000-0000-0000-0000659a4e2e"
+          (reference "C?") (unit 1)
+        )
+      )
