File: VCA.kicad_sch (KiCad schematic)
At the start: 23 parts, among them SW8 SW_SPDT, U10 TL072, U9 LM13700

Commit message: more work...
Parts:
- C35, C36, C? (x2): footprint Capacitor_SMD:C_0805_2012Metric_Pad1.18x1.45mm_HandSolder -> Capacitor_SMD:C_0805_2012Metric
- R? (x13): footprint Resistor_SMD:R_0805_2012Metric_Pad1.20x1.40mm_HandSolder -> Resistor_SMD:R_0603_1608Metric
Changed lines of the file:
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@@
       (effects (font (size 1.27 1.27)))
     )
-    (property "Footprint" "Capacitor_SMD:C_0805_2012Metric_Pad1.18x1.45mm_HandSolder" (at 63.8048 119.38 0)
+    (property "Footprint" "Capacitor_SMD:C_0805_2012Metric" (at 63.8048 119.38 0)
       (effects (font (size 1.27 1.27)) hide)
     )
@@
       (effects (font (size 1.27 1.27)))
     )
-    (property "Footprint" "Capacitor_SMD:C_0805_2012Metric_Pad1.18x1.45mm_HandSolder" (at 63.8048 127 0)
+    (property "Footprint" "Capacitor_SMD:C_0805_2012Metric" (at 63.8048 127 0)
       (effects (font (size 1.27 1.27)) hide)
     )
@@
       (effects (font (size 1.27 1.27)))
     )
-    (property "Footprint" "Resistor_SMD:R_0805_2012Metric_Pad1.20x1.40mm_HandSolder" (at 102.616 54.356 90)
+    (property "Footprint" "Resistor_SMD:R_0603_1608Metric" (at 102.616 54.356 90)
       (effects (font (size 1.27 1.27)) hide)
     )
@@
       (effects (font (size 1.27 1.27)))
     )
-    (property "Footprint" "Resistor_SMD:R_0805_2012Metric_Pad1.20x1.40mm_HandSolder" (at 102.616 89.916 90)
+    (property "Footprint" "Resistor_SMD:R_0603_1608Metric" (at 102.616 89.916 90)
       (effects (font (size 1.27 1.27)) hide)
     )
@@
       (effects (font (size 1.27 1.27)))
     )
-    (property "Footprint" "Resistor_SMD:R_0805_2012Metric_Pad1.20x1.40mm_HandSolder" (at 61.976 100.076 90)
+    (property "Footprint" "Resistor_SMD:R_0603_1608Metric" (at 61.976 100.076 90)
       (effects (font (size 1.27 1.27)) hide)
     )
@@
       (effects (font (size 1.27 1.27)))
     )
-    (property "Footprint" "Resistor_SMD:R_0805_2012Metric_Pad1.20x1.40mm_HandSolder" (at 75.946 100.076 90)
+    (property "Footprint" "Resistor_SMD:R_0603_1608Metric" (at 75.946 100.076 90)
       (effects (font (size 1.27 1.27)) hide)
     )
@@
       (effects (font (size 1.27 1.27)))
     )
-    (property "Footprint" "Resistor_SMD:R_0805_2012Metric_Pad1.20x1.40mm_HandSolder" (at 135.636 89.916 90)
+    (property "Footprint" "Resistor_SMD:R_0603_1608Metric" (at 135.636 89.916 90)
       (effects (font (size 1.27 1.27)) hide)
     )
@@
       (effects (font (size 1.27 1.27)))
     )
-    (property "Footprint" "Resistor_SMD:R_0805_2012Metric_Pad1.20x1.40mm_HandSolder" (at 161.036 77.216 90)
+    (property "Footprint" "Resistor_SMD:R_0603_1608Metric" (at 161.036 77.216 90)
       (effects (font (size 1.27 1.27)) hide)
     )
@@
       (effects (font (size 1.27 1.27)))
     )
-    (property "Footprint" "Resistor_SMD:R_0805_2012Metric_Pad1.20x1.40mm_HandSolder" (at 182.626 87.376 90)
+    (property "Footprint" "Resistor_SMD:R_0603_1608Metric" (at 182.626 87.376 90)
       (effects (font (size 1.27 1.27)) hide)
     )
@@
       (effects (font (size 1.27 1.27)))
     )
-    (property "Footprint" "Resistor_SMD:R_0805_2012Metric_Pad1.20x1.40mm_HandSolder" (at 182.626 100.076 90)
+    (property "Footprint" "Resistor_SMD:R_0603_1608Metric" (at 182.626 100.076 90)
       (effects (font (size 1.27 1.27)) hide)
     )
@@
       (effects (font (size 1.27 1.27)))
     )
-    (property "Footprint" "Resistor_SMD:R_0805_2012Metric_Pad1.20x1.40mm_HandSolder" (at 168.656 100.076 90)
+    (property "Footprint" "Resistor_SMD:R_0603_1608Metric" (at 168.656 100.076 90)
       (effects (font (size 1.27 1.27)) hide)
     )
@@
       (effects (font (size 1.27 1.27)))
     )
-    (property "Footprint" "Resistor_SMD:R_0805_2012Metric_Pad1.20x1.40mm_HandSolder" (at 164.084 122.936 90)
+    (property "Footprint" "Resistor_SMD:R_0603_1608Metric" (at 164.084 122.936 90)
       (effects (font (size 1.27 1.27)) hide)
     )
@@
       (effects (font (size 1.27 1.27)))
     )
-    (property "Footprint" "Resistor_SMD:R_0805_2012Metric_Pad1.20x1.40mm_HandSolder" (at 112.776 120.396 90)
+    (property "Footprint" "Resistor_SMD:R_0603_1608Metric" (at 112.776 120.396 90)
       (effects (font (size 1.27 1.27)) hide)
     )
@@
       (effects (font (size 1.27 1.27)))
     )
-    (property "Footprint" "Resistor_SMD:R_0805_2012Metric_Pad1.20x1.40mm_HandSolder" (at 119.634 122.936 90)
+    (property "Footprint" "Resistor_SMD:R_0603_1608Metric" (at 119.634 122.936 90)
       (effects (font (size 1.27 1.27)) hide)
     )
@@
       (effects (font (size 1.27 1.27)) (justify left))
     )
-    (property "Footprint" "Capacitor_SMD:C_0805_2012Metric_Pad1.18x1.45mm_HandSolder" (at 97.79 120.3452 0)
+    (property "Footprint" "Capacitor_SMD:C_0805_2012Metric" (at 97.79 120.3452 0)
       (effects (font (size 1.27 1.27)) hide)
     )
@@
       (effects (font (size 1.27 1.27)))
     )
-    (property "Footprint" "Resistor_SMD:R_0805_2012Metric_Pad1.20x1.40mm_HandSolder" (at 141.986 136.906 90)
+    (property "Footprint" "Resistor_SMD:R_0603_1608Metric" (at 141.986 136.906 90)
       (effects (font (size 1.27 1.27)) hide)
     )
@@
       (effects (font (size 1.27 1.27)) (justify left))
     )
-    (property "Footprint" "Capacitor_SMD:C_0805_2012Metric_Pad1.18x1.45mm_HandSolder" (at 175.26 120.3452 0)
-      (effects (font (size 1.27 1.27)) hide)
-    )
+    (property "Footprint" "Capacitor_SMD:C_0805_2012Metric" (at 175.26 120.3452 0)
+      (effects (font (size 1.27 1.27)) hide)
+    )

Commit message: finishing schematic 1.0
Parts:
- SW8: footprint SynthProjConnectors:ST-0-102-A01-T000-LF -> SynthProjConnectors:MTS-103-A01-T0

Commit message: lots of routes, added vco3, lfo2.
Parts:
- SW8: footprint SynthProjConnectors:MTS-103-A01-T0 -> SynthProjConnectors:SMTS-102
Changed lines of the file:
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@@
       (effects (font (size 1.27 1.27)))
     )
-    (property "Footprint" "SynthProjConnectors:MTS-103-A01-T0" (at 76.2 45.72 0)
+    (property "Footprint" "SynthProjConnectors:SMTS-102" (at 76.2 45.72 0)
       (effects (font (size 1.27 1.27)) hide)
     )

Commit message: more and more routing
Changed lines of the file:
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@@
     (effects (font (size 1.27 1.27)) (justify left bottom))
   )
-  (text "VCA Modulation" (at 86.36 50.8 0)
+  (text "VCA Modulation" (at 86.36 45.72 0)
     (effects (font (size 1.27 1.27)) (justify left bottom))
   )

Commit message: more and more and more and more and more routing
Parts:
- added C98, C99: 470nF, Capacitor_SMD:C_0805_2012Metric, symbol Device:C
Connections:
- net +12V: now also C98.2
- net -12V: now also C99.1
- net GNDREF: now also C98.1, C99.2
Changed lines of the file:
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@@
   (junction (at 120.65 119.38) (diameter 0) (color 0 0 0 0)
   )
+  (junction (at 64.77 134.62) (diameter 0) (color 0 0 0 0)
+  )
   (junction (at 64.77 127) (diameter 0) (color 0 0 0 0)
   )
@@
   (junction (at 119.38 88.9) (diameter 0) (color 0 0 0 0)
   )
+  (junction (at 71.755 127) (diameter 0) (color 0 0 0 0)
+  )
+  (junction (at 64.77 119.38) (diameter 0) (color 0 0 0 0)
+  )
   (junction (at 167.64 76.2) (diameter 0) (color 0 0 0 0)
   )
@@
     (stroke (width 0) (type default))
   )
+  (wire (pts (xy 64.77 127) (xy 71.755 127))
+    (stroke (width 0) (type default))
+  )
   (wire (pts (xy 120.65 119.38) (xy 129.54 119.38))
     (stroke (width 0) (type default))
@@
     (stroke (width 0) (type default))
   )
+  (wire (pts (xy 64.77 119.38) (xy 71.755 119.38))
+    (stroke (width 0) (type default))
+  )
   (wire (pts (xy 106.68 53.34) (xy 110.49 53.34))
     (stroke (width 0) (type default))
@@
   )
   (wire (pts (xy 167.64 86.36) (xy 167.64 76.2))
+    (stroke (width 0) (type default))
+  )
+  (wire (pts (xy 64.77 134.62) (xy 71.755 134.62))
     (stroke (width 0) (type default))
   )
@@
         )
       )
+    )
+  )
+  (symbol (lib_id "Device:C") (at 71.755 130.81 180) (unit 1)
+    (in_bom yes) (on_board yes) (dnp no)
+    (property "Reference" "C99" (at 78.1558 130.81 90)
+      (effects (font (size 1.27 1.27)))
+    )
+    (property "Value" "470nF" (at 75.8444 130.81 90)
+      (effects (font (size 1.27 1.27)))
+    )
+    (property "Footprint" "Capacitor_SMD:C_0805_2012Metric" (at 70.7898 127 0)
+      (effects (font (size 1.27 1.27)) hide)
+    )
+    (property "Datasheet" "~" (at 71.755 130.81 0)
+      (effects (font (size 1.27 1.27)) hide)
+    )
+    (pin "1")
+    (pin "2")
+    (instances
+      (project "SynthProj"
+        (path "/9021c97e-351f-4ed9-b393-50257df6a463/00000000-0000-0000-0000-000066d02a14"
+          (reference "C99") (unit 1)
+        )
+      )
+    )
+  )
+  (symbol (lib_id "Device:C") (at 71.755 123.19 180) (unit 1)
+    (in_bom yes) (on_board yes) (dnp no)
+    (property "Reference" "C98" (at 78.1558 123.19 90)
+      (effects (font (size 1.27 1.27)))
+    )
+    (property "Value" "470nF" (at 75.8444 123.19 90)
+      (effects (font (size 1.27 1.27)))
+    )
+    (property "Footprint" "Capacitor_SMD:C_0805_2012Metric" (at 70.7898 119.38 0)
+      (effects (font (size 1.27 1.27)) hide)
+    )
+    (property "Datasheet" "~" (at 71.755 123.19 0)
+      (effects (font (size 1.27 1.27)) hide)
+    )
+    (pin "1")
+    (pin "2")
+    (instances
+      (project "SynthProj"
+        (path "/9021c97e-351f-4ed9-b393-50257df6a463/00000000-0000-0000-0000-000066d02a14"
+          (reference "C98") (unit 1)
+        )
+        (path "/9021c97e-351f-4ed9-b393-50257df6a463/00000000-0000-0000-0000-00006611e0f5"
+          (reference "C?") (unit 1)
+        )
+      )

Commit message: created manufacturing files
Parts:
- RV? (x3): value 100k -> 50k
Other:
- note added: "Audio taper potentiometer"
Changed lines of the file:
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@@
+    (effects (font (size 1.27 1.27)) (justify left bottom))
+  )
+  (text "Audio taper potentiometer" (at 189.23 116.84 0)
     (effects (font (size 1.27 1.27)) (justify left bottom))
   )
@@
       (effects (font (size 1.27 1.27)) (justify right))
     )
-    (property "Value" "100k" (at 83.3882 54.483 0)
+    (property "Value" "50k" (at 83.3882 54.483 0)
       (effects (font (size 1.27 1.27)) (justify right))
     )
@@
       (effects (font (size 1.27 1.27)) (justify right))
     )
-    (property "Value" "100k" (at 66.8782 90.043 0)
+    (property "Value" "50k" (at 66.8782 90.043 0)
       (effects (font (size 1.27 1.27)) (justify right))
     )
@@
       (effects (font (size 1.27 1.27)) (justify right))
     )
-    (property "Value" "100k" (at 193.8782 129.413 0)
+    (property "Value" "50k" (at 193.8782 129.413 0)
       (effects (font (size 1.27 1.27)) (justify right))
     )
