File: VCO2.kicad_sch (KiCad schematic)
At the start: 61 parts, among them SW6 SW_SPDT, SW7 SW_SPDT, U6 TL072, U7 TL072, U8 TL072

Commit message: more and more and more and more and more routing
Parts:
- removed C? (x2): 4.7uF, Capacitor_SMD:C_0805_2012Metric, symbol Device:C
- removed C? (x2): 47nF, Capacitor_SMD:C_0603_1608Metric, symbol Device:C
- added C? (x4): 470nF, Capacitor_SMD:C_0805_2012Metric, symbol Device:C
Connections:
- net +12V: now also C?.2, C?.2
- net -12V: now also C?.1, C?.1
- net GNDREF: now also C?.1, C?.1, C?.2, C?.2

Commit message: created manufacturing files
Parts:
- R? (x4), RV? (x3): value 100k -> 50k
Changed lines of the file:
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@@
       (effects (font (size 1.27 1.27)) (justify right))
     )
-    (property "Value" "100k" (at 75.057 57.9882 0)
+    (property "Value" "50k" (at 75.057 57.9882 0)
       (effects (font (size 1.27 1.27)) (justify right))
     )
@@
       (effects (font (size 1.27 1.27)) (justify right))
     )
-    (property "Value" "100k" (at 76.327 40.2082 0)
+    (property "Value" "50k" (at 76.327 40.2082 0)
       (effects (font (size 1.27 1.27)) (justify right))
     )
@@
       (effects (font (size 1.27 1.27)))
     )
-    (property "Value" "100k" (at 64.77 91.7956 90)
+    (property "Value" "50k" (at 64.77 91.7956 90)
       (effects (font (size 1.27 1.27)))
     )
@@
       (effects (font (size 1.27 1.27)))
     )
-    (property "Value" "100k" (at 69.85 103.2256 90)
+    (property "Value" "50k" (at 69.85 103.2256 90)
       (effects (font (size 1.27 1.27)))
     )
@@
       (effects (font (size 1.27 1.27)))
     )
-    (property "Value" "100k" (at 69.85 113.3856 90)
+    (property "Value" "50k" (at 69.85 113.3856 90)
       (effects (font (size 1.27 1.27)))
     )
@@
       (effects (font (size 1.27 1.27)))
     )
-    (property "Value" "100k" (at 69.85 122.2756 90)
+    (property "Value" "50k" (at 69.85 122.2756 90)
       (effects (font (size 1.27 1.27)))
     )
@@
       (effects (font (size 1.27 1.27)) (justify right))
     )
-    (property "Value" "100k" (at 242.443 136.3218 0)
+    (property "Value" "50k" (at 242.443 136.3218 0)
       (effects (font (size 1.27 1.27)) (justify right))
     )
