File: SynthFaceplate/AnalogSequencerFaceplate.kicad_pcb (KiCad board)
At the start: 2 copper layers, 421.2 x 160.6 mm, 601 parts, among them J1 PWM IN, J10 Mixer Ext InA, J11 S&H_Out, J12 LFO1_Out, J13 Gate, J14 1V/Oct CV, J16 LFO2_Out, J17 PWM IN, J18 Ext In, J19 Exp CV In, J2 Exp CV In, J20 ADEG1_OUT, J21 ADEG2_OUT, J22 Lin CV In, J23 Sync, J24 Sync, J25 Master Output, J3 Lin CV In, J30 Echo_DV, J31 Echo_Repeat, J32 Echo_CV_In, J33 Echo_ExtIn, J34 ECHO_OUT, J39 Noise Out, J4 Sync, J46 Mixer Ext InB, J47 Mixer Ext InC, J5 Conn_01x16_Pin, J6 S&H_In, J7 Lin CV In, J8 Exp CV In, J9 PWM IN, Q1 MMBF4393LT1G, Q10 MMBT3904-7-F, Q11 MMBT3904-7-F, Q12 MMBF4391LT1G, Q13 MMBT3904-7-F, Q14 MMBT3904-7-F, Q15 MMBT3906LT1G, Q16 MMBF5457, Q17 MMBF5457, Q18 MMBT3906LT1G, Q19 MMBF5457, Q2 MMBT3904-7-F, Q20 MMBT3904-7-F, Q21 MMBT3904-7-F, Q22 MMBT3904-7-F, Q23 MMBT3906LT1G, Q24 MMBT3906LT1G, Q25 MMBT3904-7-F, Q26 MMBF4391LT1G, Q27 MMBT3904-7-F, Q3 MMBT3906LT1G, Q4 MMBT3904-7-F, Q5 MMBT3906LT1G, Q6 MMBF4393LT1G, Q7 MMBT3904-7-F, Q8 MMBT3904-7-F, Q9 MMBF4391LT1G, SW1 SW_SPST, SW10 SW_SPDT, SW11 SW_SPDT, SW12 SMTS-103-A1-T0, SW13 SW_Push_DPDT, SW14 SW_SPST, SW15 SW_Push, SW16 SW_SPST, SW17 SW_SPDT, SW18 SW_SPDT, SW19 SW_Push, SW2 SW_SPDT, SW20 SW_DPST, SW21 SW_DPST, SW22 SW_SPST, SW23 SW_SPST, SW24 SW_SPDT, SW25 SW_SPDT, SW26 SW_SPDT, SW27 SMTS-103-A1-T0, SW28 SW_Push_DPDT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

Commit message: working on face plate.
Parts:
- removed C1, C115, C116, C47, C48, C58, C60, C76: 1uF, Capacitor_SMD:C_0805_2012Metric
- removed C100, C104, C17, C21, C29, C33: 1nF, Capacitor_SMD:C_0603_1608Metric
- removed C101, C18, C30: 100pF, Capacitor_SMD:C_0603_1608Metric
- removed C102, C19, C31: 5n, Capacitor_SMD:C_0603_1608Metric
- removed C103, C105, C20, C22, C32, C34, C57, C59: 4.7pF, Capacitor_SMD:C_0603_1608Metric
- removed C114, C45, C46, C56: 100nF, Capacitor_SMD:C_0603_1608Metric
- removed C13, C14, C15, C16, C2, C23, C24, C25, C26, C27, C28, C3, C41, C42, C51, C52, C6, C7, C81, C94, C95, C96, C97: 470nF, Capacitor_SMD:C_0805_2012Metric
- removed C55, C78: 10uF, Capacitor_SMD:C_0805_2012Metric
- removed C72: 2.2nF, Capacitor_SMD:C_0603_1608Metric
- removed D13, D14, D15, D16, D18, D2, D26, D27, D29, D3, D30, D34, D35, D4, D5: 1N914, Diode_SMD:D_SOD-323F
- removed D20, D21, D22, D23: MMSZ5231B-7-F, Diode_SMD:D_SOD-123
- removed the G*** at (86.8, 233.9)
- removed H1, H2, H3, H4: MountingHole, MountingHole:MountingHole_3.2mm_M3_Pad
- removed J1, J17, J9: PWM IN, SynthProjConnectors:PJ-301-BM
- removed J10: Mixer Ext InA, SynthProjConnectors:PJ-301-BM
- removed J11: S&H_Out, SynthProjConnectors:PJ-301-BM
- removed J12: LFO1_Out, SynthProjConnectors:PJ-301-BM
- removed J13: Gate, SynthProjConnectors:PJ-301-BM
- removed J14: 1V/Oct CV, SynthProjConnectors:PJ-301-BM
- removed J16: LFO2_Out, SynthProjConnectors:PJ-301-BM
- removed J18: Ext In, SynthProjConnectors:PJ-301-BM
- removed J19, J2, J8: Exp CV In, SynthProjConnectors:PJ-301-BM
- removed J20: ADEG1_OUT, SynthProjConnectors:PJ-301-BM
- removed J21: ADEG2_OUT, SynthProjConnectors:PJ-301-BM
- removed J22, J3, J7: Lin CV In, SynthProjConnectors:PJ-301-BM
- removed J23, J24, J4: Sync, SynthProjConnectors:PJ-301-BM
- removed J30: Echo_DV, SynthProjConnectors:PJ-301-BM
- removed J31: Echo_Repeat, SynthProjConnectors:PJ-301-BM
- removed J32: Echo_CV_In, SynthProjConnectors:PJ-301-BM
- removed J33: Echo_ExtIn, SynthProjConnectors:PJ-301-BM
- removed J34: ECHO_OUT, SynthProjConnectors:PJ-301-BM
- removed J39: Noise Out, SynthProjConnectors:PJ-301-BM
- removed J46: Mixer Ext InB, SynthProjConnectors:PJ-301-BM
- removed J47: Mixer Ext InC, SynthProjConnectors:PJ-301-BM
- removed J5: Conn_01x16_Pin, Connector_PinHeader_2.54mm:PinHeader_2x08_P2.54mm_Vertical
- removed J6: S&H_In, SynthProjConnectors:PJ-301-BM
- removed Q10, Q11, Q13, Q20, Q25, Q7, Q8: MMBT3904-7-F, Package_TO_SOT_SMD:SOT-23-3
- removed Q12, Q26, Q9: MMBF4391LT1G, Package_TO_SOT_SMD:SOT-23-3
- removed Q15, Q18: MMBT3906LT1G, Package_TO_SOT_SMD:SOT-23-3
- removed Q16, Q17: MMBF5457, Package_TO_SOT_SMD:SOT-23-3
- removed R111, R112, R113, R114, R137, R140, R222, R244, R245: 200k, Resistor_SMD:R_0603_1608Metric
- removed R115: 680k, Resistor_SMD:R_0603_1608Metric
- removed R116, R134, R135, R141, R191, R193, R194, R197, R44, R46, R47, R50, R78, R80, R81, R84: 10k, Resistor_SMD:R_0603_1608Metric
- removed R117, R120, R122, R144, R151, R153, R187, R200, R207, R40, R53, R60, R74, R87, R94: 1M, Resistor_SMD:R_0603_1608Metric
- removed R118, R190, R43, R77: 1k, Resistor_SMD:R_0603_1608Metric
- removed R119, R121, R186, R188, R202, R3, R31, R33, R34, R35, R39, R41, R55, R73, R75, R89: 100k, Resistor_SMD:R_0603_1608Metric
- removed R146: 30k, Resistor_SMD:R_0603_1608Metric
- removed R147: 5.1k, Resistor_SMD:R_0603_1608Metric
- removed R149, R152, R196, R208, R49, R61, R83, R95: 47k, Resistor_SMD:R_0603_1608Metric
- removed R150: 91K, Resistor_SMD:R_0603_1608Metric
- removed R154, R161, R179, R32, R66: 39k, Resistor_SMD:R_0603_1608Metric
- removed R156, R178, R180, R181, R182, R65, R67, R68, R69: 50k, Resistor_SMD:R_0603_1608Metric
- removed R177, R30, R64: 4.7M, Resistor_SMD:R_0603_1608Metric
- removed R183, R198, R36, R51, R70, R85: 2k, Resistor_SMD:R_0603_1608Metric
- removed R184, R37, R71: 36k, Resistor_SMD:R_0603_1608Metric
- removed R185, R38, R72: 475, Resistor_SMD:R_0603_1608Metric
- removed R189, R209, R42, R62, R76, R96: 4.7k, Resistor_SMD:R_0603_1608Metric
- removed R192, R45, R79: 1.2M, Resistor_SMD:R_0603_1608Metric
- removed R195, R48, R82: 9.1k, Resistor_SMD:R_0603_1608Metric
- removed R199, R52, R86: 110k, Resistor_SMD:R_0603_1608Metric
- removed R201, R206, R54, R59, R88, R93: 20k, Resistor_SMD:R_0603_1608Metric
- removed R203, R56, R90: 3k, Resistor_SMD:R_0603_1608Metric
- removed R204, R57, R91: 18k, Resistor_SMD:R_0603_1608Metric
- removed R205, R58, R92: 22k, Resistor_SMD:R_0603_1608Metric
- removed R210, R63, R97: 3.3k, Resistor_SMD:R_0603_1608Metric
- removed RV10, RV15, RV45: 100, Potentiometer_SMD:Potentiometer_Bourns_TC33X_Vertical
- removed RV11, RV16, RV25, RV46: 100k, Potentiometer_SMD:Potentiometer_Bourns_TC33X_Vertical
- removed RV12, RV13, RV14, RV17, RV21, RV22, RV23, RV24, RV28, RV30, RV31, RV32, RV33, RV35, RV42, RV43, RV44, RV47, RV50, RV52, RV8, RV9: 50k, Potentiometer_THT:Potentiometer_Alps_RK09K_Single_Vertical
- removed U11: TL071, Package_SO:SO-8_3.9x4.9mm_P1.27mm
- removed U12: TL072, Package_SO:SOP-8_3.9x4.9mm_P1.27mm
- removed U15: TL074, Package_SO:SO-14_3.9x8.65mm_P1.27mm
- removed U17, U18, U19, U3, U4, U5, U6, U7, U8: TL072, Package_SO:SO-8_3.9x4.9mm_P1.27mm
- removed U31: PT2399, Package_SO:SOP-16_4.55x10.3mm_P1.27mm
- added G***: LOGO, SequencerGraphics:Dial, F.Cu at (105.0, 122.4)
- added G***: LOGO, SequencerGraphics:Dial, F.Cu at (79.7, 103.4)
- added G***: LOGO, SequencerGraphics:Dial, F.Cu at (79.7, 122.4)
- added G***: LOGO, SequencerGraphics:Dial, F.Cu at (105.0, 103.4)
- added G***: LOGO, SequencerGraphics:Dial, F.Cu at (181.0, 122.4)
- added G***: LOGO, SequencerGraphics:Dial, F.Cu at (130.3, 122.4)
- added G***: LOGO, SequencerGraphics:Dial, F.Cu at (181.0, 103.4)
- added G***: LOGO, SequencerGraphics:Dial, F.Cu at (105.1, 160.4)
- added G***: LOGO, SequencerGraphics:Dial, F.Cu at (181.0, 160.4)
- added G***: LOGO, SequencerGraphics:Dial, F.Cu at (130.4, 160.4)
- added G***: LOGO, SequencerGraphics:Dial, F.Cu at (79.8, 160.4)
- added G***: LOGO, SequencerGraphics:Dial, F.Cu at (130.3, 103.4)
- added G***: LOGO, SequencerGraphics:Dial, F.Cu at (181.0, 141.4)
Other:
- outline, holes or cut-outs redrawn
- board text added: "1 Exp"
- board text added: "1 Lin"
- board text added: "2 Exp"
- board text added: "2 Lin"
- board text added: "3 Exp"
- board text added: "3 Lin"
- board text added: "Coarse"
- board text added: "Fine"
- board text added: "PWM"
- board text added: "Pulse Width"
- board text added: "Sync"
- board text added: "VCO 1"
- board text added: "VCO 2"
- board text added: "VCO 3"
- board text removed: "External"
- board text removed: "Internal"
- board text removed: "Q Clock"
- board text removed: "Run"
- board text removed: "VCO2"
- board text removed: "VCO3"
